Commit message: Imported upstream version '2.2.1' of 'upstream'

File: clearpath_manipulators_description/srdf/arm/kinova_gen3_6dof.srdf.xacro (robot description, xacro)
@@ -1,14 +1,4 @@
 <?xml version="1.0" encoding="UTF-8"?>
 <robot xmlns:xacro="http://ros.org/wiki/xacro">
-  <xacro:macro name="kinova_gen3_6dof_group_state" params="name group_state joint_positions">
-    <group_state name="${group_state}" group="${name}">
-      <joint name="${name}_joint_1" value="${joint_positions[0]}"/>
-      <joint name="${name}_joint_2" value="${joint_positions[1]}"/>
-      <joint name="${name}_joint_3" value="${joint_positions[2]}"/>
-      <joint name="${name}_joint_4" value="${joint_positions[3]}"/>
-      <joint name="${name}_joint_5" value="${joint_positions[4]}"/>
-      <joint name="${name}_joint_6" value="${joint_positions[5]}"/>
-    </group_state>
-  </xacro:macro>
   <xacro:macro name="kinova_gen3_6dof" params="name">
     <group name="${name}">
@@ -20,14 +10,20 @@
         <joint name="${name}_joint_6"/>
     </group>
-    <xacro:kinova_gen3_6dof_group_state
-      name="${name}"
-      group_state="home"
-      joint_positions="${[0.0174, -0.5725, -0.9846, 0.1562, -1.0719, -1.7183]}"
-    />
-    <xacro:kinova_gen3_6dof_group_state
-      name="${name}"
-      group_state="zero"
-      joint_positions="${[0.0, 0.0, 0.0, 0.0, 0.0, 0.0]}"
-    />
+    <group_state name="home" group="${name}">
+        <joint name="${name}_joint_1" value="0.0174"/>
+        <joint name="${name}_joint_2" value="-0.5725"/>
+        <joint name="${name}_joint_3" value="-0.9846"/>
+        <joint name="${name}_joint_4" value="0.1562"/>
+        <joint name="${name}_joint_5" value="-1.0719"/>
+        <joint name="${name}_joint_6" value="-1.7183"/>
+    </group_state>
+    <group_state name="zero" group="${name}">
+        <joint name="${name}_joint_1" value="0"/>
+        <joint name="${name}_joint_2" value="0"/>
+        <joint name="${name}_joint_3" value="0"/>
+        <joint name="${name}_joint_4" value="0"/>
+        <joint name="${name}_joint_5" value="0"/>
+        <joint name="${name}_joint_6" value="0"/>
+    </group_state>
   </xacro:macro>
 </robot>

File: clearpath_manipulators_description/srdf/arm/kinova_gen3_7dof.srdf.xacro (robot description, xacro)
@@ -1,15 +1,4 @@
 <?xml version="1.0" encoding="UTF-8"?>
 <robot xmlns:xacro="http://ros.org/wiki/xacro">
-  <xacro:macro name="kinova_gen3_7dof_group_state" params="name group_state joint_positions">
-    <group_state name="${group_state}" group="${name}">
-      <joint name="${name}_joint_1" value="${joint_positions[0]}"/>
-      <joint name="${name}_joint_2" value="${joint_positions[1]}"/>
-      <joint name="${name}_joint_3" value="${joint_positions[2]}"/>
-      <joint name="${name}_joint_4" value="${joint_positions[3]}"/>
-      <joint name="${name}_joint_5" value="${joint_positions[4]}"/>
-      <joint name="${name}_joint_6" value="${joint_positions[5]}"/>
-      <joint name="${name}_joint_7" value="${joint_positions[6]}"/>
-    </group_state>
-  </xacro:macro>
   <xacro:macro name="kinova_gen3_7dof" params="name">
     <group name="${name}">
@@ -22,14 +11,22 @@
         <joint name="${name}_joint_7"/>
     </group>
-    <xacro:kinova_gen3_7dof_group_state
-      name="${name}"
-      group_state="home"
-      joint_positions="${[0.0174, -0.5725, -0.9846, 0.1562, -1.0719, -1.7183, -1.7183]}"
-    />
-    <xacro:kinova_gen3_7dof_group_state
-      name="${name}"
-      group_state="zero"
-      joint_positions="${[0.0, 0.0, 0.0, 0.0, 0.0, 0.0, 0.0]}"
-    />
+    <group_state name="home" group="${name}">
+        <joint name="${name}_joint_1" value="0.0174"/>
+        <joint name="${name}_joint_2" value="-0.5725"/>
+        <joint name="${name}_joint_3" value="-0.9846"/>
+        <joint name="${name}_joint_4" value="0.1562"/>
+        <joint name="${name}_joint_5" value="-1.0719"/>
+        <joint name="${name}_joint_6" value="-1.7183"/>
+        <joint name="${name}_joint_7" value="-1.7183"/>
+    </group_state>
+    <group_state name="zero" group="${name}">
+        <joint name="${name}_joint_1" value="0"/>
+        <joint name="${name}_joint_2" value="0"/>
+        <joint name="${name}_joint_3" value="0"/>
+        <joint name="${name}_joint_4" value="0"/>
+        <joint name="${name}_joint_5" value="0"/>
+        <joint name="${name}_joint_6" value="0"/>
+        <joint name="${name}_joint_7" value="0"/>
+    </group_state>
   </xacro:macro>
 </robot>

File: clearpath_manipulators_description/srdf/arm/kinova_gen3_lite.srdf.xacro (robot description, xacro)
@@ -1,14 +1,4 @@
 <?xml version="1.0" encoding="UTF-8"?>
 <robot xmlns:xacro="http://ros.org/wiki/xacro">
-  <xacro:macro name="kinova_gen3_lite_group_state" params="name group_state joint_positions">
-    <group_state name="${group_state}" group="${name}">
-      <joint name="${name}_joint_1" value="${joint_positions[0]}"/>
-      <joint name="${name}_joint_2" value="${joint_positions[1]}"/>
-      <joint name="${name}_joint_3" value="${joint_positions[2]}"/>
-      <joint name="${name}_joint_4" value="${joint_positions[3]}"/>
-      <joint name="${name}_joint_5" value="${joint_positions[4]}"/>
-      <joint name="${name}_joint_6" value="${joint_positions[5]}"/>
-    </group_state>
-  </xacro:macro>
   <xacro:macro name="kinova_gen3_lite" params="name">
     <group name="${name}">
@@ -44,14 +34,4 @@
         <joint name="${name}_joint_6" value="0"/>
     </group_state>
-    <xacro:kinova_gen3_lite_group_state
-      name="${name}"
-      group_state="home"
-      joint_positions="${[0.0, 0.0, math.pi * 1/2, math.pi * 1/2, math.pi * 1/2, math.pi * -1/2]}"
-    />
-    <xacro:kinova_gen3_lite_group_state
-      name="${name}"
-      group_state="zero"
-      joint_positions="${[0.0, 0.0, 0.0, 0.0, 0.0, 0.0]}"
-    />
   </xacro:macro>
 </robot>

File: clearpath_manipulators_description/srdf/arm/universal_robots.srdf.xacro (robot description, xacro)
@@ -1,14 +1,4 @@
 <?xml version="1.0" encoding="UTF-8"?>
 <robot xmlns:xacro="http://ros.org/wiki/xacro">
-  <xacro:macro name="universal_robots_group_state" params="name group_state joint_positions">
-    <group_state name="${group_state}" group="${name}">
-      <joint name="${name}_shoulder_pan_joint"  value="${joint_positions[0]}"/>
-      <joint name="${name}_shoulder_lift_joint" value="${joint_positions[1]}"/>
-      <joint name="${name}_elbow_joint"         value="${joint_positions[2]}"/>
-      <joint name="${name}_wrist_1_joint"       value="${joint_positions[3]}"/>
-      <joint name="${name}_wrist_2_joint"       value="${joint_positions[4]}"/>
-      <joint name="${name}_wrist_3_joint"       value="${joint_positions[5]}"/>
-    </group_state>
-  </xacro:macro>
   <xacro:macro name="universal_robots" params="name">
     <group name="${name}">
@@ -20,14 +10,28 @@
         <joint name="${name}_wrist_3_joint"/>
     </group>
-    <xacro:universal_robots_group_state
-      name="${name}"
-      group_state="home"
-      joint_positions="${[0.0, -1.5707, 1.5707, -1.5707, -1.5707, 0.0]}"
-    />
-    <xacro:universal_robots_group_state
-      name="${name}"
-      group_state="zero"
-      joint_positions="${[0.0, 0.0, 0.0, 0.0, 0.0, 0.0]}"
-    />
+    <group_state name="home" group="${name}">
+        <joint name="${name}_shoulder_pan_joint" value="0.0"/>
+        <joint name="${name}_shoulder_lift_joint" value="-1.5707"/>
+        <joint name="${name}_elbow_joint" value="1.5707"/>
+        <joint name="${name}_wrist_1_joint" value="-1.5707"/>
+        <joint name="${name}_wrist_2_joint" value="-1.5707"/>
+        <joint name="${name}_wrist_3_joint" value="0.0"/>
+      </group_state>
+    <group_state name="stow" group="${name}">
+      <joint name="${name}_shoulder_pan_joint" value="0.0"/>
+      <joint name="${name}_shoulder_lift_joint" value="-2.356"/>
+      <joint name="${name}_elbow_joint" value="2.356"/>
+      <joint name="${name}_wrist_1_joint" value="-1.5707"/>
+      <joint name="${name}_wrist_2_joint" value="-1.5707"/>
+      <joint name="${name}_wrist_3_joint" value="0.0"/>
+    </group_state>
+    <group_state name="zero" group="${name}">
+        <joint name="${name}_shoulder_pan_joint" value="0"/>
+        <joint name="${name}_shoulder_lift_joint" value="0"/>
+        <joint name="${name}_elbow_joint" value="0"/>
+        <joint name="${name}_wrist_1_joint" value="0"/>
+        <joint name="${name}_wrist_2_joint" value="0"/>
+        <joint name="${name}_wrist_3_joint" value="0"/>
+    </group_state>
   </xacro:macro>
 </robot>

File: clearpath_manipulators_description/srdf/gripper/kinova_2f_lite.srdf.xacro (robot description, xacro)
@@ -1,9 +1,4 @@
 <?xml version="1.0" encoding="UTF-8"?>
 <robot xmlns:xacro="http://ros.org/wiki/xacro">
-  <xacro:macro name="kinova_2f_lite_group_state" params="name group_state joint_positions">
-    <group_state name="${group_state}" group="${name}">
-      <joint name="${name}_right_finger_bottom_joint" value="${joint_positions[0]}"/>
-    </group_state>
-  </xacro:macro>
   <xacro:macro name="kinova_2f_lite" params="name">
     <group name="${name}">
@@ -13,14 +8,10 @@
         <joint name="${name}_left_finger_tip_joint"/>
     </group>
-    <xacro:kinova_2f_lite_group_state
-      name="${name}"
-      group_state="open"
-      joint_positions="${[0.0]}"
-    />
-    <xacro:kinova_2f_lite_group_state
-      name="${name}"
-      group_state="close"
-      joint_positions="${[0.85]}"
-    />
+    <group_state name="open" group="${name}">
+        <joint name="${name}_right_finger_bottom_joint" value="0.0"/>
+    </group_state>
+    <group_state name="close" group="${name}">
+        <joint name="${name}_right_finger_bottom_joint" value="0.85"/>
+    </group_state>
     <disable_collisions link1="${name}_right_finger_dist_link" link2="${name}_left_finger_dist_link" reason="User"/>
   </xacro:macro>

File: clearpath_manipulators_description/srdf/gripper/robotiq_2f_140.srdf.xacro (robot description, xacro)
@@ -1,9 +1,4 @@
 <?xml version="1.0" encoding="UTF-8"?>
 <robot xmlns:xacro="http://ros.org/wiki/xacro">
-  <xacro:macro name="robotiq_2f_140_group_state" params="name group_state joint_positions">
-    <group_state name="${group_state}" group="${name}">
-      <joint name="${name}_finger_joint" value="${joint_positions[0]}"/>
-    </group_state>
-  </xacro:macro>
   <xacro:macro name="robotiq_2f_140" params="name">
     <group name="${name}">
@@ -15,14 +10,10 @@
         <joint name="${name}_right_inner_finger_joint"/>
     </group>
-    <xacro:robotiq_2f_140_group_state
-      name="${name}"
-      group_state="open"
-      joint_positions="${[0.0]}"
-    />
-    <xacro:robotiq_2f_140_group_state
-      name="${name}"
-      group_state="close"
-      joint_positions="${[0.7]}"
-    />
+    <group_state name="open" group="${name}">
+        <joint name="${name}_finger_joint" value="0.0"/>
+    </group_state>
+    <group_state name="close" group="${name}">
+        <joint name="${name}_finger_joint" value="0.698"/>
+    </group_state>
     <disable_collisions link1="${name}_left_inner_knuckle" link2="${name}_left_inner_finger" reason="User"/>
     <disable_collisions link1="${name}_right_inner_knuckle" link2="${name}_right_inner_finger" reason="User"/>

File: clearpath_manipulators_description/srdf/gripper/robotiq_2f_85.srdf.xacro (robot description, xacro)
@@ -1,9 +1,4 @@
 <?xml version="1.0" encoding="UTF-8"?>
 <robot xmlns:xacro="http://ros.org/wiki/xacro">
-  <xacro:macro name="robotiq_2f_85_group_state" params="name group_state joint_positions">
-    <group_state name="${group_state}" group="${name}">
-      <joint name="${name}_robotiq_85_left_knuckle_joint" value="${joint_positions[0]}"/>
-    </group_state>
-  </xacro:macro>
   <xacro:macro name="robotiq_2f_85" params="name">
     <group name="${name}">
@@ -18,14 +13,10 @@
         <joint name="${name}_robotiq_85_right_finger_tip_joint"/>
     </group>
-    <xacro:robotiq_2f_85_group_state
-      name="${name}"
-      group_state="open"
-      joint_positions="${[0.0]}"
-    />
-    <xacro:robotiq_2f_85_group_state
-      name="${name}"
-      group_state="close"
-      joint_positions="${[0.8]}"
-    />
+    <group_state name="open" group="${name}">
+        <joint name="${name}_robotiq_85_left_knuckle_joint" value="0.0"/>
+    </group_state>
+    <group_state name="close" group="${name}">
+        <joint name="${name}_robotiq_85_left_knuckle_joint" value="0.8"/>
+    </group_state>
     <disable_collisions link1="${name}_robotiq_85_left_inner_knuckle_link" link2="${name}_robotiq_85_left_finger_tip_link" reason="User"/>
     <disable_collisions link1="${name}_robotiq_85_right_inner_knuckle_link" link2="${name}_robotiq_85_right_finger_tip_link" reason="User"/>

File: clearpath_manipulators_description/urdf/arm/kinova_gen3_6dof.urdf.xacro (robot description, xacro)
@@ -362,5 +362,5 @@
           </xacro:if>
           <xacro:if value="${sim_ignition}">
-            <plugin>ign_ros2_control/IgnitionSystem</plugin>
+            <plugin>gz_ros2_control/GazeboSimSystem</plugin>
           </xacro:if>
           <xacro:if value="${sim_isaac}">

File: clearpath_manipulators_description/urdf/arm/kinova_gen3_7dof.urdf.xacro (robot description, xacro)
@@ -477,5 +477,5 @@
           </xacro:if>
           <xacro:if value="${sim_ignition}">
-            <plugin>ign_ros2_control/IgnitionSystem</plugin>
+            <plugin>gz_ros2_control/GazeboSimSystem</plugin>
           </xacro:if>
           <xacro:if value="${sim_isaac}">

File: clearpath_manipulators_description/urdf/arm/kinova_gen3_lite.urdf.xacro (robot description, xacro)
@@ -243,5 +243,5 @@
           </xacro:if>
           <xacro:if value="${sim_ignition}">
-            <plugin>ign_ros2_control/IgnitionSystem</plugin>
+            <plugin>gz_ros2_control/GazeboSimSystem</plugin>
           </xacro:if>
           <xacro:if value="${sim_isaac}">
