Commit message: Imported upstream version '2.2.1' of 'upstream'

File: clearpath_manipulators_description/urdf/arm/universal_robots.urdf.xacro (robot description, xacro)
@@ -2,5 +2,5 @@
 <robot xmlns:xacro="http://ros.org/wiki/xacro">
   <xacro:arg name="is_sim" default="false"/>
-  <xacro:arg name="use_fake_hardware" default="false"/>
+  <xacro:arg name="use_mock_hardware" default="false"/>
   <xacro:arg name="use_manipulation_controllers" default="false"/>
   <xacro:include filename="$(find ur_description)/urdf/ur_macro.xacro"/>
@@ -19,5 +19,4 @@
     safety_pos_margin:=''
     safety_k_position:=''
-    generate_ros2_control_tag:=''
     headless_mode:=''
     robot_ip:=''
@@ -42,6 +41,6 @@
     tool_device_name:=''
     tool_tcp_port:=''
-    use_fake_hardware:=''
-    fake_sensor_commands:=''
+    use_mock_hardware:=''
+    mock_sensor_commands:=''
     sim_gazebo:=''
     sim_ignition:=''
@@ -57,5 +56,34 @@
     <xacro:property name="_safety_pos_margin" value="0.15" lazy_eval="false"/>
     <xacro:property name="_safety_k_position" value="20" lazy_eval="false"/>
-    <!-- Default Description Parameters Overwrites -->
+    <!-- Default ros2_control Parameters -->
+    <xacro:property name="_headless_mode" value="false" lazy_eval="false"/>
+    <xacro:property name="_robot_ip" value="192.168.131.40" lazy_eval="false"/>
+    <xacro:property name="_script_filename" value="$(find ur_client_library)/resources/external_control.urscript" lazy_eval="false"/>
+    <xacro:property name="_output_recipe_filename" value="$(find ur_robot_driver)/resources/rtde_output_recipe.txt" lazy_eval="false"/>
+    <xacro:property name="_input_recipe_filename" value="$(find ur_robot_driver)/resources/rtde_input_recipe.txt" lazy_eval="false"/>
+    <xacro:property name="_reverse_ip" value="0.0.0.0" lazy_eval="false"/>
+    <xacro:property name="_script_command_port" value="50004" lazy_eval="false"/>
+    <xacro:property name="_reverse_port" value="50001" lazy_eval="false"/>
+    <xacro:property name="_script_sender_port" value="50002" lazy_eval="false"/>
+    <xacro:property name="_trajectory_port" value="50003" lazy_eval="false"/>
+    <xacro:property name="_transmission_hw_interface" value="hardware_interface/PositionJointInterface" lazy_eval="false"/>
+    <xacro:property name="_non_blocking_read" value="true" lazy_eval="false"/>
+    <xacro:property name="_keep_alive_count" value="2.0" lazy_eval="false"/>
+    <!-- Default Tool Communication Parameters -->
+    <xacro:property name="_use_tool_communication" value="false" lazy_eval="false"/>
+    <xacro:property name="_tool_voltage" value="0" lazy_eval="false"/>
+    <xacro:property name="_tool_parity" value="0" lazy_eval="false"/>
+    <xacro:property name="_tool_baud_rate" value="115200" lazy_eval="false"/>
+    <xacro:property name="_tool_stop_bits" value="1" lazy_eval="false"/>
+    <xacro:property name="_tool_rx_idle_chars" value="1.5" lazy_eval="false"/>
+    <xacro:property name="_tool_tx_idle_chars" value="3.5" lazy_eval="false"/>
+    <xacro:property name="_tool_device_name" value="/tmp/ttyUR" lazy_eval="false"/>
+    <xacro:property name="_tool_tcp_port" value="54321" lazy_eval="false"/>
+    <!-- Default Simulation Parameters -->
+    <xacro:property name="_use_mock_hardware" value="false" />
+    <xacro:property name="_mock_sensor_commands" value="false" />
+    <xacro:property name="_sim_gazebo" value="false" />
+    <xacro:property name="_sim_ignition" value="$(arg is_sim)" />
+    <!-- Parameter Overwrites -->
     <xacro:if value="${initial_positions != ''}"> <xacro:property name="_initial_positions" value="${initial_positions}" lazy_eval="false"/> </xacro:if>
     <!-- if initial positions file is passed, overwrite initial positions parameter -->
@@ -68,30 +96,9 @@
     <xacro:if value="${safety_pos_margin != ''}"> <xacro:property name="_safety_pos_margin" value="${safety_pos_margin}" lazy_eval="false"/> </xacro:if>
     <xacro:if value="${safety_k_position != ''}"> <xacro:property name="_safety_k_position" value="${safety_k_position}" lazy_eval="false"/> </xacro:if>
-    <!-- Default Simulation Parameters -->
-    <xacro:property name="_use_fake_hardware" value="false" />
-    <xacro:property name="_fake_sensor_commands" value="false" />
-    <xacro:property name="_sim_gazebo" value="false" />
-    <xacro:property name="_sim_ignition" value="$(arg is_sim)" />
-    <!-- Default Simulation Parameters Overwrites -->
-    <xacro:if value="${use_fake_hardware != ''}"> <xacro:property name="_use_fake_hardware" value="${use_fake_hardware}" lazy_eval="false"/> </xacro:if>
-    <xacro:if value="${fake_sensor_commands != ''}"> <xacro:property name="_fake_sensor_commands" value="${fake_sensor_commands}" lazy_eval="false"/> </xacro:if>
-    <xacro:if value="${sim_gazebo != ''}"> <xacro:property name="_sim_gazebo" value="${sim_gazebo}" lazy_eval="false"/> </xacro:if>
-    <xacro:if value="${sim_ignition != ''}"> <xacro:property name="_sim_ignition" value="${sim_ignition}" lazy_eval="false"/> </xacro:if>
-    <!-- Default ros2_control Parameters -->
-    <xacro:property name="_generate_ros2_control_tag" value="$(arg use_manipulation_controllers)" lazy_eval="false"/>
-    <xacro:property name="_headless_mode" value="false" lazy_eval="false"/>
-    <xacro:property name="_robot_ip" value="192.168.131.40" lazy_eval="false"/>
-    <xacro:property name="_reverse_ip" value="0.0.0.0" lazy_eval="false"/>
-    <xacro:property name="_script_command_port" value="50004" lazy_eval="false"/>
-    <xacro:property name="_reverse_port" value="50001" lazy_eval="false"/>
-    <xacro:property name="_script_sender_port" value="50002" lazy_eval="false"/>
-    <xacro:property name="_trajectory_port" value="50003" lazy_eval="false"/>
-    <xacro:property name="_transmission_hw_interface" value="hardware_interface/PositionJointInterface" lazy_eval="false"/>
-    <xacro:property name="_non_blocking_read" value="true" lazy_eval="false"/>
-    <xacro:property name="_keep_alive_count" value="2.0" lazy_eval="false"/>
-    <!-- Default ros2_control Parameters Overwrites -->
-    <xacro:if value="${generate_ros2_control_tag != ''}"> <xacro:property name="_generate_ros2_control_tag" value="${generate_ros2_control_tag}" lazy_eval="false"/> </xacro:if>
     <xacro:if value="${headless_mode != ''}"> <xacro:property name="_headless_mode" value="${headless_mode}" lazy_eval="false"/> </xacro:if>
     <xacro:if value="${robot_ip != ''}"> <xacro:property name="_robot_ip" value="${robot_ip}" lazy_eval="false"/> </xacro:if>
+    <xacro:if value="${script_filename != ''}"> <xacro:property name="_script_filename" value="${script_filename}" lazy_eval="false"/> </xacro:if>
+    <xacro:if value="${output_recipe_filename != ''}"> <xacro:property name="_output_recipe_filename" value="${output_recipe_filename}" lazy_eval="false"/> </xacro:if>
+    <xacro:if value="${input_recipe_filename != ''}"> <xacro:property name="_input_recipe_filename" value="${input_recipe_filename}" lazy_eval="false"/> </xacro:if>
     <xacro:if value="${reverse_ip != ''}"> <xacro:property name="_reverse_ip" value="${reverse_ip}" lazy_eval="false"/> </xacro:if>
     <xacro:if value="${script_command_port != ''}"> <xacro:property name="_script_command_port" value="${script_command_port}" lazy_eval="false"/> </xacro:if>
@@ -102,30 +109,4 @@
     <xacro:if value="${non_blocking_read != ''}"> <xacro:property name="_non_blocking_read" value="${non_blocking_read}" lazy_eval="false"/> </xacro:if>
     <xacro:if value="${keep_alive_count != ''}"> <xacro:property name="_keep_alive_count" value="${keep_alive_count}" lazy_eval="false"/> </xacro:if>
-    <!-- Driver Dependent Parameters -->
-    <xacro:if value="${_generate_ros2_control_tag and not _use_fake_hardware and not _sim_ignition}">
-      <xacro:property name="_script_filename" value="$(find ur_client_library)/resources/external_control.urscript" lazy_eval="false"/>
-      <xacro:property name="_output_recipe_filename" value="$(find ur_robot_driver)/resources/rtde_output_recipe.txt" lazy_eval="false"/>
-      <xacro:property name="_input_recipe_filename" value="$(find ur_robot_driver)/resources/rtde_input_recipe.txt" lazy_eval="false"/>
-    </xacro:if>
-    <xacro:unless value="${_generate_ros2_control_tag and not _use_fake_hardware and not _sim_ignition}">
-      <xacro:property name="_script_filename" value="" lazy_eval="false"/>
-      <xacro:property name="_output_recipe_filename" value="" lazy_eval="false"/>
-      <xacro:property name="_input_recipe_filename" value="" lazy_eval="false"/>
-    </xacro:unless>
-    <!-- Driver Dependent Parameters Overwrites -->
-    <xacro:if value="${script_filename != ''}"> <xacro:property name="_script_filename" value="${script_filename}" lazy_eval="false"/> </xacro:if>
-    <xacro:if value="${output_recipe_filename != ''}"> <xacro:property name="_output_recipe_filename" value="${output_recipe_filename}" lazy_eval="false"/> </xacro:if>
-    <xacro:if value="${input_recipe_filename != ''}"> <xacro:property name="_input_recipe_filename" value="${input_recipe_filename}" lazy_eval="false"/> </xacro:if>
-    <!-- Default Tool Communication Parameters -->
-    <xacro:property name="_use_tool_communication" value="false" lazy_eval="false"/>
-    <xacro:property name="_tool_voltage" value="0" lazy_eval="false"/>
-    <xacro:property name="_tool_parity" value="0" lazy_eval="false"/>
-    <xacro:property name="_tool_baud_rate" value="115200" lazy_eval="false"/>
-    <xacro:property name="_tool_stop_bits" value="1" lazy_eval="false"/>
-    <xacro:property name="_tool_rx_idle_chars" value="1.5" lazy_eval="false"/>
-    <xacro:property name="_tool_tx_idle_chars" value="3.5" lazy_eval="false"/>
-    <xacro:property name="_tool_device_name" value="/tmp/ttyUR" lazy_eval="false"/>
-    <xacro:property name="_tool_tcp_port" value="54321" lazy_eval="false"/>
-    <!-- Tool Communication Parameter Overwrites -->
     <xacro:if value="${use_tool_communication != ''}"> <xacro:property name="_use_tool_communication" value="${use_tool_communication}" lazy_eval="false"/> </xacro:if>
     <xacro:if value="${tool_voltage != ''}"> <xacro:property name="_tool_voltage" value="${tool_voltage}" lazy_eval="false"/> </xacro:if>
@@ -137,10 +118,12 @@
     <xacro:if value="${tool_device_name != ''}"> <xacro:property name="_tool_device_name" value="${tool_device_name}" lazy_eval="false"/> </xacro:if>
     <xacro:if value="${tool_tcp_port != ''}"> <xacro:property name="_tool_tcp_port" value="${tool_tcp_port}" lazy_eval="false"/> </xacro:if>
-    <!-- Universal_Robots_ROS2_Description -->
+    <xacro:if value="${use_mock_hardware != ''}"> <xacro:property name="_use_mock_hardware" value="${use_mock_hardware}" lazy_eval="false"/> </xacro:if>
+    <xacro:if value="${mock_sensor_commands != ''}"> <xacro:property name="_mock_sensor_commands" value="${mock_sensor_commands}" lazy_eval="false"/> </xacro:if>
+    <xacro:if value="${sim_gazebo != ''}"> <xacro:property name="_sim_gazebo" value="${sim_gazebo}" lazy_eval="false"/> </xacro:if>
+    <xacro:if value="${sim_ignition != ''}"> <xacro:property name="_sim_ignition" value="${sim_ignition}" lazy_eval="false"/> </xacro:if>
     <xacro:ur_robot
       name="${name}"
+      tf_prefix="${_tf_prefix}"
       parent="${parent_link}"
-      tf_prefix="${_tf_prefix}"
-      initial_positions="${_initial_positions}"
       joint_limits_parameters_file="${_joint_limits_parameters_file}"
       kinematics_parameters_file="${_kinematics_parameters_file}"
@@ -150,33 +133,39 @@
       safety_pos_margin="${_safety_pos_margin}"
       safety_k_position="${_safety_k_position}"
-      generate_ros2_control_tag="${_generate_ros2_control_tag}"
-      headless_mode="${_headless_mode}"
-      robot_ip="${_robot_ip}"
-      script_filename="${_script_filename}"
-      output_recipe_filename="${_output_recipe_filename}"
-      input_recipe_filename="${_input_recipe_filename}"
-      reverse_ip="${_reverse_ip}"
-      script_command_port="${_script_command_port}"
-      reverse_port="${_reverse_port}"
-      script_sender_port="${_script_sender_port}"
-      trajectory_port="${_trajectory_port}"
-      transmission_hw_interface="${_transmission_hw_interface}"
-      non_blocking_read="{_non_blocking_read}"
-      use_tool_communication="${_use_tool_communication}"
-      tool_voltage="${_tool_voltage}"
-      tool_parity="${_tool_parity}"
-      tool_baud_rate="${_tool_baud_rate}"
-      tool_stop_bits="${_tool_stop_bits}"
-      tool_rx_idle_chars="${_tool_rx_idle_chars}"
-      tool_tx_idle_chars="${_tool_tx_idle_chars}"
-      tool_device_name="${_tool_device_name}"
-      tool_tcp_port="${_tool_tcp_port}"
-      use_fake_hardware="${_use_fake_hardware}"
-      fake_sensor_commands="${_fake_sensor_commands}"
-      sim_gazebo="${_sim_gazebo}"
-      sim_ignition="${_sim_ignition}"
       >
       <xacro:insert_block name="origin"/>
     </xacro:ur_robot>
+    <!-- Universal_Robots_ROS2_Driver HardwareInterface -->
+    <xacro:if value="$(arg use_manipulation_controllers)">
+      <xacro:include filename="$(find ur_robot_driver)/urdf/ur.ros2_control.xacro" />
+      <xacro:ur_ros2_control
+        name="${name}"
+        tf_prefix="${_tf_prefix}"
+        kinematics_parameters_file="${_kinematics_parameters_file}"
+        transmission_hw_interface="${_transmission_hw_interface}"
+        use_mock_hardware="${_use_mock_hardware}"
+        mock_sensor_commands="${_mock_sensor_commands}"
+        headless_mode="${_headless_mode}"
+        initial_positions="${_initial_positions}"
+        use_tool_communication="${_use_tool_communication}"
+        tool_voltage="${_tool_voltage}"
+        tool_parity="${_tool_parity}"
+        tool_baud_rate="${_tool_baud_rate}"
+        tool_stop_bits="${_tool_stop_bits}"
+        tool_rx_idle_chars="${_tool_rx_idle_chars}"
+        tool_tx_idle_chars="${_tool_tx_idle_chars}"
+        tool_device_name="${_tool_device_name}"
+        tool_tcp_port="${_tool_tcp_port}"
+        robot_ip="${_robot_ip}"
+        script_filename="${_script_filename}"
+        output_recipe_filename="${_output_recipe_filename}"
+        input_recipe_filename="${_input_recipe_filename}"
+        reverse_ip="${_reverse_ip}"
+        script_command_port="${_script_command_port}"
+        reverse_port="${_reverse_port}"
+        script_sender_port="${_script_sender_port}"
+        trajectory_port="${_trajectory_port}"
+      />
+    </xacro:if>
   </xacro:macro>
 </robot>

File: clearpath_manipulators_description/urdf/gripper/kinova_2f_lite.urdf.xacro (robot description, xacro)
@@ -196,5 +196,5 @@
             </xacro:if>
               <xacro:if value="${sim_ignition}">
-                  <plugin>ign_ros2_control/IgnitionSystem</plugin>
+                  <plugin>gz_ros2_control/GazeboSimSystem</plugin>
               </xacro:if>
               <xacro:if value="${use_fake_hardware}">

File: clearpath_manipulators_description/urdf/gripper/robotiq_2f_140.urdf.xacro (robot description, xacro)
@@ -283,5 +283,5 @@
           </xacro:if>
           <xacro:if value="${sim_gazebo}">
-            <plugin>ign_ros2_control/IgnitionSystem</plugin>
+            <plugin>gz_ros2_control/GazeboSimSystem</plugin>
           </xacro:if>
           <xacro:if value="${use_fake_hardware}">

File: clearpath_platform_description/urdf/a200/a200.urdf.xacro (robot description, xacro)
@@ -90,5 +90,5 @@
     </xacro:a200_wheel>
     <gazebo>
-      <plugin filename="libignition-gazebo-wheel-slip-system.so" name="ignition::gazebo::systems::WheelSlip">
+      <plugin filename="libgz-sim-wheel-slip-system.so" name="gz::sim::systems::WheelSlip">
         <wheel link_name="front_left_wheel">
           <slip_compliance_lateral>1.0</slip_compliance_lateral>
@@ -145,5 +145,5 @@
         <hardware>
           <xacro:if value="$(arg is_sim)">
-            <plugin>ign_ros2_control/IgnitionSystem</plugin>
+            <plugin>gz_ros2_control/GazeboSimSystem</plugin>
           </xacro:if>
           <xacro:unless value="$(arg is_sim)">

File: clearpath_platform_description/urdf/common.urdf.xacro (robot description, xacro)
@@ -113,25 +113,3 @@
       </xacro:if>
     </xacro:macro>
-    <xacro:macro name="clearpath_material" params="name:='' color_rgba:='' texture_file:=''">
-      <xacro:if value="${name != ''}">
-        <material name="${name}">
-          <xacro:if value="${color_rgba != ''}">
-            <color rgba="${color_rgba}"/>
-          </xacro:if>
-          <xacro:if value="${texture_file != ''}">
-            <texture filename="${texture_file}"/>
-          </xacro:if>
-        </material>
-      </xacro:if>
-      <xacro:unless value="${name != ''}">
-        <material>
-          <xacro:if value="${color_rgba != ''}">
-            <color rgba="${color_rgba}"/>
-          </xacro:if>
-          <xacro:if value="${texture_file != ''}">
-            <texture filename="${texture_file}"/>
-          </xacro:if>
-        </material>
-      </xacro:unless>
-    </xacro:macro>
 </robot>

File: clearpath_platform_description/urdf/dd100/dd100.urdf.xacro (robot description, xacro)
@@ -55,5 +55,5 @@
     </xacro:dd100_wheel>
     <gazebo>
-      <plugin filename="libignition-gazebo-wheel-slip-system.so" name="ignition::gazebo::systems::WheelSlip">
+      <plugin filename="libgz-sim-wheel-slip-system.so" name="gz::sim::systems::WheelSlip">
         <wheel link_name="front_left_wheel_link">
           <slip_compliance_lateral>1.0</slip_compliance_lateral>
@@ -135,5 +135,5 @@
         <update_rate>50</update_rate>
         <visualize>true</visualize>
-        <ignition_frame_id>imu_0_link</ignition_frame_id>
+        <gz_frame_id>imu_0_link</gz_frame_id>
         <topic>$(arg namespace)/sensors/imu_0/data_raw</topic>
       </sensor>
@@ -202,5 +202,5 @@
         <hardware>
           <xacro:if value="$(arg is_sim)">
-            <plugin>ign_ros2_control/IgnitionSystem</plugin>
+            <plugin>gz_ros2_control/GazeboSimSystem</plugin>
           </xacro:if>
           <xacro:unless value="$(arg is_sim)">

File: clearpath_platform_description/urdf/dd150/dd150.urdf.xacro (robot description, xacro)
@@ -55,5 +55,5 @@
     </xacro:dd150_wheel>
     <gazebo>
-      <plugin filename="libignition-gazebo-wheel-slip-system.so" name="ignition::gazebo::systems::WheelSlip">
+      <plugin filename="libgz-sim-wheel-slip-system.so" name="gz::sim::systems::WheelSlip">
         <wheel link_name="front_left_wheel_link">
           <slip_compliance_lateral>1.0</slip_compliance_lateral>
@@ -135,5 +135,5 @@
         <update_rate>50</update_rate>
         <visualize>true</visualize>
-        <ignition_frame_id>imu_0_link</ignition_frame_id>
+        <gz_frame_id>imu_0_link</gz_frame_id>
         <topic>$(arg namespace)/sensors/imu_0/data_raw</topic>
       </sensor>
@@ -190,5 +190,5 @@
         <hardware>
           <xacro:if value="$(arg is_sim)">
-            <plugin>ign_ros2_control/IgnitionSystem</plugin>
+            <plugin>gz_ros2_control/GazeboSimSystem</plugin>
           </xacro:if>
           <xacro:unless value="$(arg is_sim)">

File: clearpath_platform_description/urdf/do100/do100.urdf.xacro (robot description, xacro)
@@ -4,5 +4,4 @@
   <xacro:arg name="is_sim" default="false" />
   <xacro:arg name="gazebo_controllers" default="$(find clearpath_control)/config/do100/control.yaml"/>
-  <xacro:arg name="use_platform_controllers" default="true"/>
   <!-- Included URDF/Xacro Files -->
   <xacro:include filename="$(find clearpath_platform_description)/urdf/do100/wheels/wheel.urdf.xacro"/>
@@ -63,5 +62,5 @@
     </xacro:do100_wheel>
     <gazebo>
-      <plugin filename="libignition-gazebo-wheel-slip-system.so" name="ignition::gazebo::systems::WheelSlip">
+      <plugin filename="libgz-sim-wheel-slip-system.so" name="gz::sim::systems::WheelSlip">
         <wheel link_name="front_left_wheel_link">
           <slip_compliance_lateral>1.0</slip_compliance_lateral>
@@ -107,5 +106,5 @@
         <update_rate>50</update_rate>
         <visualize>true</visualize>
-        <ignition_frame_id>imu_0_link</ignition_frame_id>
+        <gz_frame_id>imu_0_link</gz_frame_id>
       </sensor>
     </gazebo>
@@ -169,41 +168,39 @@
     <xacro:include filename="$(find clearpath_platform_description)/urdf/generic/gazebo.urdf.xacro"/>
     <!-- ROS2 controls -->
-    <xacro:if value="$(arg use_platform_controllers)">
-      <ros2_control name="do100_hardware" type="system">
-        <hardware>
-          <xacro:if value="$(arg is_sim)">
-            <plugin>ign_ros2_control/IgnitionSystem</plugin>
-          </xacro:if>
-          <xacro:unless value="$(arg is_sim)">
-            <plugin>clearpath_hardware_interfaces/PumaHardware</plugin>
-          </xacro:unless>
-        </hardware>
-        <joint name="front_left_wheel_joint">
-          <command_interface name="velocity"/>
-          <state_interface name="position"/>
-          <state_interface name="velocity"/>
-        </joint>
-        <joint name="front_right_wheel_joint">
-          <command_interface name="velocity"/>
-          <state_interface name="position"/>
-          <state_interface name="velocity"/>
-        </joint>
-        <joint name="rear_left_wheel_joint">
-          <command_interface name="velocity"/>
-          <state_interface name="position"/>
-          <state_interface name="velocity"/>
-        </joint>
-        <joint name="rear_right_wheel_joint">
-          <command_interface name="velocity"/>
-          <state_interface name="position"/>
-          <state_interface name="velocity"/>
-        </joint>
-      </ros2_control>
-    </xacro:if>
+    <ros2_control name="do100_hardware" type="system">
+      <hardware>
+        <xacro:if value="$(arg is_sim)">
+          <plugin>gz_ros2_control/GazeboSimSystem</plugin>
+        </xacro:if>
+        <xacro:unless value="$(arg is_sim)">
+          <plugin>clearpath_hardware_interfaces/PumaHardware</plugin>
+        </xacro:unless>
+      </hardware>
+      <joint name="front_left_wheel_joint">
+        <command_interface name="velocity"/>
+        <state_interface name="position"/>
+        <state_interface name="velocity"/>
+      </joint>
+      <joint name="front_right_wheel_joint">
+        <command_interface name="velocity"/>
+        <state_interface name="position"/>
+        <state_interface name="velocity"/>
+      </joint>
+      <joint name="rear_left_wheel_joint">
+        <command_interface name="velocity"/>
+        <state_interface name="position"/>
+        <state_interface name="velocity"/>
+      </joint>
+      <joint name="rear_right_wheel_joint">
+        <command_interface name="velocity"/>
+        <state_interface name="position"/>
+        <state_interface name="velocity"/>
+      </joint>
+    </ros2_control>
   </xacro:macro>
   <!-- Joint State Publisher -->
   <plugin
-    filename="ignition-gazebo-joint-state-publisher-system"
-    name="ignition::gazebo::systems::JointStatePublisher"
+    filename="gz-sim-joint-state-publisher-system"
+    name="gz::sim::systems::JointStatePublisher"
   />
 </robot>
