Commit message: Imported upstream version '2.2.1' of 'upstream'

File: clearpath_platform_description/urdf/do150/do150.urdf.xacro (robot description, xacro)
@@ -4,5 +4,4 @@
   <xacro:arg name="is_sim" default="false" />
   <xacro:arg name="gazebo_controllers" default="$(find clearpath_control)/config/do150/control.yaml"/>
-  <xacro:arg name="use_platform_controllers" default="true"/>
   <!-- Included URDF/Xacro Files -->
   <xacro:include filename="$(find clearpath_platform_description)/urdf/do100/do100.urdf.xacro"/>

File: clearpath_platform_description/urdf/generic/gazebo.urdf.xacro (robot description, xacro)
@@ -3,9 +3,9 @@
   <xacro:if value="$(arg is_sim)">
     <gazebo>
-      <plugin filename="libign_ros2_control-system.so" name="ign_ros2_control::IgnitionROS2ControlPlugin">
+      <plugin filename="libgz_ros2_control-system.so" name="gz_ros2_control::GazeboSimROS2ControlPlugin">
         <parameters>$(arg gazebo_controllers)</parameters>
         <ros>
           <remapping>~/odom:=platform/odom</remapping>
-          <remapping>~/cmd_vel_unstamped:=platform/cmd_vel_unstamped</remapping>
+          <remapping>~/cmd_vel:=platform/cmd_vel</remapping>
           <remapping>/tf:=tf</remapping>
           <remapping>/tf_static:=tf_static</remapping>
@@ -20,5 +20,5 @@
     </gazebo>
     <gazebo>
-      <plugin filename="libignition-gazebo-pose-publisher-system.so" name="ignition::gazebo::systems::PosePublisher">
+      <plugin filename="libgz-sim-pose-publisher-system.so" name="gz::sim::systems::PosePublisher">
         <publish_link_pose>true</publish_link_pose>
         <publish_nested_model_pose>true</publish_nested_model_pose>
