Commit message: Rebase from 'upstream'

File: clearpath_manipulators_description/srdf/arm/franka.srdf.xacro (robot description, xacro)
@@ -1,24 +1,24 @@
 <?xml version="1.0" encoding="UTF-8"?>
 <robot xmlns:xacro="http://ros.org/wiki/xacro">
-  <xacro:macro name="franka_group_state" params="name group_state joint_positions arm_id:=fr3">
+  <xacro:macro name="franka_group_state" params="name group_state joint_positions robot_type:=fr3">
     <group_state name="${group_state}" group="${name}">
-      <joint name="${name}_${arm_id}_joint1" value="${joint_positions[0]}"/>
-      <joint name="${name}_${arm_id}_joint2" value="${joint_positions[1]}"/>
-      <joint name="${name}_${arm_id}_joint3" value="${joint_positions[2]}"/>
-      <joint name="${name}_${arm_id}_joint4" value="${joint_positions[3]}"/>
-      <joint name="${name}_${arm_id}_joint5" value="${joint_positions[4]}"/>
-      <joint name="${name}_${arm_id}_joint6" value="${joint_positions[5]}"/>
-      <joint name="${name}_${arm_id}_joint7" value="${joint_positions[6]}"/>
+      <joint name="${name}_${robot_type}_joint1" value="${joint_positions[0]}"/>
+      <joint name="${name}_${robot_type}_joint2" value="${joint_positions[1]}"/>
+      <joint name="${name}_${robot_type}_joint3" value="${joint_positions[2]}"/>
+      <joint name="${name}_${robot_type}_joint4" value="${joint_positions[3]}"/>
+      <joint name="${name}_${robot_type}_joint5" value="${joint_positions[4]}"/>
+      <joint name="${name}_${robot_type}_joint6" value="${joint_positions[5]}"/>
+      <joint name="${name}_${robot_type}_joint7" value="${joint_positions[6]}"/>
     </group_state>
   </xacro:macro>
-  <xacro:macro name="franka" params="name arm_id:=fr3">
+  <xacro:macro name="franka" params="name robot_type:=fr3">
     <group name="${name}">
-      <joint name="${name}_${arm_id}_joint1"/>
-      <joint name="${name}_${arm_id}_joint2"/>
-      <joint name="${name}_${arm_id}_joint3"/>
-      <joint name="${name}_${arm_id}_joint4"/>
-      <joint name="${name}_${arm_id}_joint5"/>
-      <joint name="${name}_${arm_id}_joint6"/>
-      <joint name="${name}_${arm_id}_joint7"/>
+      <joint name="${name}_${robot_type}_joint1"/>
+      <joint name="${name}_${robot_type}_joint2"/>
+      <joint name="${name}_${robot_type}_joint3"/>
+      <joint name="${name}_${robot_type}_joint4"/>
+      <joint name="${name}_${robot_type}_joint5"/>
+      <joint name="${name}_${robot_type}_joint6"/>
+      <joint name="${name}_${robot_type}_joint7"/>
     </group>
     <xacro:franka_group_state
@@ -26,5 +26,5 @@
       group_state="zero"
       joint_positions="${[0.0, 0.0, 0.0, 0.0, 0.0, 0.0, 0.0]}"
-      arm_id="${arm_id}"
+      robot_type="${robot_type}"
     />
     <xacro:franka_group_state
@@ -32,5 +32,5 @@
       group_state="home"
       joint_positions="${[0.0, -math.pi/4, 0.0, -math.pi * 7/8, 0.0, math.pi * 3/4, 0.0]}"
-      arm_id="${arm_id}"
+      robot_type="${robot_type}"
     />
   </xacro:macro>

File: clearpath_manipulators_description/srdf/gripper/franka_gripper.srdf.xacro (robot description, xacro)
@@ -1,14 +1,14 @@
 <?xml version="1.0" encoding="UTF-8"?>
 <robot xmlns:xacro="http://ros.org/wiki/xacro">
-  <xacro:macro name="franka_gripper_group_state" params="name group_state joint_positions arm_id:=fr3">
+  <xacro:macro name="franka_gripper_group_state" params="name group_state joint_positions robot_type:=fr3">
     <group_state name="${group_state}" group="${name}">
-      <joint name="${name}_${arm_id}_finger_joint1" value="${joint_positions[0]}"/>
-      <joint name="${name}_${arm_id}_finger_joint2" value="${joint_positions[0]}"/>
+      <joint name="${name}_${robot_type}_finger_joint1" value="${joint_positions[0]}"/>
+      <joint name="${name}_${robot_type}_finger_joint2" value="${joint_positions[0]}"/>
     </group_state>
   </xacro:macro>
-  <xacro:macro name="franka_gripper" params="name arm_id:=fr3">
+  <xacro:macro name="franka_gripper" params="name robot_type:=fr3">
     <group name="${name}">
-        <joint name="${name}_${arm_id}_finger_joint1"/>
-        <joint name="${name}_${arm_id}_finger_joint2"/>
+        <joint name="${name}_${robot_type}_finger_joint1"/>
+        <joint name="${name}_${robot_type}_finger_joint2"/>
     </group>
     <xacro:franka_gripper_group_state
@@ -16,5 +16,5 @@
       group_state="open"
       joint_positions="${[0.04]}"
-      arm_id="${arm_id}"
+      robot_type="${robot_type}"
     />
     <xacro:franka_gripper_group_state
@@ -22,5 +22,5 @@
       group_state="close"
       joint_positions="${[0.0]}"
-      arm_id="${arm_id}"
+      robot_type="${robot_type}"
     />
   </xacro:macro>
