Commit message: Imported upstream version '2.3.0' of 'upstream'

File: clearpath_sensors_description/urdf/swiftnav_duro.urdf.xacro (robot description, xacro)
@@ -2,24 +2,8 @@
 <robot xmlns:xacro="http://www.ros.org/wiki/xacro">
   <xacro:macro name="swiftnav_duro" params="name parent_link *origin">
-    <link name="${name}_link">
-      <visual>
-        <material name="clearpath_white"/>
-        <geometry>
-          <mesh filename="package://clearpath_sensors_description/meshes/swift_antenna.stl"/>
-        </geometry>
-      </visual>
-      <collision>
-        <material name="clearpath_white"/>
-        <origin xyz="0.0000 -0.0000 0.0324"/>
-        <geometry>
-          <sphere radius="0.1122" />
-        </geometry>
-      </collision>
-    </link>
-    <joint name="${name}_joint" type="fixed">
-      <child link="${name}_link"/>
-      <parent link="${parent_link}"/>
+    <xacro:include filename="$(find clearpath_sensors_description)/urdf/gnss_antenna.urdf.xacro" />
+    <xacro:gnss_antenna prefix="${name}" parent_link="${parent_link}" type="spherical">
       <xacro:insert_block name="origin"/>
-    </joint>
+    </xacro:gnss_antenna>
     <gazebo reference="${name}_link">
       <sensor name="${name}" type="navsat">
