Commit message: Rebase from 'upstream'

File: clearpath_sensors_description/urdf/fixposition.urdf.xacro (robot description, xacro)
@@ -74,4 +74,12 @@
             />
         </xacro:gnss_antenna>
+        <gazebo reference="${name}_gps_0_link">
+            <sensor name="${name}_gps_0" type="navsat">
+                <always_on>1</always_on>
+                <update_rate>1</update_rate>
+                <gz_frame_id>${name}_gps_0_link</gz_frame_id>
+                <topic>$(arg namespace)/sensors/${name}/gps_0/fix</topic>
+            </sensor>
+        </gazebo>
         <xacro:if value="${num_antennas > 1}">
             <xacro:gnss_antenna
@@ -84,4 +92,12 @@
                 />
             </xacro:gnss_antenna>
+            <gazebo reference="${name}_gps_1_link">
+                <sensor name="${name}_gps_1" type="navsat">
+                    <always_on>1</always_on>
+                    <update_rate>1</update_rate>
+                    <gz_frame_id>${name}_gps_1_link</gz_frame_id>
+                    <topic>$(arg namespace)/sensors/${name}/gps_1/fix</topic>
+                </sensor>
+            </gazebo>
         </xacro:if>
     </xacro:macro>

File: clearpath_sensors_description/urdf/ouster_os1.urdf.xacro (robot description, xacro)
@@ -19,4 +19,5 @@
     parent_link
     cap:=halo
+    base:=base
     *origin
     samples_h:=1024 min_ang_h:=${-pi} max_ang_h:=${pi}
@@ -28,7 +29,14 @@
     <xacro:property name="lidar_height" value="0.05835"/>
     <xacro:property name="lidar_diameter" value="0.087"/>
-    <xacro:property name="base_mass" value="0."/>
-    <xacro:property name="base_height" value="0.0225"/>
-    <xacro:property name="base_length" value="0.110"/>
+    <xacro:if value="${base == 'base'}">
+      <xacro:property name="base_mass" value="0.0"/>
+      <xacro:property name="base_height" value="0.0225"/>
+      <xacro:property name="base_length" value="0.110"/>
+    </xacro:if>
+    <xacro:unless value="${base == 'base'}">
+      <xacro:property name="base_mass" value="0.0"/>
+      <xacro:property name="base_height" value="0.0"/>
+      <xacro:property name="base_length" value="0.0"/>
+    </xacro:unless>
     <xacro:property name="fins_mass" value="0.079"/>
     <xacro:property name="fins_height" value="0.022"/>
@@ -38,31 +46,36 @@
     <xacro:property name="halo_diameter" value="0.08679"/>
     <!-- Base Link -->
-    <link name="${name}_base_link">
-      <inertial>
-        <mass value="${base_mass}"/>
-        <origin xyz="0 0 ${base_height/2}"/>
-        <xacro:ouster_box_inertia
-          mass="${base_mass}"
-          x="${base_length}"
-          y="${base_length}"
-          z="${base_height}"
-        />
-      </inertial>
-      <visual>
-        <material name="ouster_grey">
-          <color rgba="0.8 0.8 0.8 1.0"/>
-        </material>
-        <origin xyz="0 0 ${base_height}"/>
-        <geometry>
-          <mesh filename="package://clearpath_sensors_description/meshes/ouster/os1_base.dae"/>
-        </geometry>
-      </visual>
-      <collision>
-        <origin xyz="0 0 ${base_height/2}"/>
-        <geometry>
-          <box size="${base_length} ${base_length} ${base_height}"/>
-        </geometry>
-      </collision>
+    <xacro:if value="${base == 'base'}">
+      <link name="${name}_base_link">
+        <inertial>
+          <mass value="${base_mass}"/>
+          <origin xyz="0 0 ${base_height/2}"/>
+          <xacro:ouster_box_inertia
+            mass="${base_mass}"
+            x="${base_length}"
+            y="${base_length}"
+            z="${base_height}"
+          />
+        </inertial>
+        <visual>
+          <material name="ouster_grey">
+            <color rgba="0.8 0.8 0.8 1.0"/>
+          </material>
+          <origin xyz="0 0 ${base_height}"/>
+          <geometry>
+            <mesh filename="package://clearpath_sensors_description/meshes/ouster/os1_base.dae"/>
+          </geometry>
+        </visual>
+        <collision>
+          <origin xyz="0 0 ${base_height/2}"/>
+          <geometry>
+            <box size="${base_length} ${base_length} ${base_height}"/>
+          </geometry>
+        </collision>
     </link>
+  </xacro:if>
+  <xacro:unless value="${base == 'base'}">
+    <link name="${name}_base_link" />
+  </xacro:unless>
     <!-- Lidar Link -->
     <link name="${name}_link">

File: clearpath_sensors_description/urdf/phidgets_spatial.urdf.xacro (robot description, xacro)
@@ -25,5 +25,5 @@
         <update_rate>${update_rate}</update_rate>
         <visualize>true</visualize>
-        <ignition_frame_id>${name}_link</ignition_frame_id>
+        <gz_frame_id>${name}_link</gz_frame_id>
         <topic>$(arg namespace)/sensors/${name}/data</topic>
       </sensor>

File: clearpath_sensors_description/urdf/seyond_lidar.urdf.xacro (robot description, xacro)
@@ -2,7 +2,13 @@
 <robot xmlns:xacro="http://ros.org/wiki/xacro">
     <xacro:macro name="seyond_lidar" params="name parent_link *origin
-                                             ang_res_h:=0.002617993877991494 min_ang_h:=-1.0471975511965976 max_ang_h:=1.0471975511965976
-                                             ang_res_v:=0.006283185307179586 min_ang_v:=-0.6108652381980153 max_ang_v:=0.6108652381980153
-                                             update_rate:=20 min_range:=0.1 max_range:=150.0">
+                                             ang_res_h:=0.002617993877991494
+                                             min_ang_h:=-1.0471975511965976
+                                             max_ang_h:=1.0471975511965976
+                                             ang_res_v:=0.006283185307179586
+                                             min_ang_v:=-0.6108652381980153
+                                             max_ang_v:=0.6108652381980153
+                                             update_rate:=20
+                                             min_range:=0.1
+                                             max_range:=150.0">
         <link name="${name}_base_link">
             <inertial>
@@ -47,6 +53,6 @@
             <origin xyz="0 0 0.042" rpy="0 0 0" />
         </joint>
-        <xacro:property name="samples_h" value="${round((max_ang_h - min_ang_h) * 180 / (ang_res_h * pi))}"/>
-        <xacro:property name="samples_v" value="${round((max_ang_v - min_ang_v) * 180 / (ang_res_v * pi))}"/>
+        <xacro:property name="samples_h" value="${round((max_ang_h - min_ang_h) / ang_res_h)}"/>
+        <xacro:property name="samples_v" value="${round((max_ang_v - min_ang_v) / ang_res_v)}"/>
         <gazebo reference="${name}_laser">
             <sensor name="${name}" type="gpu_lidar">
