Commit message: Imported upstream version '1.3.4' of 'upstream'

File: clearpath_mounts_description/urdf/pacs/riser_leg.urdf.xacro (robot description, xacro)
@@ -47,5 +47,5 @@
       <child link="${name}_link" />
       <parent link="${parent_link}" />
-      <xacro:insert_block name="origin" />
+      <insert_block name="origin" />
     </joint>
     <joint name="${name}_mount_joint" type="fixed">

File: clearpath_mounts_description/urdf/post.urdf.xacro (robot description, xacro)
@@ -139,5 +139,5 @@
       <child link="${name}_link" />
       <parent link="${parent_link}" />
-      <xacro:insert_block name="origin" />
+      <insert_block name="origin" />
     </joint>
     <joint name="${name}_mount_joint" type="fixed">

File: clearpath_platform_description/urdf/common.urdf.xacro (robot description, xacro)
@@ -65,6 +65,5 @@
     -->
     <xacro:macro name="row_mounts" params="name parent_link row column columns x:=0 y:=0 z:=0 spacing:=0.08  iteration:=0">
-      <xacro:property name="chr" value="${dict(d97='a', d98='b', d99='c', d100='d', d101='e', d102='f', d103='g', d104='h', d105='i', d106='j', d107='k', d108='l', d109='m', d110='n', d111='o', d112='p', d113='q', d114='r', d115='s', d116='t', d117='u', d118='v', d119='w', d120='x',
-      d121='y', d122='z')}" />
+      <xacro:property name="chr" value="${dict(d97='a', d98='b', d99='c', d100='d', d101='e', d102='f', d103='g', d104='h')}" />
       <xacro:if value="${columns > iteration}">
         <xacro:property name="coordinate" value="${chr['d' + str(python.ord(column))] + python.str(row)}" />
@@ -114,3 +113,25 @@
       </xacro:if>
     </xacro:macro>
+    <xacro:macro name="clearpath_material" params="name:='' color_rgba:='' texture_file:=''">
+      <xacro:if value="${name != ''}">
+        <material name="${name}">
+          <xacro:if value="${color_rgba != ''}">
+            <color rgba="${color_rgba}"/>
+          </xacro:if>
+          <xacro:if value="${texture_file != ''}">
+            <texture filename="${texture_file}"/>
+          </xacro:if>
+        </material>
+      </xacro:if>
+      <xacro:unless value="${name != ''}">
+        <material>
+          <xacro:if value="${color_rgba != ''}">
+            <color rgba="${color_rgba}"/>
+          </xacro:if>
+          <xacro:if value="${texture_file != ''}">
+            <texture filename="${texture_file}"/>
+          </xacro:if>
+        </material>
+      </xacro:unless>
+    </xacro:macro>
 </robot>

File: clearpath_platform_description/urdf/r100/r100.urdf.xacro (robot description, xacro)
@@ -4,4 +4,5 @@
   <xacro:arg name="is_sim" default="false" />
   <xacro:arg name="gazebo_controllers" default="$(find clearpath_control)/config/r100/control.yaml"/>
+  <xacro:arg name="use_platform_controllers" default="true"/>
   <!-- Includes -->
   <xacro:include filename="$(find clearpath_platform_description)/urdf/r100/wheels/wheel.urdf.xacro"/>
@@ -18,5 +19,5 @@
     <xacro:property name="deck_height" value="0.280" />
     <xacro:property name="deck_thickness" value="0.005" />
-    <xacro:property name="riser_height" value="0.070" />
+    <xacro:property name="riser_height" value="0.055" />
     <xacro:property name="axle_offset" value="0.0500" />
     <xacro:property name="rocker_offset" value="0.319" />
@@ -110,5 +111,5 @@
           <mesh filename="package://clearpath_platform_description/meshes/r100/end-cover.stl" />
         </geometry>
-        <material name="clearpath_red" />
+        <material name="clearpath_black" />
       </visual>
     </link>
@@ -139,5 +140,5 @@
           <mesh filename="package://clearpath_platform_description/meshes/r100/lights.stl" />
         </geometry>
-        <material name="clearpath_black" />
+        <material name="clearpath_red" />
       </visual>
     </link>
@@ -207,5 +208,5 @@
     </xacro:r100_rocker>
     <gazebo>
-      <plugin filename="libgz-sim-wheel-slip-system.so" name="gz::sim::systems::WheelSlip">
+      <plugin filename="libignition-gazebo-wheel-slip-system.so" name="ignition::gazebo::systems::WheelSlip">
         <wheel link_name="front_left_wheel_link">
           <slip_compliance_lateral>1.0</slip_compliance_lateral>
@@ -252,5 +253,5 @@
         <update_rate>50</update_rate>
         <visualize>true</visualize>
-        <gz_frame_id>imu_0_link</gz_frame_id>
+        <ignition_frame_id>imu_0_link</ignition_frame_id>
       </sensor>
     </gazebo>
@@ -265,34 +266,36 @@
     <xacro:include filename="$(find clearpath_platform_description)/urdf/generic/gazebo.urdf.xacro"/>
     <!-- ROS2 controls -->
-    <ros2_control name="r100_hardware" type="system">
-      <hardware>
-        <xacro:if value="$(arg is_sim)">
-          <plugin>gz_ros2_control/GazeboSimSystem</plugin>
-        </xacro:if>
-        <xacro:unless value="$(arg is_sim)">
-          <plugin>clearpath_hardware_interfaces/PumaHardware</plugin>
-        </xacro:unless>
-      </hardware>
-      <joint name="front_left_wheel_joint">
-        <command_interface name="velocity"/>
-        <state_interface name="position"/>
-        <state_interface name="velocity"/>
-      </joint>
-      <joint name="front_right_wheel_joint">
-        <command_interface name="velocity"/>
-        <state_interface name="position"/>
-        <state_interface name="velocity"/>
-      </joint>
-      <joint name="rear_left_wheel_joint">
-        <command_interface name="velocity"/>
-        <state_interface name="position"/>
-        <state_interface name="velocity"/>
-      </joint>
-      <joint name="rear_right_wheel_joint">
-        <command_interface name="velocity"/>
-        <state_interface name="position"/>
-        <state_interface name="velocity"/>
-      </joint>
-    </ros2_control>
+    <xacro:if value="$(arg use_platform_controllers)">
+      <ros2_control name="r100_hardware" type="system">
+        <hardware>
+          <xacro:if value="$(arg is_sim)">
+            <plugin>ign_ros2_control/IgnitionSystem</plugin>
+          </xacro:if>
+          <xacro:unless value="$(arg is_sim)">
+            <plugin>clearpath_hardware_interfaces/PumaHardware</plugin>
+          </xacro:unless>
+        </hardware>
+        <joint name="front_left_wheel_joint">
+          <command_interface name="velocity"/>
+          <state_interface name="position"/>
+          <state_interface name="velocity"/>
+        </joint>
+        <joint name="front_right_wheel_joint">
+          <command_interface name="velocity"/>
+          <state_interface name="position"/>
+          <state_interface name="velocity"/>
+        </joint>
+        <joint name="rear_left_wheel_joint">
+          <command_interface name="velocity"/>
+          <state_interface name="position"/>
+          <state_interface name="velocity"/>
+        </joint>
+        <joint name="rear_right_wheel_joint">
+          <command_interface name="velocity"/>
+          <state_interface name="position"/>
+          <state_interface name="velocity"/>
+        </joint>
+      </ros2_control>
+    </xacro:if>
   </xacro:macro>
 </robot>

File: clearpath_sensors_description/urdf/ouster_os1.urdf.xacro (robot description, xacro)
@@ -19,5 +19,4 @@
     parent_link
     cap:=halo
-    base:=base
     *origin
     samples_h:=1024 min_ang_h:=${-pi} max_ang_h:=${pi}
@@ -29,14 +28,7 @@
     <xacro:property name="lidar_height" value="0.05835"/>
     <xacro:property name="lidar_diameter" value="0.087"/>
-    <xacro:if value="${base == 'base'}">
-      <xacro:property name="base_mass" value="0.0"/>
-      <xacro:property name="base_height" value="0.0225"/>
-      <xacro:property name="base_length" value="0.110"/>
-    </xacro:if>
-    <xacro:unless value="${base == 'base'}">
-      <xacro:property name="base_mass" value="0.0"/>
-      <xacro:property name="base_height" value="0.0"/>
-      <xacro:property name="base_length" value="0.0"/>
-    </xacro:unless>
+    <xacro:property name="base_mass" value="0."/>
+    <xacro:property name="base_height" value="0.0225"/>
+    <xacro:property name="base_length" value="0.110"/>
     <xacro:property name="fins_mass" value="0.079"/>
     <xacro:property name="fins_height" value="0.022"/>
@@ -46,36 +38,31 @@
     <xacro:property name="halo_diameter" value="0.08679"/>
     <!-- Base Link -->
-    <xacro:if value="${base == 'base'}">
-      <link name="${name}_base_link">
-        <inertial>
-          <mass value="${base_mass}"/>
-          <origin xyz="0 0 ${base_height/2}"/>
-          <xacro:ouster_box_inertia
-            mass="${base_mass}"
-            x="${base_length}"
-            y="${base_length}"
-            z="${base_height}"
-          />
-        </inertial>
-        <visual>
-          <material name="ouster_grey">
-            <color rgba="0.8 0.8 0.8 1.0"/>
-          </material>
-          <origin xyz="0 0 ${base_height}"/>
-          <geometry>
-            <mesh filename="package://clearpath_sensors_description/meshes/ouster/os1_base.dae"/>
-          </geometry>
-        </visual>
-        <collision>
-          <origin xyz="0 0 ${base_height/2}"/>
-          <geometry>
-            <box size="${base_length} ${base_length} ${base_height}"/>
-          </geometry>
-        </collision>
+    <link name="${name}_base_link">
+      <inertial>
+        <mass value="${base_mass}"/>
+        <origin xyz="0 0 ${base_height/2}"/>
+        <xacro:ouster_box_inertia
+          mass="${base_mass}"
+          x="${base_length}"
+          y="${base_length}"
+          z="${base_height}"
+        />
+      </inertial>
+      <visual>
+        <material name="ouster_grey">
+          <color rgba="0.8 0.8 0.8 1.0"/>
+        </material>
+        <origin xyz="0 0 ${base_height}"/>
+        <geometry>
+          <mesh filename="package://clearpath_sensors_description/meshes/ouster/os1_base.dae"/>
+        </geometry>
+      </visual>
+      <collision>
+        <origin xyz="0 0 ${base_height/2}"/>
+        <geometry>
+          <box size="${base_length} ${base_length} ${base_height}"/>
+        </geometry>
+      </collision>
     </link>
-  </xacro:if>
-  <xacro:unless value="${base == 'base'}">
-    <link name="${name}_base_link" />
-  </xacro:unless>
     <!-- Lidar Link -->
     <link name="${name}_link">

File: clearpath_sensors_description/urdf/phidgets_spatial.urdf.xacro (robot description, xacro)
@@ -25,5 +25,5 @@
         <update_rate>${update_rate}</update_rate>
         <visualize>true</visualize>
-        <gz_frame_id>${name}_link</gz_frame_id>
+        <ignition_frame_id>${name}_link</ignition_frame_id>
         <topic>$(arg namespace)/sensors/${name}/data</topic>
       </sensor>
