Commit message: Imported upstream version '2.6.3' of 'upstream'

File: clearpath_manipulators_description/urdf/arm/universal_robots.urdf.xacro (robot description, xacro)
@@ -2,5 +2,5 @@
 <robot xmlns:xacro="http://ros.org/wiki/xacro">
   <xacro:arg name="is_sim" default="false"/>
-  <xacro:arg name="use_fake_hardware" default="false"/>
+  <xacro:arg name="use_mock_hardware" default="false"/>
   <xacro:arg name="use_manipulation_controllers" default="false"/>
   <xacro:include filename="$(find ur_description)/urdf/ur_macro.xacro"/>
@@ -19,5 +19,4 @@
     safety_pos_margin:=''
     safety_k_position:=''
-    generate_ros2_control_tag:=''
     headless_mode:=''
     robot_ip:=''
@@ -42,9 +41,10 @@
     tool_device_name:=''
     tool_tcp_port:=''
-    use_fake_hardware:=''
-    fake_sensor_commands:=''
+    use_mock_hardware:=''
+    mock_sensor_commands:=''
     sim_gazebo:=''
     sim_ignition:=''
     ">
+    <xacro:property name="use_manipulation_controllers" value="$(arg use_manipulation_controllers)"/>
     <!-- Default Description Parameters -->
     <xacro:property name="_tf_prefix" value="${name}_" lazy_eval="false"/>
@@ -69,15 +69,14 @@
     <xacro:if value="${safety_k_position != ''}"> <xacro:property name="_safety_k_position" value="${safety_k_position}" lazy_eval="false"/> </xacro:if>
     <!-- Default Simulation Parameters -->
-    <xacro:property name="_use_fake_hardware" value="false" />
-    <xacro:property name="_fake_sensor_commands" value="false" />
+    <xacro:property name="_use_mock_hardware" value="false" />
+    <xacro:property name="_mock_sensor_commands" value="false" />
     <xacro:property name="_sim_gazebo" value="false" />
     <xacro:property name="_sim_ignition" value="$(arg is_sim)" />
     <!-- Default Simulation Parameters Overwrites -->
-    <xacro:if value="${use_fake_hardware != ''}"> <xacro:property name="_use_fake_hardware" value="${use_fake_hardware}" lazy_eval="false"/> </xacro:if>
-    <xacro:if value="${fake_sensor_commands != ''}"> <xacro:property name="_fake_sensor_commands" value="${fake_sensor_commands}" lazy_eval="false"/> </xacro:if>
+    <xacro:if value="${use_mock_hardware != ''}"> <xacro:property name="_use_mock_hardware" value="${use_mock_hardware}" lazy_eval="false"/> </xacro:if>
+    <xacro:if value="${mock_sensor_commands != ''}"> <xacro:property name="_mock_sensor_commands" value="${mock_sensor_commands}" lazy_eval="false"/> </xacro:if>
     <xacro:if value="${sim_gazebo != ''}"> <xacro:property name="_sim_gazebo" value="${sim_gazebo}" lazy_eval="false"/> </xacro:if>
     <xacro:if value="${sim_ignition != ''}"> <xacro:property name="_sim_ignition" value="${sim_ignition}" lazy_eval="false"/> </xacro:if>
     <!-- Default ros2_control Parameters -->
-    <xacro:property name="_generate_ros2_control_tag" value="$(arg use_manipulation_controllers)" lazy_eval="false"/>
     <xacro:property name="_headless_mode" value="false" lazy_eval="false"/>
     <xacro:property name="_robot_ip" value="192.168.131.40" lazy_eval="false"/>
@@ -91,5 +90,4 @@
     <xacro:property name="_keep_alive_count" value="2.0" lazy_eval="false"/>
     <!-- Default ros2_control Parameters Overwrites -->
-    <xacro:if value="${generate_ros2_control_tag != ''}"> <xacro:property name="_generate_ros2_control_tag" value="${generate_ros2_control_tag}" lazy_eval="false"/> </xacro:if>
     <xacro:if value="${headless_mode != ''}"> <xacro:property name="_headless_mode" value="${headless_mode}" lazy_eval="false"/> </xacro:if>
     <xacro:if value="${robot_ip != ''}"> <xacro:property name="_robot_ip" value="${robot_ip}" lazy_eval="false"/> </xacro:if>
@@ -103,10 +101,10 @@
     <xacro:if value="${keep_alive_count != ''}"> <xacro:property name="_keep_alive_count" value="${keep_alive_count}" lazy_eval="false"/> </xacro:if>
     <!-- Driver Dependent Parameters -->
-    <xacro:if value="${_generate_ros2_control_tag and not _use_fake_hardware and not _sim_ignition}">
+    <xacro:if value="${use_manipulation_controllers and not _use_mock_hardware and not _sim_ignition}">
       <xacro:property name="_script_filename" value="$(find ur_client_library)/resources/external_control.urscript" lazy_eval="false"/>
       <xacro:property name="_output_recipe_filename" value="$(find ur_robot_driver)/resources/rtde_output_recipe.txt" lazy_eval="false"/>
       <xacro:property name="_input_recipe_filename" value="$(find ur_robot_driver)/resources/rtde_input_recipe.txt" lazy_eval="false"/>
     </xacro:if>
-    <xacro:unless value="${_generate_ros2_control_tag and not _use_fake_hardware and not _sim_ignition}">
+    <xacro:unless value="${use_manipulation_controllers and not _use_mock_hardware and not _sim_ignition}">
       <xacro:property name="_script_filename" value="" lazy_eval="false"/>
       <xacro:property name="_output_recipe_filename" value="" lazy_eval="false"/>
@@ -137,10 +135,9 @@
     <xacro:if value="${tool_device_name != ''}"> <xacro:property name="_tool_device_name" value="${tool_device_name}" lazy_eval="false"/> </xacro:if>
     <xacro:if value="${tool_tcp_port != ''}"> <xacro:property name="_tool_tcp_port" value="${tool_tcp_port}" lazy_eval="false"/> </xacro:if>
-    <!-- Universal_Robots_ROS2_Description -->
+    <!-- Universal Robots ROS2 Description -->
     <xacro:ur_robot
       name="${name}"
+      tf_prefix="${_tf_prefix}"
       parent="${parent_link}"
-      tf_prefix="${_tf_prefix}"
-      initial_positions="${_initial_positions}"
       joint_limits_parameters_file="${_joint_limits_parameters_file}"
       kinematics_parameters_file="${_kinematics_parameters_file}"
@@ -150,33 +147,39 @@
       safety_pos_margin="${_safety_pos_margin}"
       safety_k_position="${_safety_k_position}"
-      generate_ros2_control_tag="${_generate_ros2_control_tag}"
-      headless_mode="${_headless_mode}"
-      robot_ip="${_robot_ip}"
-      script_filename="${_script_filename}"
-      output_recipe_filename="${_output_recipe_filename}"
-      input_recipe_filename="${_input_recipe_filename}"
-      reverse_ip="${_reverse_ip}"
-      script_command_port="${_script_command_port}"
-      reverse_port="${_reverse_port}"
-      script_sender_port="${_script_sender_port}"
-      trajectory_port="${_trajectory_port}"
-      transmission_hw_interface="${_transmission_hw_interface}"
-      non_blocking_read="{_non_blocking_read}"
-      use_tool_communication="${_use_tool_communication}"
-      tool_voltage="${_tool_voltage}"
-      tool_parity="${_tool_parity}"
-      tool_baud_rate="${_tool_baud_rate}"
-      tool_stop_bits="${_tool_stop_bits}"
-      tool_rx_idle_chars="${_tool_rx_idle_chars}"
-      tool_tx_idle_chars="${_tool_tx_idle_chars}"
-      tool_device_name="${_tool_device_name}"
-      tool_tcp_port="${_tool_tcp_port}"
-      use_fake_hardware="${_use_fake_hardware}"
-      fake_sensor_commands="${_fake_sensor_commands}"
-      sim_gazebo="${_sim_gazebo}"
-      sim_ignition="${_sim_ignition}"
       >
       <xacro:insert_block name="origin"/>
     </xacro:ur_robot>
+    <!-- Universal_Robots_ROS2_Driver HardwareInterface -->
+    <xacro:if value="${use_manipulation_controllers}">
+      <xacro:include filename="$(find ur_robot_driver)/urdf/ur.ros2_control.xacro" />
+      <xacro:ur_ros2_control
+        name="${name}"
+        tf_prefix="${_tf_prefix}"
+        kinematics_parameters_file="${_kinematics_parameters_file}"
+        transmission_hw_interface="${_transmission_hw_interface}"
+        use_mock_hardware="${_use_mock_hardware}"
+        mock_sensor_commands="${_mock_sensor_commands}"
+        headless_mode="${_headless_mode}"
+        initial_positions="${_initial_positions}"
+        use_tool_communication="${_use_tool_communication}"
+        tool_voltage="${_tool_voltage}"
+        tool_parity="${_tool_parity}"
+        tool_baud_rate="${_tool_baud_rate}"
+        tool_stop_bits="${_tool_stop_bits}"
+        tool_rx_idle_chars="${_tool_rx_idle_chars}"
+        tool_tx_idle_chars="${_tool_tx_idle_chars}"
+        tool_device_name="${_tool_device_name}"
+        tool_tcp_port="${_tool_tcp_port}"
+        robot_ip="${_robot_ip}"
+        script_filename="${_script_filename}"
+        output_recipe_filename="${_output_recipe_filename}"
+        input_recipe_filename="${_input_recipe_filename}"
+        reverse_ip="${_reverse_ip}"
+        script_command_port="${_script_command_port}"
+        reverse_port="${_reverse_port}"
+        script_sender_port="${_script_sender_port}"
+        trajectory_port="${_trajectory_port}"
+      />
+    </xacro:if>
   </xacro:macro>
 </robot>

File: clearpath_manipulators_description/urdf/lift/ewellix.urdf.xacro (robot description, xacro)
@@ -16,5 +16,5 @@
     generate_ros2_control_tag:=''
     use_fake_hardware:=''
-    sim_ignition:=''
+    sim_gazebo:=''
     port=''
     baud=''
@@ -32,5 +32,5 @@
     <!-- Default Simulation Parameters -->
     <xacro:property name="_use_fake_hardware" value="false" />
-    <xacro:property name="_sim_ignition" value="$(arg is_sim)" />
+    <xacro:property name="_sim_gazebo" value="$(arg is_sim)" />
     <!-- Default Hardware Parameters -->
     <xacro:property name="_port" value="/dev/ttyUSB0"/>
@@ -47,5 +47,5 @@
     <xacro:if value="${generate_ros2_control_tag != ''}"> <xacro:property name="_generate_ros2_control_tag" value="${generate_ros2_control_tag}" lazy_eval="false"/> </xacro:if>
     <xacro:if value="${use_fake_hardware != ''}"> <xacro:property name="_use_fake_hardware" value="${use_fake_hardware}" lazy_eval="false"/> </xacro:if>
-    <xacro:if value="${sim_ignition != ''}"> <xacro:property name="_sim_ignition" value="${sim_ignition}" lazy_eval="false"/> </xacro:if>
+    <xacro:if value="${sim_gazebo != ''}"> <xacro:property name="_sim_gazebo" value="${sim_gazebo}" lazy_eval="false"/> </xacro:if>
     <xacro:if value="${port != ''}"> <xacro:property name="_port" value="${port}" lazy_eval="false"/> </xacro:if>
     <xacro:if value="${baud != ''}"> <xacro:property name="_baud" value="${baud}" lazy_eval="false"/> </xacro:if>
@@ -63,5 +63,5 @@
       generate_ros2_control_tag="${_generate_ros2_control_tag}"
       use_fake_hardware="${_use_fake_hardware}"
-      sim_ignition="${_sim_ignition}"
+      sim_gazebo="${_sim_gazebo}"
       port="${_port}"
       baud="${_baud}"

File: clearpath_platform_description/urdf/common.urdf.xacro (robot description, xacro)
@@ -65,5 +65,6 @@
     -->
     <xacro:macro name="row_mounts" params="name parent_link row column columns x:=0 y:=0 z:=0 spacing:=0.08  iteration:=0">
-      <xacro:property name="chr" value="${dict(d97='a', d98='b', d99='c', d100='d', d101='e', d102='f', d103='g', d104='h')}" />
+      <xacro:property name="chr" value="${dict(d97='a', d98='b', d99='c', d100='d', d101='e', d102='f', d103='g', d104='h', d105='i', d106='j', d107='k', d108='l', d109='m', d110='n', d111='o', d112='p', d113='q', d114='r', d115='s', d116='t', d117='u', d118='v', d119='w', d120='x',
+      d121='y', d122='z')}" />
       <xacro:if value="${columns > iteration}">
         <xacro:property name="coordinate" value="${chr['d' + str(python.ord(column))] + python.str(row)}" />
@@ -113,25 +114,3 @@
       </xacro:if>
     </xacro:macro>
-    <xacro:macro name="clearpath_material" params="name:='' color_rgba:='' texture_file:=''">
-      <xacro:if value="${name != ''}">
-        <material name="${name}">
-          <xacro:if value="${color_rgba != ''}">
-            <color rgba="${color_rgba}"/>
-          </xacro:if>
-          <xacro:if value="${texture_file != ''}">
-            <texture filename="${texture_file}"/>
-          </xacro:if>
-        </material>
-      </xacro:if>
-      <xacro:unless value="${name != ''}">
-        <material>
-          <xacro:if value="${color_rgba != ''}">
-            <color rgba="${color_rgba}"/>
-          </xacro:if>
-          <xacro:if value="${texture_file != ''}">
-            <texture filename="${texture_file}"/>
-          </xacro:if>
-        </material>
-      </xacro:unless>
-    </xacro:macro>
 </robot>

File: clearpath_platform_description/urdf/do100/do100.urdf.xacro (robot description, xacro)
@@ -63,5 +63,5 @@
     </xacro:do100_wheel>
     <gazebo>
-      <plugin filename="libignition-gazebo-wheel-slip-system.so" name="ignition::gazebo::systems::WheelSlip">
+      <plugin filename="libgz-sim-wheel-slip-system.so" name="gz::sim::systems::WheelSlip">
         <wheel link_name="front_left_wheel_link">
           <slip_compliance_lateral>1.0</slip_compliance_lateral>
@@ -107,5 +107,5 @@
         <update_rate>50</update_rate>
         <visualize>true</visualize>
-        <ignition_frame_id>imu_0_link</ignition_frame_id>
+        <gz_frame_id>imu_0_link</gz_frame_id>
       </sensor>
     </gazebo>
@@ -204,6 +204,6 @@
   <!-- Joint State Publisher -->
   <plugin
-    filename="ignition-gazebo-joint-state-publisher-system"
-    name="ignition::gazebo::systems::JointStatePublisher"
+    filename="gz-sim-joint-state-publisher-system"
+    name="gz::sim::systems::JointStatePublisher"
   />
 </robot>

File: clearpath_platform_description/urdf/r100/r100.urdf.xacro (robot description, xacro)
@@ -19,5 +19,5 @@
     <xacro:property name="deck_height" value="0.280" />
     <xacro:property name="deck_thickness" value="0.005" />
-    <xacro:property name="riser_height" value="0.055" />
+    <xacro:property name="riser_height" value="0.070" />
     <xacro:property name="axle_offset" value="0.0500" />
     <xacro:property name="rocker_offset" value="0.319" />
@@ -111,5 +111,5 @@
           <mesh filename="package://clearpath_platform_description/meshes/r100/end-cover.stl" />
         </geometry>
-        <material name="clearpath_black" />
+        <material name="clearpath_red" />
       </visual>
     </link>
@@ -140,5 +140,5 @@
           <mesh filename="package://clearpath_platform_description/meshes/r100/lights.stl" />
         </geometry>
-        <material name="clearpath_red" />
+        <material name="clearpath_black" />
       </visual>
     </link>
@@ -208,5 +208,5 @@
     </xacro:r100_rocker>
     <gazebo>
-      <plugin filename="libignition-gazebo-wheel-slip-system.so" name="ignition::gazebo::systems::WheelSlip">
+      <plugin filename="libgz-sim-wheel-slip-system.so" name="gz::sim::systems::WheelSlip">
         <wheel link_name="front_left_wheel_link">
           <slip_compliance_lateral>1.0</slip_compliance_lateral>
@@ -253,5 +253,5 @@
         <update_rate>50</update_rate>
         <visualize>true</visualize>
-        <ignition_frame_id>imu_0_link</ignition_frame_id>
+        <gz_frame_id>imu_0_link</gz_frame_id>
       </sensor>
     </gazebo>

File: clearpath_sensors_description/urdf/swiftnav_duro.urdf.xacro (robot description, xacro)
@@ -2,29 +2,13 @@
 <robot xmlns:xacro="http://www.ros.org/wiki/xacro">
   <xacro:macro name="swiftnav_duro" params="name parent_link *origin">
-    <link name="${name}_link">
-      <visual>
-        <material name="clearpath_white"/>
-        <geometry>
-          <mesh filename="package://clearpath_sensors_description/meshes/swift_antenna.stl"/>
-        </geometry>
-      </visual>
-      <collision>
-        <material name="clearpath_white"/>
-        <origin xyz="0.0000 -0.0000 0.0324"/>
-        <geometry>
-          <sphere radius="0.1122" />
-        </geometry>
-      </collision>
-    </link>
-    <joint name="${name}_joint" type="fixed">
-      <child link="${name}_link"/>
-      <parent link="${parent_link}"/>
+    <xacro:include filename="$(find clearpath_sensors_description)/urdf/gnss_antenna.urdf.xacro" />
+    <xacro:gnss_antenna prefix="${name}" parent_link="${parent_link}" type="spherical">
       <xacro:insert_block name="origin"/>
-    </joint>
+    </xacro:gnss_antenna>
     <gazebo reference="${name}_link">
       <sensor name="${name}" type="navsat">
         <always_on>1</always_on>
         <update_rate>1</update_rate>
-        <ignition_frame_id>${name}_link</ignition_frame_id>
+        <gz_frame_id>${name}_link</gz_frame_id>
         <topic>$(arg namespace)/sensors/${name}/navsat</topic>
       </sensor>
