Commit message: Imported upstream version '1.3.8' of 'upstream'

File: clearpath_platform_description/urdf/do100/do100.urdf.xacro (robot description, xacro)
@@ -3,12 +3,18 @@
   <xacro:arg name="namespace" default="" />
   <xacro:arg name="is_sim" default="false" />
-  <xacro:arg name="gazebo_controllers" default="$(find clearpath_control)/config/do100/control/omni_4wd.yaml"/>
+  <xacro:arg name="gazebo_controllers" default="$(find clearpath_control)/config/do100/control.yaml"/>
+  <xacro:arg name="use_platform_controllers" default="true"/>
+  <!-- Included URDF/Xacro Files -->
+  <xacro:include filename="$(find clearpath_platform_description)/urdf/do100/wheels/wheel.urdf.xacro"/>
   <xacro:property name="PI" value="${math.pi}" />
   <!-- D0100 Platform Macro -->
-  <xacro:macro name="do100" params="control:='omni_4wd' front_wheels:='mecanum' rear_wheels:='mecanum'">
+  <xacro:macro name="do100" params="wheel:='defaut'">
     <!-- Variables -->
     <xacro:property name="wheelbase" value="0.570" />
     <xacro:property name="track" value="0.3708" />
     <xacro:property name="wheel_vertical_offset" value="0.035145" />
+    <xacro:property name="wheel_radius" value="0.050" />
+    <xacro:property name="wheel_mass" value="0.4" />
+    <xacro:property name="wheel_width" value="0.050" />
     <xacro:property name="dummy_inertia" value="1e-09"/>
     <!-- Chassis -->
@@ -43,26 +49,45 @@
         </inertial>
     </link>
-    <!-- Add wheels -->
-    <xacro:include filename="$(find clearpath_platform_description)/urdf/do100/drivetrain/wheels.urdf.xacro"/>
-    <xacro:do100_drivetrain_wheels front_wheels="${front_wheels}" rear_wheels="${rear_wheels}"/>
-    <!-- Add drivetrain -->
-    <xacro:include filename="$(find clearpath_platform_description)/urdf/generic/drivetrain/drivetrain.urdf.xacro"/>
-    <!-- Hardware  -->
-    <xacro:if value="$(arg is_sim)">
-      <xacro:property name="hardware_plugin" value="gz_ros2_control/GazeboSimSystem"/>
-    </xacro:if>
-    <xacro:unless value="$(arg is_sim)">
-      <xacro:property name="hardware_plugin" value="clearpath_hardware_interfaces/PumaHardware"/>
-    </xacro:unless>
-    <xacro:unless value="${control == 'omni_4wd' or control == 'diff_4wd'}">
-      <xacro:error message="Invalid drivetrain control ${control}"/>
-    </xacro:unless>
-    <xacro:generic_drivetrain
-      name="do100"
-      control="${control}"
-      front_wheels="${front_wheels}"
-      rear_wheels="${rear_wheels}"
-      hardware_plugin="${hardware_plugin}"
-    />
+    <!-- Wheels -->
+    <xacro:do100_wheel prefix="front_left" side="-1">
+      <origin xyz="${wheelbase/2} ${track/2+wheel_width/2} ${wheel_vertical_offset}" rpy="0 0 0" />
+    </xacro:do100_wheel>
+    <xacro:do100_wheel prefix="front_right" side="1">
+      <origin xyz="${wheelbase/2} ${-track/2-wheel_width/2} ${wheel_vertical_offset}" rpy="0 0 0" />
+    </xacro:do100_wheel>
+    <xacro:do100_wheel prefix="rear_left" side="1">
+      <origin xyz="${-wheelbase/2} ${track/2+wheel_width/2} ${wheel_vertical_offset}" rpy="0 0 0" />
+    </xacro:do100_wheel>
+    <xacro:do100_wheel prefix="rear_right" side="-1">
+      <origin xyz="${-wheelbase/2} ${-track/2-wheel_width/2} ${wheel_vertical_offset}" rpy="0 0 0" />
+    </xacro:do100_wheel>
+    <gazebo>
+      <plugin filename="libignition-gazebo-wheel-slip-system.so" name="ignition::gazebo::systems::WheelSlip">
+        <wheel link_name="front_left_wheel_link">
+          <slip_compliance_lateral>1.0</slip_compliance_lateral>
+          <slip_compliance_longitudinal>1.0</slip_compliance_longitudinal>
+          <wheel_normal_force>20</wheel_normal_force>
+          <wheel_radius>${wheel_radius}</wheel_radius>
+        </wheel>
+        <wheel link_name="front_right_wheel_link">
+          <slip_compliance_lateral>1.0</slip_compliance_lateral>
+          <slip_compliance_longitudinal>1.0</slip_compliance_longitudinal>
+          <wheel_normal_force>20</wheel_normal_force>
+          <wheel_radius>${wheel_radius}</wheel_radius>
+        </wheel>
+        <wheel link_name="rear_left_wheel_link">
+          <slip_compliance_lateral>1.0</slip_compliance_lateral>
+          <slip_compliance_longitudinal>1.0</slip_compliance_longitudinal>
+          <wheel_normal_force>20</wheel_normal_force>
+          <wheel_radius>${wheel_radius}</wheel_radius>
+        </wheel>
+        <wheel link_name="rear_right_wheel_link">
+          <slip_compliance_lateral>1.0</slip_compliance_lateral>
+          <slip_compliance_longitudinal>1.0</slip_compliance_longitudinal>
+          <wheel_normal_force>20</wheel_normal_force>
+          <wheel_radius>${wheel_radius}</wheel_radius>
+        </wheel>
+      </plugin>
+    </gazebo>
     <!-- Internal IMU -->
     <link name="imu_0_link">
@@ -82,5 +107,5 @@
         <update_rate>50</update_rate>
         <visualize>true</visualize>
-        <gz_frame_id>imu_0_link</gz_frame_id>
+        <ignition_frame_id>imu_0_link</ignition_frame_id>
       </sensor>
     </gazebo>
@@ -141,9 +166,44 @@
       <child link="rear_bumper_mount" />
     </joint>
+    <!-- Gazebo Controller -->
+    <xacro:include filename="$(find clearpath_platform_description)/urdf/generic/gazebo.urdf.xacro"/>
+    <!-- ROS2 controls -->
+    <xacro:if value="$(arg use_platform_controllers)">
+      <ros2_control name="do100_hardware" type="system">
+        <hardware>
+          <xacro:if value="$(arg is_sim)">
+            <plugin>ign_ros2_control/IgnitionSystem</plugin>
+          </xacro:if>
+          <xacro:unless value="$(arg is_sim)">
+            <plugin>clearpath_hardware_interfaces/PumaHardware</plugin>
+          </xacro:unless>
+        </hardware>
+        <joint name="front_left_wheel_joint">
+          <command_interface name="velocity"/>
+          <state_interface name="position"/>
+          <state_interface name="velocity"/>
+        </joint>
+        <joint name="front_right_wheel_joint">
+          <command_interface name="velocity"/>
+          <state_interface name="position"/>
+          <state_interface name="velocity"/>
+        </joint>
+        <joint name="rear_left_wheel_joint">
+          <command_interface name="velocity"/>
+          <state_interface name="position"/>
+          <state_interface name="velocity"/>
+        </joint>
+        <joint name="rear_right_wheel_joint">
+          <command_interface name="velocity"/>
+          <state_interface name="position"/>
+          <state_interface name="velocity"/>
+        </joint>
+      </ros2_control>
+    </xacro:if>
   </xacro:macro>
   <!-- Joint State Publisher -->
   <plugin
-    filename="gz-sim-joint-state-publisher-system"
-    name="gz::sim::systems::JointStatePublisher"
+    filename="ignition-gazebo-joint-state-publisher-system"
+    name="ignition::gazebo::systems::JointStatePublisher"
   />
 </robot>

File: clearpath_platform_description/urdf/do150/do150.urdf.xacro (robot description, xacro)
@@ -3,147 +3,18 @@
   <xacro:arg name="namespace" default="" />
   <xacro:arg name="is_sim" default="false" />
-  <xacro:arg name="gazebo_controllers" default="$(find clearpath_control)/config/do150/control/omni_4wd.yaml"/>
-  <xacro:property name="PI" value="${math.pi}" />
-  <!-- D0150 Platform Macro -->
-  <xacro:macro name="do150" params="control:='omni_4wd' front_wheels:='mecanum' rear_wheels:='mecanum'">
-    <!-- Variables -->
-    <xacro:property name="wheelbase" value="0.570" />
-    <xacro:property name="track" value="0.3708" />
-    <xacro:property name="wheel_vertical_offset" value="0.035145" />
-    <xacro:property name="dummy_inertia" value="1e-09"/>
-    <!-- Chassis -->
-    <link name="base_link"></link>
-    <joint name="base_link_joint" type="fixed">
-      <origin xyz="0 0 0" rpy="0 0 0" />
-      <parent link="base_link"/>
-      <child link="chassis_link" />
-    </joint>
-    <link name="chassis_link">
-      <visual>
-        <origin xyz="0 0 0" rpy="0 0 0"/>
-        <geometry>
-          <mesh filename="package://clearpath_platform_description/meshes/do100/omni_chassis.dae"/>
-        </geometry>
-      </visual>
-      <collision>
-        <origin xyz="0 0 0"/>
-        <geometry>
-          <mesh filename="package://clearpath_platform_description/meshes/do100/omni_chassis_collision.stl"/>
-        </geometry>
-      </collision>
-      <inertial>
-        <!-- Center of mass -->
-        <origin xyz="0 0 0" rpy="0 0 0"/>
-        <mass value="14"/>
-        <!-- Moments of inertia: ( chassis without wheels ) -->
-        <inertia
-          ixx="0.35498" ixy="0" ixz="0"
-          iyy="0.7266" iyz="0"
-          izz="1.0553"/>
-        </inertial>
-    </link>
-    <!-- Add wheels (Same as DO100) -->
-    <xacro:include filename="$(find clearpath_platform_description)/urdf/do100/drivetrain/wheels.urdf.xacro"/>
-    <xacro:do100_drivetrain_wheels front_wheels="${front_wheels}" rear_wheels="${rear_wheels}"/>
-    <!-- Add drivetrain -->
-    <xacro:include filename="$(find clearpath_platform_description)/urdf/generic/drivetrain/drivetrain.urdf.xacro"/>
-    <!-- Hardware  -->
-    <xacro:if value="$(arg is_sim)">
-      <xacro:property name="hardware_plugin" value="gz_ros2_control/GazeboSimSystem"/>
-    </xacro:if>
-    <xacro:unless value="$(arg is_sim)">
-      <xacro:property name="hardware_plugin" value="clearpath_hardware_interfaces/PumaHardware"/>
-    </xacro:unless>
-    <xacro:unless value="${control == 'omni_4wd' or control == 'diff_4wd'}">
-      <xacro:error message="Invalid drivetrain control ${control}"/>
-    </xacro:unless>
-    <xacro:generic_drivetrain
-      name="do150"
-      control="${control}"
-      front_wheels="${front_wheels}"
-      rear_wheels="${rear_wheels}"
-      hardware_plugin="${hardware_plugin}"
-    />
-    <!-- Internal IMU -->
-    <link name="imu_0_link">
-      <inertial>
-        <mass value="0.001"/>
-        <origin xyz="0 0 0" rpy="0 0 0"/>
-        <inertia ixx="${dummy_inertia}" ixy="0.0" ixz="0.0" iyy="${dummy_inertia}" iyz="0.0" izz="${dummy_inertia}"/>
-      </inertial>
-    </link>
-    <joint name="imu_joint" type="fixed">
-      <parent link="chassis_link" />
-      <child link="imu_0_link" />
-    </joint>
-    <gazebo reference="imu_0_link">
-      <sensor type="imu" name="imu_0">
-        <always_on>true</always_on>
-        <update_rate>50</update_rate>
-        <visualize>true</visualize>
-        <gz_frame_id>imu_0_link</gz_frame_id>
-      </sensor>
-    </gazebo>
-    <!-- Mounting Hard Points -->
-    <link name="default_mount"/>
-    <link name="front_2_mount"/>
-    <link name="front_1_mount"/>
-    <link name="front_0_mount"/>
-    <link name="rear_2_mount"/>
-    <link name="rear_1_mount"/>
-    <link name="rear_0_mount"/>
-    <joint name="default_mount_joint" type="fixed">
-      <origin xyz="0 0 0.069023" rpy="0 0 0" />
-      <parent link="chassis_link"/>
-      <child link="default_mount" />
-    </joint>
-    <joint name="front_0_mount_joint" type="fixed">
-      <origin xyz="0.080 0 0" rpy="0 0 0" />
-      <parent link="default_mount"/>
-      <child link="front_0_mount" />
-    </joint>
-    <joint name="front_1_mount_joint" type="fixed">
-      <origin xyz="0.080 0 0" rpy="0 0 0" />
-      <parent link="front_0_mount"/>
-      <child link="front_1_mount" />
-    </joint>
-    <joint name="front_2_mount_joint" type="fixed">
-      <origin xyz="0.080 0 0" rpy="0 0 0" />
-      <parent link="front_1_mount"/>
-      <child link="front_2_mount" />
-    </joint>
-    <joint name="rear_0_mount_joint" type="fixed">
-      <origin xyz="-0.080 0 0" rpy="0 0 0" />
-      <parent link="default_mount"/>
-      <child link="rear_0_mount" />
-    </joint>
-    <joint name="rear_1_mount_joint" type="fixed">
-      <origin xyz="-0.080 0 0" rpy="0 0 0" />
-      <parent link="rear_0_mount"/>
-      <child link="rear_1_mount" />
-    </joint>
-    <joint name="rear_2_mount_joint" type="fixed">
-      <origin xyz="-0.080 0 0" rpy="0 0 0" />
-      <parent link="rear_1_mount"/>
-      <child link="rear_2_mount" />
-    </joint>
-    <!-- Bumper Mounts -->
-    <link name="front_bumper_mount"/>
-    <link name="rear_bumper_mount"/>
-    <joint name="front_bumper_mount_joint" type="fixed">
-      <origin xyz="0.34159 0 0.0345115" rpy="0 0 0" />
-      <parent link="chassis_link"/>
-      <child link="front_bumper_mount" />
-    </joint>
-    <joint name="rear_bumper_mount_joint" type="fixed">
-      <origin xyz="-0.34159 0 0.0345115" rpy="0 0 0" />
-      <parent link="chassis_link"/>
-      <child link="rear_bumper_mount" />
-    </joint>
+  <xacro:arg name="gazebo_controllers" default="$(find clearpath_control)/config/do150/control.yaml"/>
+  <xacro:arg name="use_platform_controllers" default="true"/>
+  <!-- Included URDF/Xacro Files -->
+  <xacro:include filename="$(find clearpath_platform_description)/urdf/do100/do100.urdf.xacro"/>
+  <!-- D0100 Platform Macro -->
+  <xacro:macro name="do150" params="wheel:='defaut'">
+    <xacro:do100 wheel="${wheel}"/>
   </xacro:macro>
   <!-- Joint State Publisher -->
-  <plugin
-    filename="gz-sim-joint-state-publisher-system"
-    name="gz::sim::systems::JointStatePublisher"
-  />
+  <gazebo>
+    <plugin
+      filename="ignition-gazebo-joint-state-publisher-system"
+      name="ignition::gazebo::systems::JointStatePublisher"
+    />
+  </gazebo>
 </robot>

File: clearpath_platform_description/urdf/r100/r100.urdf.xacro (robot description, xacro)
@@ -3,8 +3,15 @@
   <xacro:arg name="namespace" default="" />
   <xacro:arg name="is_sim" default="false" />
-  <xacro:arg name="gazebo_controllers" default="$(find clearpath_control)/config/r100/control/omni_4wd.yaml"/>
+  <xacro:arg name="gazebo_controllers" default="$(find clearpath_control)/config/r100/control.yaml"/>
+  <xacro:arg name="use_platform_controllers" default="true"/>
+  <!-- Includes -->
+  <xacro:include filename="$(find clearpath_platform_description)/urdf/r100/wheels/wheel.urdf.xacro"/>
+  <xacro:include filename="$(find clearpath_platform_description)/urdf/r100/rocker.urdf.xacro"/>
   <!-- R100 Platform Macro -->
-  <xacro:macro name="r100" params="control:='omni_4wd' front_wheels:='mecanum' rear_wheels:='mecanum'">
+  <xacro:macro name="r100" params="wheel:='defaut'">
     <!-- Variables -->
+    <xacro:property name="wheel_radius" value="0.0759" />
+    <xacro:property name="wheel_width" value="0.0790" />
+    <xacro:property name="wheel_mass" value="2.5" />
     <xacro:property name="chassis_length" value="0.960" />
     <xacro:property name="chassis_width" value="0.793" />
@@ -12,5 +19,5 @@
     <xacro:property name="deck_height" value="0.280" />
     <xacro:property name="deck_thickness" value="0.005" />
-    <xacro:property name="riser_height" value="0.070" />
+    <xacro:property name="riser_height" value="0.055" />
     <xacro:property name="axle_offset" value="0.0500" />
     <xacro:property name="rocker_offset" value="0.319" />
@@ -193,26 +200,39 @@
       </collision>
     </link>
-    <!-- Add wheels -->
-    <xacro:include filename="$(find clearpath_platform_description)/urdf/r100/drivetrain/wheels.urdf.xacro"/>
-    <xacro:r100_drivetrain_wheels front_wheels="${front_wheels}" rear_wheels="${rear_wheels}"/>
-    <!-- Add drivetrain -->
-    <xacro:include filename="$(find clearpath_platform_description)/urdf/generic/drivetrain/drivetrain.urdf.xacro"/>
-    <!-- Hardware  -->
-    <xacro:if value="$(arg is_sim)">
-      <xacro:property name="hardware_plugin" value="gz_ros2_control/GazeboSimSystem"/>
-    </xacro:if>
-    <xacro:unless value="$(arg is_sim)">
-      <xacro:property name="hardware_plugin" value="clearpath_hardware_interfaces/PumaHardware"/>
-    </xacro:unless>
-    <xacro:unless value="${control == 'omni_4wd' or control == 'diff_4wd'}">
-      <xacro:error message="Invalid drivetrain control ${control}"/>
-    </xacro:unless>
-    <xacro:generic_drivetrain
-      name="r100"
-      control="${control}"
-      front_wheels="${front_wheels}"
-      rear_wheels="${rear_wheels}"
-      hardware_plugin="${hardware_plugin}"
-    />
+    <!-- Rocker -->
+    <xacro:r100_rocker prefix="front" joint_type="fixed" location="1" >
+      <limit lower="-0.08726" upper="0.08726" effort="0" velocity="0" />
+    </xacro:r100_rocker>
+    <xacro:r100_rocker prefix="rear" joint_type="fixed" location="-1" >
+      <limit effort="0" velocity="0" />
+    </xacro:r100_rocker>
+    <gazebo>
+      <plugin filename="libignition-gazebo-wheel-slip-system.so" name="ignition::gazebo::systems::WheelSlip">
+        <wheel link_name="front_left_wheel_link">
+          <slip_compliance_lateral>1.0</slip_compliance_lateral>
+          <slip_compliance_longitudinal>1.0</slip_compliance_longitudinal>
+          <wheel_normal_force>200</wheel_normal_force>
+          <wheel_radius>${wheel_radius}</wheel_radius>
+        </wheel>
+        <wheel link_name="front_right_wheel_link">
+          <slip_compliance_lateral>1.0</slip_compliance_lateral>
+          <slip_compliance_longitudinal>1.0</slip_compliance_longitudinal>
+          <wheel_normal_force>200</wheel_normal_force>
+          <wheel_radius>${wheel_radius}</wheel_radius>
+        </wheel>
+        <wheel link_name="rear_left_wheel_link">
+          <slip_compliance_lateral>1.0</slip_compliance_lateral>
+          <slip_compliance_longitudinal>1.0</slip_compliance_longitudinal>
+          <wheel_normal_force>200</wheel_normal_force>
+          <wheel_radius>${wheel_radius}</wheel_radius>
+        </wheel>
+        <wheel link_name="rear_right_wheel_link">
+          <slip_compliance_lateral>1.0</slip_compliance_lateral>
+          <slip_compliance_longitudinal>1.0</slip_compliance_longitudinal>
+          <wheel_normal_force>200</wheel_normal_force>
+          <wheel_radius>${wheel_radius}</wheel_radius>
+        </wheel>
+      </plugin>
+    </gazebo>
     <!-- Internal IMU -->
     <link name="imu_0_link">
@@ -233,5 +253,5 @@
         <update_rate>50</update_rate>
         <visualize>true</visualize>
-        <gz_frame_id>imu_0_link</gz_frame_id>
+        <ignition_frame_id>imu_0_link</ignition_frame_id>
       </sensor>
     </gazebo>
@@ -243,4 +263,39 @@
       <origin xyz="0 0 ${riser_height + deck_thickness}" rpy="0 0 0"/>
     </joint>
+    <!-- Gazebo Controller -->
+    <xacro:include filename="$(find clearpath_platform_description)/urdf/generic/gazebo.urdf.xacro"/>
+    <!-- ROS2 controls -->
+    <xacro:if value="$(arg use_platform_controllers)">
+      <ros2_control name="r100_hardware" type="system">
+        <hardware>
+          <xacro:if value="$(arg is_sim)">
+            <plugin>ign_ros2_control/IgnitionSystem</plugin>
+          </xacro:if>
+          <xacro:unless value="$(arg is_sim)">
+            <plugin>clearpath_hardware_interfaces/PumaHardware</plugin>
+          </xacro:unless>
+        </hardware>
+        <joint name="front_left_wheel_joint">
+          <command_interface name="velocity"/>
+          <state_interface name="position"/>
+          <state_interface name="velocity"/>
+        </joint>
+        <joint name="front_right_wheel_joint">
+          <command_interface name="velocity"/>
+          <state_interface name="position"/>
+          <state_interface name="velocity"/>
+        </joint>
+        <joint name="rear_left_wheel_joint">
+          <command_interface name="velocity"/>
+          <state_interface name="position"/>
+          <state_interface name="velocity"/>
+        </joint>
+        <joint name="rear_right_wheel_joint">
+          <command_interface name="velocity"/>
+          <state_interface name="position"/>
+          <state_interface name="velocity"/>
+        </joint>
+      </ros2_control>
+    </xacro:if>
   </xacro:macro>
 </robot>

File: clearpath_sensors_description/urdf/ouster_os1.urdf.xacro (robot description, xacro)
@@ -73,9 +73,9 @@
           </geometry>
         </collision>
-    </link>
-  </xacro:if>
-  <xacro:unless value="${base == 'base'}">
-    <link name="${name}_base_link" />
-  </xacro:unless>
+      </link>
+    </xacro:if>
+    <xacro:unless value="${base == 'base'}">
+      <link name="${name}_base_link" />
+    </xacro:unless>
     <!-- Lidar Link -->
     <link name="${name}_link">
