Commit message: Rebase from 'upstream'

File: clearpath_manipulators_description/urdf/arm/kinova_gen3_6dof.urdf.xacro (robot description, xacro)
@@ -549,5 +549,5 @@
             <optical_frame_id>color_optical_frame</optical_frame_id>
           </camera>
-          <ignition_frame_id>camera_color_frame</ignition_frame_id>
+          <gz_frame_id>camera_color_frame</gz_frame_id>
           <always_on>1</always_on>
           <update_rate>6</update_rate>

File: clearpath_manipulators_description/urdf/arm/kinova_gen3_7dof.urdf.xacro (robot description, xacro)
@@ -679,5 +679,5 @@
             <optical_frame_id>color_optical_frame</optical_frame_id>
           </camera>
-          <ignition_frame_id>camera_color_frame</ignition_frame_id>
+          <gz_frame_id>camera_color_frame</gz_frame_id>
           <always_on>1</always_on>
           <update_rate>6</update_rate>

File: clearpath_manipulators_description/urdf/arm/universal_robots.urdf.xacro (robot description, xacro)
@@ -58,14 +58,32 @@
     <xacro:property name="_safety_k_position" value="20" lazy_eval="false"/>
     <!-- Default Description Parameters Overwrites -->
-    <xacro:if value="${initial_positions != ''}"> <xacro:property name="_initial_positions" value="${initial_positions}" lazy_eval="false"/> </xacro:if>
+    <xacro:if value="${initial_positions != ''}">
+      <xacro:property name="_initial_positions" value="${initial_positions}" lazy_eval="false"/>
+    </xacro:if>
     <!-- if initial positions file is passed, overwrite initial positions parameter -->
-    <xacro:if value="${initial_positions_file != ''}"> <xacro:property name="_initial_positions" value="${xacro.load_yaml(initial_positions_file)}" lazy_eval="false"/> </xacro:if>
-    <xacro:if value="${joint_limits_parameters_file != ''}"> <xacro:property name="_joint_limits_parameters_file" value="${joint_limits_parameters_file}" lazy_eval="false"/> </xacro:if>
-    <xacro:if value="${kinematics_parameters_file != ''}"> <xacro:property name="_kinematics_parameters_file" value="${kinematics_parameters_file}" lazy_eval="false"/> </xacro:if>
-    <xacro:if value="${physical_parameters_file != ''}"> <xacro:property name="_physical_parameters_file" value="${physical_parameters_file}" lazy_eval="false"/> </xacro:if>
-    <xacro:if value="${visual_parameters_file != ''}"> <xacro:property name="$_visual_parameters_file" value="${visual_parameters_file}" lazy_eval="false"/> </xacro:if>
-    <xacro:if value="${safety_limits != ''}"> <xacro:property name="_safety_limits" value="${safety_limits}" lazy_eval="false"/> </xacro:if>
-    <xacro:if value="${safety_pos_margin != ''}"> <xacro:property name="_safety_pos_margin" value="${safety_pos_margin}" lazy_eval="false"/> </xacro:if>
-    <xacro:if value="${safety_k_position != ''}"> <xacro:property name="_safety_k_position" value="${safety_k_position}" lazy_eval="false"/> </xacro:if>
+    <xacro:if value="${initial_positions_file != ''}">
+      <xacro:property name="_initial_positions" value="${xacro.load_yaml(initial_positions_file)}" lazy_eval="false"/>
+    </xacro:if>
+    <xacro:if value="${joint_limits_parameters_file != ''}">
+      <xacro:property name="_joint_limits_parameters_file" value="${joint_limits_parameters_file}" lazy_eval="false"/>
+    </xacro:if>
+    <xacro:if value="${kinematics_parameters_file != ''}">
+      <xacro:property name="_kinematics_parameters_file" value="${kinematics_parameters_file}" lazy_eval="false"/>
+    </xacro:if>
+    <xacro:if value="${physical_parameters_file != ''}">
+      <xacro:property name="_physical_parameters_file" value="${physical_parameters_file}" lazy_eval="false"/>
+    </xacro:if>
+    <xacro:if value="${visual_parameters_file != ''}">
+      <xacro:property name="_visual_parameters_file" value="${visual_parameters_file}" lazy_eval="false"/>
+    </xacro:if>
+    <xacro:if value="${safety_limits != ''}">
+      <xacro:property name="_safety_limits" value="${safety_limits}" lazy_eval="false"/>
+    </xacro:if>
+    <xacro:if value="${safety_pos_margin != ''}">
+      <xacro:property name="_safety_pos_margin" value="${safety_pos_margin}" lazy_eval="false"/>
+    </xacro:if>
+    <xacro:if value="${safety_k_position != ''}">
+      <xacro:property name="_safety_k_position" value="${safety_k_position}" lazy_eval="false"/>
+    </xacro:if>
     <!-- Default Simulation Parameters -->
     <xacro:property name="_use_mock_hardware" value="false" />
@@ -74,8 +92,16 @@
     <xacro:property name="_sim_ignition" value="$(arg is_sim)" />
     <!-- Default Simulation Parameters Overwrites -->
-    <xacro:if value="${use_mock_hardware != ''}"> <xacro:property name="_use_mock_hardware" value="${use_mock_hardware}" lazy_eval="false"/> </xacro:if>
-    <xacro:if value="${mock_sensor_commands != ''}"> <xacro:property name="_mock_sensor_commands" value="${mock_sensor_commands}" lazy_eval="false"/> </xacro:if>
-    <xacro:if value="${sim_gazebo != ''}"> <xacro:property name="_sim_gazebo" value="${sim_gazebo}" lazy_eval="false"/> </xacro:if>
-    <xacro:if value="${sim_ignition != ''}"> <xacro:property name="_sim_ignition" value="${sim_ignition}" lazy_eval="false"/> </xacro:if>
+    <xacro:if value="${use_mock_hardware != ''}">
+      <xacro:property name="_use_mock_hardware" value="${use_mock_hardware}" lazy_eval="false"/>
+    </xacro:if>
+    <xacro:if value="${mock_sensor_commands != ''}">
+      <xacro:property name="_mock_sensor_commands" value="${mock_sensor_commands}" lazy_eval="false"/>
+    </xacro:if>
+    <xacro:if value="${sim_gazebo != ''}">
+      <xacro:property name="_sim_gazebo" value="${sim_gazebo}" lazy_eval="false"/>
+    </xacro:if>
+    <xacro:if value="${sim_ignition != ''}">
+      <xacro:property name="_sim_ignition" value="${sim_ignition}" lazy_eval="false"/>
+    </xacro:if>
     <!-- Default ros2_control Parameters -->
     <xacro:property name="_headless_mode" value="false" lazy_eval="false"/>
@@ -90,14 +116,34 @@
     <xacro:property name="_keep_alive_count" value="2.0" lazy_eval="false"/>
     <!-- Default ros2_control Parameters Overwrites -->
-    <xacro:if value="${headless_mode != ''}"> <xacro:property name="_headless_mode" value="${headless_mode}" lazy_eval="false"/> </xacro:if>
-    <xacro:if value="${robot_ip != ''}"> <xacro:property name="_robot_ip" value="${robot_ip}" lazy_eval="false"/> </xacro:if>
-    <xacro:if value="${reverse_ip != ''}"> <xacro:property name="_reverse_ip" value="${reverse_ip}" lazy_eval="false"/> </xacro:if>
-    <xacro:if value="${script_command_port != ''}"> <xacro:property name="_script_command_port" value="${script_command_port}" lazy_eval="false"/> </xacro:if>
-    <xacro:if value="${reverse_port != ''}"> <xacro:property name="_reverse_port" value="${reverse_port}" lazy_eval="false"/> </xacro:if>
-    <xacro:if value="${script_sender_port != ''}"> <xacro:property name="_script_sender_port" value="${script_sender_port}" lazy_eval="false"/> </xacro:if>
-    <xacro:if value="${trajectory_port != ''}"> <xacro:property name="_trajectory_port" value="${trajectory_port}" lazy_eval="false"/> </xacro:if>
-    <xacro:if value="${transmission_hw_interface != ''}"> <xacro:property name="_transmission_hw_interface" value="${transmission_hw_interface}" lazy_eval="false"/> </xacro:if>
-    <xacro:if value="${non_blocking_read != ''}"> <xacro:property name="_non_blocking_read" value="${non_blocking_read}" lazy_eval="false"/> </xacro:if>
-    <xacro:if value="${keep_alive_count != ''}"> <xacro:property name="_keep_alive_count" value="${keep_alive_count}" lazy_eval="false"/> </xacro:if>
+    <xacro:if value="${headless_mode != ''}">
+      <xacro:property name="_headless_mode" value="${headless_mode}" lazy_eval="false"/>
+    </xacro:if>
+    <xacro:if value="${robot_ip != ''}">
+      <xacro:property name="_robot_ip" value="${robot_ip}" lazy_eval="false"/>
+    </xacro:if>
+    <xacro:if value="${reverse_ip != ''}">
+      <xacro:property name="_reverse_ip" value="${reverse_ip}" lazy_eval="false"/>
+    </xacro:if>
+    <xacro:if value="${script_command_port != ''}">
+      <xacro:property name="_script_command_port" value="${script_command_port}" lazy_eval="false"/>
+    </xacro:if>
+    <xacro:if value="${reverse_port != ''}">
+      <xacro:property name="_reverse_port" value="${reverse_port}" lazy_eval="false"/>
+    </xacro:if>
+    <xacro:if value="${script_sender_port != ''}">
+      <xacro:property name="_script_sender_port" value="${script_sender_port}" lazy_eval="false"/>
+    </xacro:if>
+    <xacro:if value="${trajectory_port != ''}">
+      <xacro:property name="_trajectory_port" value="${trajectory_port}" lazy_eval="false"/>
+    </xacro:if>
+    <xacro:if value="${transmission_hw_interface != ''}">
+      <xacro:property name="_transmission_hw_interface" value="${transmission_hw_interface}" lazy_eval="false"/>
+    </xacro:if>
+    <xacro:if value="${non_blocking_read != ''}">
+      <xacro:property name="_non_blocking_read" value="${non_blocking_read}" lazy_eval="false"/>
+    </xacro:if>
+    <xacro:if value="${keep_alive_count != ''}">
+      <xacro:property name="_keep_alive_count" value="${keep_alive_count}" lazy_eval="false"/>
+    </xacro:if>
     <!-- Driver Dependent Parameters -->
     <xacro:if value="${use_manipulation_controllers and not _use_mock_hardware and not _sim_ignition}">
@@ -112,7 +158,13 @@
     </xacro:unless>
     <!-- Driver Dependent Parameters Overwrites -->
-    <xacro:if value="${script_filename != ''}"> <xacro:property name="_script_filename" value="${script_filename}" lazy_eval="false"/> </xacro:if>
-    <xacro:if value="${output_recipe_filename != ''}"> <xacro:property name="_output_recipe_filename" value="${output_recipe_filename}" lazy_eval="false"/> </xacro:if>
-    <xacro:if value="${input_recipe_filename != ''}"> <xacro:property name="_input_recipe_filename" value="${input_recipe_filename}" lazy_eval="false"/> </xacro:if>
+    <xacro:if value="${script_filename != ''}">
+      <xacro:property name="_script_filename" value="${script_filename}" lazy_eval="false"/>
+    </xacro:if>
+    <xacro:if value="${output_recipe_filename != ''}">
+      <xacro:property name="_output_recipe_filename" value="${output_recipe_filename}" lazy_eval="false"/>
+    </xacro:if>
+    <xacro:if value="${input_recipe_filename != ''}">
+      <xacro:property name="_input_recipe_filename" value="${input_recipe_filename}" lazy_eval="false"/>
+    </xacro:if>
     <!-- Default Tool Communication Parameters -->
     <xacro:property name="_use_tool_communication" value="false" lazy_eval="false"/>
@@ -126,13 +178,31 @@
     <xacro:property name="_tool_tcp_port" value="54321" lazy_eval="false"/>
     <!-- Tool Communication Parameter Overwrites -->
-    <xacro:if value="${use_tool_communication != ''}"> <xacro:property name="_use_tool_communication" value="${use_tool_communication}" lazy_eval="false"/> </xacro:if>
-    <xacro:if value="${tool_voltage != ''}"> <xacro:property name="_tool_voltage" value="${tool_voltage}" lazy_eval="false"/> </xacro:if>
-    <xacro:if value="${tool_parity != ''}"> <xacro:property name="_tool_parity" value="${tool_parity}" lazy_eval="false"/> </xacro:if>
-    <xacro:if value="${tool_baud_rate != ''}"> <xacro:property name="_tool_baud_rate" value="${tool_baud_rate}" lazy_eval="false"/> </xacro:if>
-    <xacro:if value="${tool_stop_bits != ''}"> <xacro:property name="_tool_stop_bits" value="${tool_stop_bits}" lazy_eval="false"/> </xacro:if>
-    <xacro:if value="${tool_rx_idle_chars != ''}"> <xacro:property name="_tool_rx_idle_chars" value="${tool_rx_idle_chars}" lazy_eval="false"/> </xacro:if>
-    <xacro:if value="${tool_tx_idle_chars != ''}"> <xacro:property name="_tool_tx_idle_chars" value="${tool_tx_idle_chars}" lazy_eval="false"/> </xacro:if>
-    <xacro:if value="${tool_device_name != ''}"> <xacro:property name="_tool_device_name" value="${tool_device_name}" lazy_eval="false"/> </xacro:if>
-    <xacro:if value="${tool_tcp_port != ''}"> <xacro:property name="_tool_tcp_port" value="${tool_tcp_port}" lazy_eval="false"/> </xacro:if>
+    <xacro:if value="${use_tool_communication != ''}">
+      <xacro:property name="_use_tool_communication" value="${use_tool_communication}" lazy_eval="false"/>
+    </xacro:if>
+    <xacro:if value="${tool_voltage != ''}">
+      <xacro:property name="_tool_voltage" value="${tool_voltage}" lazy_eval="false"/>
+    </xacro:if>
+    <xacro:if value="${tool_parity != ''}">
+      <xacro:property name="_tool_parity" value="${tool_parity}" lazy_eval="false"/>
+    </xacro:if>
+    <xacro:if value="${tool_baud_rate != ''}">
+      <xacro:property name="_tool_baud_rate" value="${tool_baud_rate}" lazy_eval="false"/>
+    </xacro:if>
+    <xacro:if value="${tool_stop_bits != ''}">
+      <xacro:property name="_tool_stop_bits" value="${tool_stop_bits}" lazy_eval="false"/>
+    </xacro:if>
+    <xacro:if value="${tool_rx_idle_chars != ''}">
+      <xacro:property name="_tool_rx_idle_chars" value="${tool_rx_idle_chars}" lazy_eval="false"/>
+    </xacro:if>
+    <xacro:if value="${tool_tx_idle_chars != ''}">
+      <xacro:property name="_tool_tx_idle_chars" value="${tool_tx_idle_chars}" lazy_eval="false"/>
+    </xacro:if>
+    <xacro:if value="${tool_device_name != ''}">
+      <xacro:property name="_tool_device_name" value="${tool_device_name}" lazy_eval="false"/>
+    </xacro:if>
+    <xacro:if value="${tool_tcp_port != ''}">
+      <xacro:property name="_tool_tcp_port" value="${tool_tcp_port}" lazy_eval="false"/>
+    </xacro:if>
     <!-- Universal Robots ROS2 Description -->
     <xacro:ur_robot
@@ -146,40 +216,82 @@
       safety_limits="${_safety_limits}"
       safety_pos_margin="${_safety_pos_margin}"
-      safety_k_position="${_safety_k_position}"
-      >
+      safety_k_position="${_safety_k_position}">
       <xacro:insert_block name="origin"/>
     </xacro:ur_robot>
-    <!-- Universal_Robots_ROS2_Driver HardwareInterface -->
-    <xacro:if value="${use_manipulation_controllers}">
-      <xacro:include filename="$(find ur_robot_driver)/urdf/ur.ros2_control.xacro" />
-      <xacro:ur_ros2_control
-        name="${name}"
-        tf_prefix="${_tf_prefix}"
-        kinematics_parameters_file="${_kinematics_parameters_file}"
-        transmission_hw_interface="${_transmission_hw_interface}"
-        use_mock_hardware="${_use_mock_hardware}"
-        mock_sensor_commands="${_mock_sensor_commands}"
-        headless_mode="${_headless_mode}"
-        initial_positions="${_initial_positions}"
-        use_tool_communication="${_use_tool_communication}"
-        tool_voltage="${_tool_voltage}"
-        tool_parity="${_tool_parity}"
-        tool_baud_rate="${_tool_baud_rate}"
-        tool_stop_bits="${_tool_stop_bits}"
-        tool_rx_idle_chars="${_tool_rx_idle_chars}"
-        tool_tx_idle_chars="${_tool_tx_idle_chars}"
-        tool_device_name="${_tool_device_name}"
-        tool_tcp_port="${_tool_tcp_port}"
-        robot_ip="${_robot_ip}"
-        script_filename="${_script_filename}"
-        output_recipe_filename="${_output_recipe_filename}"
-        input_recipe_filename="${_input_recipe_filename}"
-        reverse_ip="${_reverse_ip}"
-        script_command_port="${_script_command_port}"
-        reverse_port="${_reverse_port}"
-        script_sender_port="${_script_sender_port}"
-        trajectory_port="${_trajectory_port}"
-      />
-    </xacro:if>
+    <!-- Use the right ros2_control depending on sim vs real -->
+    <xacro:if value="${_sim_ignition}">
+      <ros2_control name="${name}_hardware" type="system">
+        <hardware>
+          <plugin>gz_ros2_control/GazeboSimSystem</plugin>
+        </hardware>
+        <joint name="${name}_shoulder_pan_joint">
+          <command_interface name="position"/>
+          <state_interface name="position"/>
+          <state_interface name="velocity"/>
+        </joint>
+        <joint name="${name}_shoulder_lift_joint">
+          <command_interface name="position"/>
+          <state_interface name="position"/>
+          <state_interface name="velocity"/>
+        </joint>
+        <joint name="${name}_elbow_joint">
+          <command_interface name="position"/>
+          <state_interface name="position"/>
+          <state_interface name="velocity"/>
+        </joint>
+        <joint name="${name}_wrist_1_joint">
+          <command_interface name="position"/>
+          <state_interface name="position"/>
+          <state_interface name="velocity"/>
+        </joint>
+        <joint name="${name}_wrist_2_joint">
+          <command_interface name="position"/>
+          <state_interface name="position"/>
+          <state_interface name="velocity"/>
+        </joint>
+        <joint name="${name}_wrist_3_joint">
+          <command_interface name="position"/>
+          <state_interface name="position"/>
+          <state_interface name="velocity"/>
+        </joint>
+      </ros2_control>
+      <gazebo>
+        <plugin filename="gz_ros2_control-system"
+                name="gz_ros2_control::GazeboSimROS2ControlPlugin"/>
+      </gazebo>
+    </xacro:if>
+    <!-- REAL ROBOT: only include the UR driver when NOT sim -->
+    <xacro:unless value="${_sim_ignition}">
+      <xacro:if value="${use_manipulation_controllers}">
+        <xacro:include filename="$(find ur_robot_driver)/urdf/ur.ros2_control.xacro" />
+        <xacro:ur_ros2_control
+          name="${name}"
+          tf_prefix="${_tf_prefix}"
+          kinematics_parameters_file="${_kinematics_parameters_file}"
+          transmission_hw_interface="${_transmission_hw_interface}"
+          use_mock_hardware="${_use_mock_hardware}"
+          mock_sensor_commands="${_mock_sensor_commands}"
+          headless_mode="${_headless_mode}"
+          initial_positions="${_initial_positions}"
+          use_tool_communication="${_use_tool_communication}"
+          tool_voltage="${_tool_voltage}"
+          tool_parity="${_tool_parity}"
+          tool_baud_rate="${_tool_baud_rate}"
+          tool_stop_bits="${_tool_stop_bits}"
+          tool_rx_idle_chars="${_tool_rx_idle_chars}"
+          tool_tx_idle_chars="${_tool_tx_idle_chars}"
+          tool_device_name="${_tool_device_name}"
+          tool_tcp_port="${_tool_tcp_port}"
+          robot_ip="${_robot_ip}"
+          script_filename="${_script_filename}"
+          output_recipe_filename="${_output_recipe_filename}"
+          input_recipe_filename="${_input_recipe_filename}"
+          reverse_ip="${_reverse_ip}"
+          script_command_port="${_script_command_port}"
+          reverse_port="${_reverse_port}"
+          script_sender_port="${_script_sender_port}"
+          trajectory_port="${_trajectory_port}"/>
+      </xacro:if>
+    </xacro:unless>
   </xacro:macro>
 </robot>

File: clearpath_manipulators_description/urdf/gripper/kinova_2f_lite.urdf.xacro (robot description, xacro)
@@ -79,5 +79,5 @@
       <child link="${name}_right_finger_prox_link" />
       <axis xyz="0 0 -1" />
-      <limit lower="0.0" upper="0.85" effort="1000" velocity="0.6" />
+      <limit lower="-0.1" upper="0.96" effort="10" velocity="0.6" />
     </joint>
     <!-- Right Finger Dist -->
@@ -146,5 +146,5 @@
       <child link="${name}_left_finger_prox_link" />
       <axis xyz="0 0 1" />
-      <limit lower="0.0" upper="0.85" effort="1000" velocity="1000" />
+      <limit lower="-0.1" upper="0.96" effort="10" velocity="0.6" />
       <mimic joint="${name}_right_finger_bottom_joint" multiplier="1.0" offset="0.0" />
     </joint>

File: clearpath_sensors_description/urdf/ouster_os1.urdf.xacro (robot description, xacro)
@@ -205,5 +205,5 @@
         <visualize>true</visualize>
         <always_on>true</always_on>
-        <ignition_frame_id>${name}_sensor_link</ignition_frame_id>
+        <gz_frame_id>${name}_sensor_link</gz_frame_id>
         <topic>$(arg namespace)/sensors/${name}/scan</topic>
         <lidar>
