Commit message: Imported upstream version '1.3.6' of 'upstream'

File: clearpath_platform_description/urdf/dd100/dd100.urdf.xacro (robot description, xacro)
@@ -3,10 +3,15 @@
   <xacro:arg name="namespace" default="" />
   <xacro:arg name="is_sim" default="false" />
-  <xacro:arg name="gazebo_controllers" default="$(find clearpath_control)/config/dd100/control/diff_fwd.yaml"/>
+  <xacro:arg name="gazebo_controllers" default="$(find clearpath_control)/config/dd100/control.yaml"/>
   <xacro:arg name="use_platform_controllers" default="true"/>
+  <!-- Included URDF/XACRO Files -->
+  <xacro:include filename="$(find clearpath_platform_description)/urdf/dd100/wheels/wheel.urdf.xacro"/>
   <xacro:property name="PI" value="${math.pi}" />
   <!-- DD100 Platform Macro -->
-  <xacro:macro name="dd100" params="control:='diff_fwd' front_wheels:='indoor' rear_wheels:='caster'">
+  <xacro:macro name="dd100" params="wheel:='default'">
     <!-- Variables -->
+    <xacro:property name="wheel_radius" value="0.049" />
+    <xacro:property name="wheel_mass" value="0.111" />
+    <xacro:property name="wheel_width" value="0.02032" />
     <xacro:property name="wheel_x_offset" value="0.0989838" />
     <xacro:property name="wheel_z_offset" value="0.0345" />
@@ -42,26 +47,75 @@
         </inertial>
     </link>
-    <!-- Add wheels -->
-    <xacro:include filename="$(find clearpath_platform_description)/urdf/dd100/drivetrain/wheels.urdf.xacro"/>
-    <xacro:dd100_drivetrain_wheels front_wheels="${front_wheels}" rear_wheels="${rear_wheels}"/>
-    <!-- Add drivetrain -->
-    <xacro:include filename="$(find clearpath_platform_description)/urdf/generic/drivetrain/drivetrain.urdf.xacro"/>
-    <!-- Hardware  -->
-    <xacro:if value="$(arg is_sim)">
-      <xacro:property name="hardware_plugin" value="gz_ros2_control/GazeboSimSystem"/>
-    </xacro:if>
-    <xacro:unless value="$(arg is_sim)">
-      <xacro:property name="hardware_plugin" value="clearpath_hardware_interfaces/PumaHardware"/>
-    </xacro:unless>
-    <xacro:unless value="${control == 'diff_fwd'}">
-      <xacro:error message="Invalid drivetrain control ${control}"/>
-    </xacro:unless>
-    <xacro:generic_drivetrain
-      name="dd100"
-      control="${control}"
-      front_wheels="${front_wheels}"
-      rear_wheels="${rear_wheels}"
-      hardware_plugin="${hardware_plugin}"
-    />
+    <!-- Wheels -->
+    <xacro:dd100_wheel prefix="front_left">
+      <origin xyz="${wheel_x_offset} ${wheelbase+wheel_width/2} ${wheel_z_offset}" rpy="0 0 0" />
+    </xacro:dd100_wheel>
+    <xacro:dd100_wheel prefix="front_right">
+      <origin xyz="${wheel_x_offset} ${-wheelbase-wheel_width/2} ${wheel_z_offset}" rpy="0 0 0" />
+    </xacro:dd100_wheel>
+    <gazebo>
+      <plugin filename="libignition-gazebo-wheel-slip-system.so" name="ignition::gazebo::systems::WheelSlip">
+        <wheel link_name="front_left_wheel_link">
+          <slip_compliance_lateral>1.0</slip_compliance_lateral>
+          <slip_compliance_longitudinal>1.0</slip_compliance_longitudinal>
+          <wheel_normal_force>39.2</wheel_normal_force>
+          <wheel_radius>${wheel_radius}</wheel_radius>
+        </wheel>
+        <wheel link_name="front_right_wheel_link">
+          <slip_compliance_lateral>1.0</slip_compliance_lateral>
+          <slip_compliance_longitudinal>1.0</slip_compliance_longitudinal>
+          <wheel_normal_force>39.2</wheel_normal_force>
+          <wheel_radius>${wheel_radius}</wheel_radius>
+        </wheel>
+      </plugin>
+    </gazebo>
+    <!-- Caster -->
+    <link name="rear_caster">
+      <visual>
+        <origin rpy="0 0 0" xyz="0 0 0"/>
+        <geometry>
+          <sphere radius="0.01"/>
+        </geometry>
+        <material name="clearpath_black"/>
+      </visual>
+      <collision>
+        <geometry>
+          <sphere radius="0.01"/>
+        </geometry>
+        <origin rpy="0 0 0" xyz="0 0 0"/>
+        <surface>
+          <friction>
+            <ode>
+              <mu>0.0</mu>
+              <mu2>0.0</mu2>
+              <slip1>1.0</slip1>
+              <slip2>1.0</slip2>
+            </ode>
+          </friction>
+        </surface>
+      </collision>
+      <inertial>
+        <mass value="0.1" />
+        <origin xyz="0 0 0" />
+        <inertia ixx="0.001" ixy="0.0" ixz="0.0"
+                iyy="0.001" iyz="0.0"
+                izz="0.001" />
+      </inertial>
+    </link>
+    <joint name="rear_caster_joint" type="fixed">
+      <parent link="chassis_link"/>
+      <child link="rear_caster"/>
+      <origin xyz="-0.244 0 -0.00674" rpy="0 0 0"/>
+    </joint>
+    <gazebo reference="rear_caster">
+      <turnGravityOff>false</turnGravityOff>
+      <kp>1000000.0</kp>
+      <kd>100.0</kd>
+      <mu1>0.2</mu1>
+      <mu2>0.2</mu2>
+      <fdir1>1 0 0</fdir1>
+      <minDepth>0.00</minDepth>
+      <implicitSpringDamper>1</implicitSpringDamper>
+    </gazebo>
     <!-- Internal IMU -->
     <link name="imu_0_link">
@@ -81,5 +135,5 @@
         <update_rate>50</update_rate>
         <visualize>true</visualize>
-        <gz_frame_id>imu_0_link</gz_frame_id>
+        <ignition_frame_id>imu_0_link</ignition_frame_id>
         <topic>$(arg namespace)/sensors/imu_0/data_raw</topic>
       </sensor>
@@ -141,4 +195,29 @@
       <child link="rear_bumper_mount" />
     </joint>
+    <!-- Gazebo Controller -->
+    <xacro:include filename="$(find clearpath_platform_description)/urdf/generic/gazebo.urdf.xacro"/>
+    <!-- ROS2 controls -->
+    <xacro:if value="$(arg use_platform_controllers)">
+      <ros2_control name="dd100_hardware" type="system">
+        <hardware>
+          <xacro:if value="$(arg is_sim)">
+            <plugin>ign_ros2_control/IgnitionSystem</plugin>
+          </xacro:if>
+          <xacro:unless value="$(arg is_sim)">
+            <plugin>clearpath_hardware_interfaces/PumaHardware</plugin>
+          </xacro:unless>
+        </hardware>
+        <joint name="front_left_wheel_joint">
+          <command_interface name="velocity"/>
+          <state_interface name="position"/>
+          <state_interface name="velocity"/>
+        </joint>
+        <joint name="front_right_wheel_joint">
+          <command_interface name="velocity"/>
+          <state_interface name="position"/>
+          <state_interface name="velocity"/>
+        </joint>
+      </ros2_control>
+    </xacro:if>
   </xacro:macro>
 </robot>

File: clearpath_platform_description/urdf/dd150/dd150.urdf.xacro (robot description, xacro)
@@ -3,10 +3,15 @@
   <xacro:arg name="namespace" default="" />
   <xacro:arg name="is_sim" default="false" />
-  <xacro:arg name="gazebo_controllers" default="$(find clearpath_control)/config/dd150/control/diff_fwd.yaml"/>
+  <xacro:arg name="gazebo_controllers" default="$(find clearpath_control)/config/dd150/control.yaml"/>
   <xacro:arg name="use_platform_controllers" default="true"/>
-  <xacro:property name="PI" value="${math.pi}" />
+  <!-- Included URDF/XACRO Files -->
+  <xacro:include filename="$(find clearpath_platform_description)/urdf/dd150/wheels/wheel.urdf.xacro"/>
+  <xacro:property name="PI" value="3.1415926535897931" />
   <!-- DD150 Platform Macro -->
-  <xacro:macro name="dd150" params="control:='diff_fwd' front_wheels:='indoor' rear_wheels:='caster'">
+  <xacro:macro name="dd150" params="wheel:='default'">
     <!-- Variables -->
+    <xacro:property name="wheel_radius" value="0.049" />
+    <xacro:property name="wheel_mass" value="0.111" />
+    <xacro:property name="wheel_width" value="0.02032" />
     <xacro:property name="wheel_x_offset" value="0.0989838" />
     <xacro:property name="wheel_z_offset" value="0.0345" />
@@ -42,26 +47,75 @@
         </inertial>
     </link>
-    <!-- Add wheels -->
-    <xacro:include filename="$(find clearpath_platform_description)/urdf/dd100/drivetrain/wheels.urdf.xacro"/>
-    <xacro:dd100_drivetrain_wheels front_wheels="${front_wheels}" rear_wheels="${rear_wheels}"/>
-    <!-- Add drivetrain -->
-    <xacro:include filename="$(find clearpath_platform_description)/urdf/generic/drivetrain/drivetrain.urdf.xacro"/>
-    <!-- Hardware  -->
-    <xacro:if value="$(arg is_sim)">
-      <xacro:property name="hardware_plugin" value="gz_ros2_control/GazeboSimSystem"/>
-    </xacro:if>
-    <xacro:unless value="$(arg is_sim)">
-      <xacro:property name="hardware_plugin" value="clearpath_hardware_interfaces/PumaHardware"/>
-    </xacro:unless>
-    <xacro:unless value="${control == 'diff_fwd'}">
-      <xacro:error message="Invalid drivetrain control ${control}"/>
-    </xacro:unless>
-    <xacro:generic_drivetrain
-      name="dd150"
-      control="${control}"
-      front_wheels="${front_wheels}"
-      rear_wheels="${rear_wheels}"
-      hardware_plugin="${hardware_plugin}"
-    />
+    <!-- Wheels -->
+    <xacro:dd150_wheel prefix="front_left">
+      <origin xyz="${wheel_x_offset} ${wheelbase+wheel_width/2} ${wheel_z_offset}" rpy="0 0 0" />
+    </xacro:dd150_wheel>
+    <xacro:dd150_wheel prefix="front_right">
+      <origin xyz="${wheel_x_offset} ${-wheelbase-wheel_width/2} ${wheel_z_offset}" rpy="0 0 0" />
+    </xacro:dd150_wheel>
+    <gazebo>
+      <plugin filename="libignition-gazebo-wheel-slip-system.so" name="ignition::gazebo::systems::WheelSlip">
+        <wheel link_name="front_left_wheel_link">
+          <slip_compliance_lateral>1.0</slip_compliance_lateral>
+          <slip_compliance_longitudinal>1.0</slip_compliance_longitudinal>
+          <wheel_normal_force>39.2</wheel_normal_force>
+          <wheel_radius>${wheel_radius}</wheel_radius>
+        </wheel>
+        <wheel link_name="front_right_wheel_link">
+          <slip_compliance_lateral>1.0</slip_compliance_lateral>
+          <slip_compliance_longitudinal>1.0</slip_compliance_longitudinal>
+          <wheel_normal_force>39.2</wheel_normal_force>
+          <wheel_radius>${wheel_radius}</wheel_radius>
+        </wheel>
+      </plugin>
+    </gazebo>
+    <!-- Caster -->
+    <link name="rear_caster">
+      <visual>
+        <origin rpy="0 0 0" xyz="0 0 0"/>
+        <geometry>
+          <sphere radius="0.01"/>
+        </geometry>
+        <material name="clearpath_black"/>
+      </visual>
+      <collision>
+        <geometry>
+          <sphere radius="0.01"/>
+        </geometry>
+        <origin rpy="0 0 0" xyz="0 0 0"/>
+        <surface>
+          <friction>
+            <ode>
+              <mu>0.0</mu>
+              <mu2>0.0</mu2>
+              <slip1>1.0</slip1>
+              <slip2>1.0</slip2>
+            </ode>
+          </friction>
+        </surface>
+      </collision>
+      <inertial>
+        <mass value="0.1" />
+        <origin xyz="0 0 0" />
+        <inertia ixx="0.001" ixy="0.0" ixz="0.0"
+                iyy="0.001" iyz="0.0"
+                izz="0.001" />
+      </inertial>
+    </link>
+    <joint name="rear_caster_joint" type="fixed">
+      <parent link="chassis_link"/>
+      <child link="rear_caster"/>
+      <origin xyz="-0.244 0 -0.00674" rpy="0 0 0"/>
+    </joint>
+    <gazebo reference="rear_caster">
+      <turnGravityOff>false</turnGravityOff>
+      <kp>1000000.0</kp>
+      <kd>100.0</kd>
+      <mu1>0.2</mu1>
+      <mu2>0.2</mu2>
+      <fdir1>1 0 0</fdir1>
+      <minDepth>0.00</minDepth>
+      <implicitSpringDamper>1</implicitSpringDamper>
+    </gazebo>
     <!-- Internal IMU -->
     <link name="imu_0_link">
@@ -81,5 +135,5 @@
         <update_rate>50</update_rate>
         <visualize>true</visualize>
-        <gz_frame_id>imu_0_link</gz_frame_id>
+        <ignition_frame_id>imu_0_link</ignition_frame_id>
         <topic>$(arg namespace)/sensors/imu_0/data_raw</topic>
       </sensor>
@@ -87,18 +141,16 @@
     <!-- Mounting Hard Points -->
     <link name="default_mount"/>
-    <link name="front_2_mount"/>
     <link name="front_1_mount"/>
     <link name="front_0_mount"/>
-    <link name="rear_2_mount"/>
     <link name="rear_1_mount"/>
     <link name="rear_0_mount"/>
     <joint name="default_mount_joint" type="fixed">
-      <origin xyz="0 0 0" rpy="0 0 0"/>
-      <parent link="front_0_mount"/>
-      <child link="default_mount"/>
+      <origin xyz="-0.0124 0 0.064263" rpy="0 0 0" />
+      <parent link="chassis_link"/>
+      <child link="default_mount" />
     </joint>
     <joint name="front_0_mount_joint" type="fixed">
-      <origin xyz="0.040 0 0.064263" rpy="0 0 0" />
-      <parent link="chassis_link"/>
+      <origin xyz="0.1324 0 0" rpy="0 0 0" />
+      <parent link="default_mount"/>
       <child link="front_0_mount" />
     </joint>
@@ -108,12 +160,7 @@
       <child link="front_1_mount" />
     </joint>
-    <joint name="front_2_mount_joint" type="fixed">
-      <origin xyz="0.080 0 0" rpy="0 0 0" />
-      <parent link="front_1_mount"/>
-      <child link="front_2_mount" />
-    </joint>
     <joint name="rear_0_mount_joint" type="fixed">
-      <origin xyz="-0.040 0 0.064263" rpy="0 0 0" />
-      <parent link="chassis_link"/>
+      <origin xyz="-0.080 0 0.0" rpy="0 0 0" />
+      <parent link="default_mount"/>
       <child link="rear_0_mount" />
     </joint>
@@ -122,9 +169,4 @@
       <parent link="rear_0_mount"/>
       <child link="rear_1_mount" />
-    </joint>
-    <joint name="rear_2_moint_joint" type="fixed">
-      <origin xyz="-0.080 0 0" rpy="0 0 0" />
-      <parent link="rear_1_mount"/>
-      <child link="rear_2_mount" />
     </joint>
     <!-- Bumper Mounts -->
@@ -141,4 +183,29 @@
       <child link="rear_bumper_mount" />
     </joint>
+    <!-- Gazebo Controller -->
+    <xacro:include filename="$(find clearpath_platform_description)/urdf/generic/gazebo.urdf.xacro"/>
+    <!-- ROS2 controls -->
+    <xacro:if value="$(arg use_platform_controllers)">
+      <ros2_control name="dd150_hardware" type="system">
+        <hardware>
+          <xacro:if value="$(arg is_sim)">
+            <plugin>ign_ros2_control/IgnitionSystem</plugin>
+          </xacro:if>
+          <xacro:unless value="$(arg is_sim)">
+            <plugin>clearpath_hardware_interfaces/PumaHardware</plugin>
+          </xacro:unless>
+        </hardware>
+        <joint name="front_left_wheel_joint">
+          <command_interface name="velocity"/>
+          <state_interface name="position"/>
+          <state_interface name="velocity"/>
+        </joint>
+        <joint name="front_right_wheel_joint">
+          <command_interface name="velocity"/>
+          <state_interface name="position"/>
+          <state_interface name="velocity"/>
+        </joint>
+      </ros2_control>
+    </xacro:if>
   </xacro:macro>
 </robot>

File: clearpath_platform_description/urdf/j100/j100.urdf.xacro (robot description, xacro)
@@ -2,4 +2,5 @@
 <robot name="j100"
   xmlns:xacro="http://www.ros.org/wiki/xacro">
+  <xacro:include filename="$(find clearpath_platform_description)/urdf/j100/wheels/wheel.urdf.xacro"/>
   <xacro:arg name="is_sim" default="false" />
   <xacro:arg name="prefix" default="" />
@@ -12,4 +13,6 @@
   <xacro:property name="wheel_vertical_offset" value="0.0345" />
   <xacro:property name="footprint_vertical_offset" value="-0.0655" />
+  <xacro:property name="wheel_radius" value="0.098" />
+  <xacro:property name="wheel_width" value="0.040" />
   <xacro:property name="chassis_length" value="0.420" />
   <xacro:property name="chassis_width" value="0.310" />
@@ -17,5 +20,45 @@
   <xacro:property name="dummy_inertia" value="1e-09"/>
   <xacro:property name="mount_spacing" value="0.120" />
-  <xacro:macro name="j100" params="control:='diff_fwd' front_wheels:='outdoor' rear_wheels:='outdoor'">
+  <xacro:macro name="j100" params="wheel:='default'">
+    <xacro:j100_wheel prefix="front_left">
+      <origin xyz="${wheelbase/2} ${track/2} ${wheel_vertical_offset}" rpy="0 0 0" />
+    </xacro:j100_wheel>
+    <xacro:j100_wheel prefix="front_right">
+      <origin xyz="${wheelbase/2} ${-track/2} ${wheel_vertical_offset}" rpy="0 0 0" />
+    </xacro:j100_wheel>
+    <xacro:j100_wheel prefix="rear_left">
+      <origin xyz="${-wheelbase/2} ${track/2} ${wheel_vertical_offset}" rpy="0 0 0" />
+    </xacro:j100_wheel>
+    <xacro:j100_wheel prefix="rear_right">
+      <origin xyz="${-wheelbase/2} ${-track/2} ${wheel_vertical_offset}" rpy="0 0 0" />
+    </xacro:j100_wheel>
+    <gazebo>
+      <plugin filename="libignition-gazebo-wheel-slip-system.so" name="ignition::gazebo::systems::WheelSlip">
+        <wheel link_name="front_left_wheel_link">
+          <slip_compliance_lateral>1.0</slip_compliance_lateral>
+          <slip_compliance_longitudinal>1.0</slip_compliance_longitudinal>
+          <wheel_normal_force>40</wheel_normal_force>
+          <wheel_radius>${wheel_radius}</wheel_radius>
+        </wheel>
+        <wheel link_name="front_right_wheel_link">
+          <slip_compliance_lateral>1.0</slip_compliance_lateral>
+          <slip_compliance_longitudinal>1.0</slip_compliance_longitudinal>
+          <wheel_normal_force>40</wheel_normal_force>
+          <wheel_radius>${wheel_radius}</wheel_radius>
+        </wheel>
+        <wheel link_name="rear_left_wheel_link">
+          <slip_compliance_lateral>1.0</slip_compliance_lateral>
+          <slip_compliance_longitudinal>1.0</slip_compliance_longitudinal>
+          <wheel_normal_force>40</wheel_normal_force>
+          <wheel_radius>${wheel_radius}</wheel_radius>
+        </wheel>
+        <wheel link_name="rear_right_wheel_link">
+          <slip_compliance_lateral>1.0</slip_compliance_lateral>
+          <slip_compliance_longitudinal>1.0</slip_compliance_longitudinal>
+          <wheel_normal_force>40</wheel_normal_force>
+          <wheel_radius>${wheel_radius}</wheel_radius>
+        </wheel>
+      </plugin>
+    </gazebo>
     <link name="base_link"></link>
     <joint name="base_link_joint" type="fixed">
@@ -44,23 +87,4 @@
       </inertial>
     </link>
-    <!-- Add wheels -->
-    <xacro:include filename="$(find clearpath_platform_description)/urdf/j100/drivetrain/wheels.urdf.xacro"/>
-    <xacro:j100_drivetrain_wheels front_wheels="${front_wheels}" rear_wheels="${rear_wheels}"/>
-    <!-- Add drivetrain -->
-    <xacro:include filename="$(find clearpath_platform_description)/urdf/generic/drivetrain/drivetrain.urdf.xacro"/>
-    <!-- Hardware  -->
-    <xacro:if value="$(arg is_sim)">
-      <xacro:property name="hardware_plugin" value="gz_ros2_control/GazeboSimSystem"/>
-    </xacro:if>
-    <xacro:unless value="$(arg is_sim)">
-      <xacro:property name="hardware_plugin" value="clearpath_hardware_interfaces/J100Hardware"/>
-    </xacro:unless>
-    <xacro:generic_drivetrain
-      name="j100"
-      control="${control}"
-      front_wheels="${front_wheels}"
-      rear_wheels="${rear_wheels}"
-      hardware_plugin="${hardware_plugin}"
-    />
     <link name="imu_0_link">
       <inertial>
@@ -79,5 +103,5 @@
         <update_rate>50</update_rate>
         <visualize>true</visualize>
-        <gz_frame_id>imu_0_link</gz_frame_id>
+        <ignition_frame_id>imu_0_link</ignition_frame_id>
         <topic>$(arg namespace)/sensors/imu_0/data_raw</topic>
       </sensor>
@@ -101,5 +125,5 @@
         <always_on>1</always_on>
         <update_rate>10</update_rate>
-        <gz_frame_id>gps_0_link</gz_frame_id>
+        <ignition_frame_id>gps_0_link</ignition_frame_id>
         <topic>$(arg namespace)/sensors/gps_0/navsat</topic>
       </sensor>
@@ -123,4 +147,39 @@
       <origin xyz="${mount_spacing} 0 0" />
     </joint>
+    <!-- Gazebo Controller -->
+    <xacro:include filename="$(find clearpath_platform_description)/urdf/generic/gazebo.urdf.xacro"/>
+    <!-- ROS2 controls -->
+    <xacro:if value="$(arg use_platform_controllers)">
+      <ros2_control name="j100_hardware" type="system">
+        <hardware>
+          <xacro:if value="$(arg is_sim)">
+            <plugin>ign_ros2_control/IgnitionSystem</plugin>
+          </xacro:if>
+          <xacro:unless value="$(arg is_sim)">
+            <plugin>clearpath_hardware_interfaces/J100Hardware</plugin>
+          </xacro:unless>
+        </hardware>
+        <joint name="front_left_wheel_joint">
+          <command_interface name="velocity"/>
+          <state_interface name="position"/>
+          <state_interface name="velocity"/>
+        </joint>
+        <joint name="rear_left_wheel_joint">
+          <command_interface name="velocity"/>
+          <state_interface name="position"/>
+          <state_interface name="velocity"/>
+        </joint>
+        <joint name="front_right_wheel_joint">
+          <command_interface name="velocity"/>
+          <state_interface name="position"/>
+          <state_interface name="velocity"/>
+        </joint>
+        <joint name="rear_right_wheel_joint">
+          <command_interface name="velocity"/>
+          <state_interface name="position"/>
+          <state_interface name="velocity"/>
+        </joint>
+      </ros2_control>
+    </xacro:if>
   </xacro:macro>
 </robot>
