Commit message: Rebase from 'upstream'

File: clearpath_platform_description/urdf/a300/a300.urdf.xacro (robot description, xacro)
@@ -132,11 +132,13 @@
       <xacro:property name="hardware_plugin" value="clearpath_hardware_interfaces/LynxHardware"/>
     </xacro:unless>
-    <xacro:generic_drivetrain
-      name="a300"
-      control="${control}"
-      front_wheels="${front_wheels}"
-      rear_wheels="${rear_wheels}"
-      hardware_plugin="${hardware_plugin}"
-    />
+    <xacro:if value="$(arg use_platform_controllers)">
+      <xacro:generic_drivetrain
+        name="a300"
+        control="${control}"
+        front_wheels="${front_wheels}"
+        rear_wheels="${rear_wheels}"
+        hardware_plugin="${hardware_plugin}"
+      />
+    </xacro:if>
     <!-- Base Footprint: on the ground below the robot -->
     <link name="base_footprint"/>

File: clearpath_platform_description/urdf/dd100/dd100.urdf.xacro (robot description, xacro)
@@ -57,11 +57,13 @@
       <xacro:error message="Invalid drivetrain control ${control}"/>
     </xacro:unless>
-    <xacro:generic_drivetrain
-      name="dd100"
-      control="${control}"
-      front_wheels="${front_wheels}"
-      rear_wheels="${rear_wheels}"
-      hardware_plugin="${hardware_plugin}"
-    />
+    <xacro:if value="$(arg use_platform_controllers)">
+      <xacro:generic_drivetrain
+        name="dd100"
+        control="${control}"
+        front_wheels="${front_wheels}"
+        rear_wheels="${rear_wheels}"
+        hardware_plugin="${hardware_plugin}"
+      />
+    </xacro:if>
     <!-- Internal IMU -->
     <link name="imu_0_link">

File: clearpath_platform_description/urdf/dd150/dd150.urdf.xacro (robot description, xacro)
@@ -57,11 +57,13 @@
       <xacro:error message="Invalid drivetrain control ${control}"/>
     </xacro:unless>
-    <xacro:generic_drivetrain
-      name="dd150"
-      control="${control}"
-      front_wheels="${front_wheels}"
-      rear_wheels="${rear_wheels}"
-      hardware_plugin="${hardware_plugin}"
-    />
+    <xacro:if value="$(arg use_platform_controllers)">
+      <xacro:generic_drivetrain
+        name="dd150"
+        control="${control}"
+        front_wheels="${front_wheels}"
+        rear_wheels="${rear_wheels}"
+        hardware_plugin="${hardware_plugin}"
+      />
+    </xacro:if>
     <!-- Internal IMU -->
     <link name="imu_0_link">

File: clearpath_platform_description/urdf/j100/j100.urdf.xacro (robot description, xacro)
@@ -56,11 +56,13 @@
       <xacro:property name="hardware_plugin" value="clearpath_hardware_interfaces/J100Hardware"/>
     </xacro:unless>
-    <xacro:generic_drivetrain
-      name="j100"
-      control="${control}"
-      front_wheels="${front_wheels}"
-      rear_wheels="${rear_wheels}"
-      hardware_plugin="${hardware_plugin}"
-    />
+    <xacro:if value="$(arg use_platform_controllers)">
+      <xacro:generic_drivetrain
+        name="j100"
+        control="${control}"
+        front_wheels="${front_wheels}"
+        rear_wheels="${rear_wheels}"
+        hardware_plugin="${hardware_plugin}"
+      />
+    </xacro:if>
     <link name="imu_0_link">
       <inertial>

File: clearpath_platform_description/urdf/r100/r100.urdf.xacro (robot description, xacro)
@@ -104,5 +104,5 @@
           <mesh filename="package://clearpath_platform_description/meshes/r100/end-cover.stl" />
         </geometry>
-        <material name="clearpath_red" />
+        <material name="clearpath_black" />
       </visual>
     </link>
@@ -133,5 +133,5 @@
           <mesh filename="package://clearpath_platform_description/meshes/r100/lights.stl" />
         </geometry>
-        <material name="clearpath_black" />
+        <material name="clearpath_red" />
       </visual>
     </link>
