Commit message: Rebase from 'upstream'

File: clearpath_platform_description/urdf/common.urdf.xacro (robot description, xacro)
@@ -36,4 +36,5 @@
       <color rgba="0.1 0.1 0.1   1"/>
     </material>
+    <xacro:property name="guard_include_zed" value="true" lazy_eval="true"/>
     <!--
         Standard Mount: adds link (w/o geometry) at given position

File: clearpath_sensors_description/urdf/stereolabs_zed.urdf.xacro (robot description, xacro)
@@ -1,5 +1,8 @@
 <?xml version="1.0"?>
 <robot xmlns:xacro="http://www.ros.org/wiki/xacro">
-  <xacro:include filename="$(find zed_wrapper)/urdf/zed_macro.urdf.xacro" />
+  <xacro:if value="${guard_include_zed}">
+    <xacro:property name="guard_include_zed" value="false" lazy_eval="false"/>
+    <xacro:include filename="$(find zed_wrapper)/urdf/zed_macro.urdf.xacro"/>
+  </xacro:if>
   <xacro:macro name="stereolabs_zed" params="
     name
