Commit message: Imported upstream version '1.3.5' of 'upstream'

File: clearpath_manipulators_description/urdf/lift/ewellix.urdf.xacro (robot description, xacro)
@@ -16,5 +16,5 @@
     generate_ros2_control_tag:=''
     use_fake_hardware:=''
-    sim_gazebo:=''
+    sim_ignition:=''
     port=''
     baud=''
@@ -32,5 +32,5 @@
     <!-- Default Simulation Parameters -->
     <xacro:property name="_use_fake_hardware" value="false" />
-    <xacro:property name="_sim_gazebo" value="$(arg is_sim)" />
+    <xacro:property name="_sim_ignition" value="$(arg is_sim)" />
     <!-- Default Hardware Parameters -->
     <xacro:property name="_port" value="/dev/ttyUSB0"/>
@@ -47,5 +47,5 @@
     <xacro:if value="${generate_ros2_control_tag != ''}"> <xacro:property name="_generate_ros2_control_tag" value="${generate_ros2_control_tag}" lazy_eval="false"/> </xacro:if>
     <xacro:if value="${use_fake_hardware != ''}"> <xacro:property name="_use_fake_hardware" value="${use_fake_hardware}" lazy_eval="false"/> </xacro:if>
-    <xacro:if value="${sim_gazebo != ''}"> <xacro:property name="_sim_gazebo" value="${sim_gazebo}" lazy_eval="false"/> </xacro:if>
+    <xacro:if value="${sim_ignition != ''}"> <xacro:property name="_sim_ignition" value="${sim_ignition}" lazy_eval="false"/> </xacro:if>
     <xacro:if value="${port != ''}"> <xacro:property name="_port" value="${port}" lazy_eval="false"/> </xacro:if>
     <xacro:if value="${baud != ''}"> <xacro:property name="_baud" value="${baud}" lazy_eval="false"/> </xacro:if>
@@ -63,5 +63,5 @@
       generate_ros2_control_tag="${_generate_ros2_control_tag}"
       use_fake_hardware="${_use_fake_hardware}"
-      sim_gazebo="${_sim_gazebo}"
+      sim_ignition="${_sim_ignition}"
       port="${_port}"
       baud="${_baud}"

File: clearpath_platform_description/urdf/do100/do100.urdf.xacro (robot description, xacro)
@@ -63,5 +63,5 @@
     </xacro:do100_wheel>
     <gazebo>
-      <plugin filename="libgz-sim-wheel-slip-system.so" name="gz::sim::systems::WheelSlip">
+      <plugin filename="libignition-gazebo-wheel-slip-system.so" name="ignition::gazebo::systems::WheelSlip">
         <wheel link_name="front_left_wheel_link">
           <slip_compliance_lateral>1.0</slip_compliance_lateral>
@@ -107,5 +107,5 @@
         <update_rate>50</update_rate>
         <visualize>true</visualize>
-        <gz_frame_id>imu_0_link</gz_frame_id>
+        <ignition_frame_id>imu_0_link</ignition_frame_id>
       </sensor>
     </gazebo>
@@ -204,6 +204,6 @@
   <!-- Joint State Publisher -->
   <plugin
-    filename="gz-sim-joint-state-publisher-system"
-    name="gz::sim::systems::JointStatePublisher"
+    filename="ignition-gazebo-joint-state-publisher-system"
+    name="ignition::gazebo::systems::JointStatePublisher"
   />
 </robot>

File: clearpath_platform_description/urdf/r100/r100.urdf.xacro (robot description, xacro)
@@ -19,5 +19,5 @@
     <xacro:property name="deck_height" value="0.280" />
     <xacro:property name="deck_thickness" value="0.005" />
-    <xacro:property name="riser_height" value="0.070" />
+    <xacro:property name="riser_height" value="0.055" />
     <xacro:property name="axle_offset" value="0.0500" />
     <xacro:property name="rocker_offset" value="0.319" />
@@ -111,5 +111,5 @@
           <mesh filename="package://clearpath_platform_description/meshes/r100/end-cover.stl" />
         </geometry>
-        <material name="clearpath_red" />
+        <material name="clearpath_black" />
       </visual>
     </link>
@@ -140,5 +140,5 @@
           <mesh filename="package://clearpath_platform_description/meshes/r100/lights.stl" />
         </geometry>
-        <material name="clearpath_black" />
+        <material name="clearpath_red" />
       </visual>
     </link>
@@ -208,5 +208,5 @@
     </xacro:r100_rocker>
     <gazebo>
-      <plugin filename="libgz-sim-wheel-slip-system.so" name="gz::sim::systems::WheelSlip">
+      <plugin filename="libignition-gazebo-wheel-slip-system.so" name="ignition::gazebo::systems::WheelSlip">
         <wheel link_name="front_left_wheel_link">
           <slip_compliance_lateral>1.0</slip_compliance_lateral>
@@ -253,5 +253,5 @@
         <update_rate>50</update_rate>
         <visualize>true</visualize>
-        <gz_frame_id>imu_0_link</gz_frame_id>
+        <ignition_frame_id>imu_0_link</ignition_frame_id>
       </sensor>
     </gazebo>

Commit message: Imported upstream version '1.3.7' of 'upstream'

File: clearpath_manipulators_description/urdf/lift/ewellix.urdf.xacro (robot description, xacro)
@@ -11,4 +11,5 @@
     ewellix_type:=tlt_x25
     add_plate:=True
+    add_mount:=True
     parameters_file:=''
     initial_positions:=''
@@ -16,5 +17,5 @@
     generate_ros2_control_tag:=''
     use_fake_hardware:=''
-    sim_gazebo:=''
+    sim_ignition:=''
     port=''
     baud=''
@@ -32,5 +33,5 @@
     <!-- Default Simulation Parameters -->
     <xacro:property name="_use_fake_hardware" value="false" />
-    <xacro:property name="_sim_gazebo" value="$(arg is_sim)" />
+    <xacro:property name="_sim_ignition" value="$(arg is_sim)" />
     <!-- Default Hardware Parameters -->
     <xacro:property name="_port" value="/dev/ttyUSB0"/>
@@ -47,5 +48,5 @@
     <xacro:if value="${generate_ros2_control_tag != ''}"> <xacro:property name="_generate_ros2_control_tag" value="${generate_ros2_control_tag}" lazy_eval="false"/> </xacro:if>
     <xacro:if value="${use_fake_hardware != ''}"> <xacro:property name="_use_fake_hardware" value="${use_fake_hardware}" lazy_eval="false"/> </xacro:if>
-    <xacro:if value="${sim_gazebo != ''}"> <xacro:property name="_sim_gazebo" value="${sim_gazebo}" lazy_eval="false"/> </xacro:if>
+    <xacro:if value="${sim_ignition != ''}"> <xacro:property name="_sim_ignition" value="${sim_ignition}" lazy_eval="false"/> </xacro:if>
     <xacro:if value="${port != ''}"> <xacro:property name="_port" value="${port}" lazy_eval="false"/> </xacro:if>
     <xacro:if value="${baud != ''}"> <xacro:property name="_baud" value="${baud}" lazy_eval="false"/> </xacro:if>
@@ -59,9 +60,10 @@
       tf_prefix="${_tf_prefix}"
       add_plate="${add_plate}"
+      add_mount="${add_mount}"
       initial_positions="${_initial_positions}"
       parameters_file="${_parameters_file}"
       generate_ros2_control_tag="${_generate_ros2_control_tag}"
       use_fake_hardware="${_use_fake_hardware}"
-      sim_gazebo="${_sim_gazebo}"
+      sim_ignition="${_sim_ignition}"
       port="${_port}"
       baud="${_baud}"

Commit message: Rebase from 'upstream'

File: clearpath_manipulators_description/urdf/lift/ewellix.urdf.xacro (robot description, xacro)
@@ -11,4 +11,5 @@
     ewellix_type:=tlt_x25
     add_plate:=True
+    add_mount:=True
     parameters_file:=''
     initial_positions:=''
@@ -59,4 +60,5 @@
       tf_prefix="${_tf_prefix}"
       add_plate="${add_plate}"
+      add_mount="${add_mount}"
       initial_positions="${_initial_positions}"
       parameters_file="${_parameters_file}"

File: clearpath_sensors_description/urdf/ouster_os1.urdf.xacro (robot description, xacro)
@@ -19,4 +19,5 @@
     parent_link
     cap:=halo
+    base:=base
     *origin
     samples_h:=1024 min_ang_h:=${-pi} max_ang_h:=${pi}
@@ -28,7 +29,14 @@
     <xacro:property name="lidar_height" value="0.05835"/>
     <xacro:property name="lidar_diameter" value="0.087"/>
-    <xacro:property name="base_mass" value="0."/>
-    <xacro:property name="base_height" value="0.0225"/>
-    <xacro:property name="base_length" value="0.110"/>
+    <xacro:if value="${base == 'base'}">
+      <xacro:property name="base_mass" value="0.0"/>
+      <xacro:property name="base_height" value="0.0225"/>
+      <xacro:property name="base_length" value="0.110"/>
+    </xacro:if>
+    <xacro:unless value="${base == 'base'}">
+      <xacro:property name="base_mass" value="0.0"/>
+      <xacro:property name="base_height" value="0.0"/>
+      <xacro:property name="base_length" value="0.0"/>
+    </xacro:unless>
     <xacro:property name="fins_mass" value="0.079"/>
     <xacro:property name="fins_height" value="0.022"/>
@@ -38,31 +46,36 @@
     <xacro:property name="halo_diameter" value="0.08679"/>
     <!-- Base Link -->
-    <link name="${name}_base_link">
-      <inertial>
-        <mass value="${base_mass}"/>
-        <origin xyz="0 0 ${base_height/2}"/>
-        <xacro:ouster_box_inertia
-          mass="${base_mass}"
-          x="${base_length}"
-          y="${base_length}"
-          z="${base_height}"
-        />
-      </inertial>
-      <visual>
-        <material name="ouster_grey">
-          <color rgba="0.8 0.8 0.8 1.0"/>
-        </material>
-        <origin xyz="0 0 ${base_height}"/>
-        <geometry>
-          <mesh filename="package://clearpath_sensors_description/meshes/ouster/os1_base.dae"/>
-        </geometry>
-      </visual>
-      <collision>
-        <origin xyz="0 0 ${base_height/2}"/>
-        <geometry>
-          <box size="${base_length} ${base_length} ${base_height}"/>
-        </geometry>
-      </collision>
-    </link>
+    <xacro:if value="${base == 'base'}">
+      <link name="${name}_base_link">
+        <inertial>
+          <mass value="${base_mass}"/>
+          <origin xyz="0 0 ${base_height/2}"/>
+          <xacro:ouster_box_inertia
+            mass="${base_mass}"
+            x="${base_length}"
+            y="${base_length}"
+            z="${base_height}"
+          />
+        </inertial>
+        <visual>
+          <material name="ouster_grey">
+            <color rgba="0.8 0.8 0.8 1.0"/>
+          </material>
+          <origin xyz="0 0 ${base_height}"/>
+          <geometry>
+            <mesh filename="package://clearpath_sensors_description/meshes/ouster/os1_base.dae"/>
+          </geometry>
+        </visual>
+        <collision>
+          <origin xyz="0 0 ${base_height/2}"/>
+          <geometry>
+            <box size="${base_length} ${base_length} ${base_height}"/>
+          </geometry>
+        </collision>
+      </link>
+    </xacro:if>
+    <xacro:unless value="${base == 'base'}">
+      <link name="${name}_base_link" />
+    </xacro:unless>
     <!-- Lidar Link -->
     <link name="${name}_link">

Commit message: Imported upstream version '2.7.4' of 'upstream'

File: clearpath_manipulators_description/urdf/lift/ewellix.urdf.xacro (robot description, xacro)
@@ -11,5 +11,4 @@
     ewellix_type:=tlt_x25
     add_plate:=True
-    add_mount:=True
     parameters_file:=''
     initial_positions:=''
@@ -17,5 +16,5 @@
     generate_ros2_control_tag:=''
     use_fake_hardware:=''
-    sim_ignition:=''
+    sim_gazebo:=''
     port=''
     baud=''
@@ -33,5 +32,5 @@
     <!-- Default Simulation Parameters -->
     <xacro:property name="_use_fake_hardware" value="false" />
-    <xacro:property name="_sim_ignition" value="$(arg is_sim)" />
+    <xacro:property name="_sim_gazebo" value="$(arg is_sim)" />
     <!-- Default Hardware Parameters -->
     <xacro:property name="_port" value="/dev/ttyUSB0"/>
@@ -48,5 +47,5 @@
     <xacro:if value="${generate_ros2_control_tag != ''}"> <xacro:property name="_generate_ros2_control_tag" value="${generate_ros2_control_tag}" lazy_eval="false"/> </xacro:if>
     <xacro:if value="${use_fake_hardware != ''}"> <xacro:property name="_use_fake_hardware" value="${use_fake_hardware}" lazy_eval="false"/> </xacro:if>
-    <xacro:if value="${sim_ignition != ''}"> <xacro:property name="_sim_ignition" value="${sim_ignition}" lazy_eval="false"/> </xacro:if>
+    <xacro:if value="${sim_gazebo != ''}"> <xacro:property name="_sim_gazebo" value="${sim_gazebo}" lazy_eval="false"/> </xacro:if>
     <xacro:if value="${port != ''}"> <xacro:property name="_port" value="${port}" lazy_eval="false"/> </xacro:if>
     <xacro:if value="${baud != ''}"> <xacro:property name="_baud" value="${baud}" lazy_eval="false"/> </xacro:if>
@@ -60,10 +59,9 @@
       tf_prefix="${_tf_prefix}"
       add_plate="${add_plate}"
-      add_mount="${add_mount}"
       initial_positions="${_initial_positions}"
       parameters_file="${_parameters_file}"
       generate_ros2_control_tag="${_generate_ros2_control_tag}"
       use_fake_hardware="${_use_fake_hardware}"
-      sim_ignition="${_sim_ignition}"
+      sim_gazebo="${_sim_gazebo}"
       port="${_port}"
       baud="${_baud}"

File: clearpath_sensors_description/urdf/ouster_os1.urdf.xacro (robot description, xacro)
@@ -73,9 +73,9 @@
           </geometry>
         </collision>
-      </link>
-    </xacro:if>
-    <xacro:unless value="${base == 'base'}">
-      <link name="${name}_base_link" />
-    </xacro:unless>
+    </link>
+  </xacro:if>
+  <xacro:unless value="${base == 'base'}">
+    <link name="${name}_base_link" />
+  </xacro:unless>
     <!-- Lidar Link -->
     <link name="${name}_link">

Commit message: Rebase from 'upstream'

File: clearpath_manipulators_description/urdf/lift/ewellix.urdf.xacro (robot description, xacro)
@@ -10,5 +10,6 @@
     *origin
     ewellix_type:=tlt_x25
-    add_plate:=True
+    add_plate:=''
+    add_mount:=''
     parameters_file:=''
     initial_positions:=''
@@ -34,4 +35,6 @@
     <xacro:property name="_sim_gazebo" value="$(arg is_sim)" />
     <!-- Default Hardware Parameters -->
+    <xacro:property name="_add_plate" value="True"/>
+    <xacro:property name="_add_mount" value="True"/>
     <xacro:property name="_port" value="/dev/ttyUSB0"/>
     <xacro:property name="_baud" value="38400"/>
@@ -48,4 +51,6 @@
     <xacro:if value="${use_fake_hardware != ''}"> <xacro:property name="_use_fake_hardware" value="${use_fake_hardware}" lazy_eval="false"/> </xacro:if>
     <xacro:if value="${sim_gazebo != ''}"> <xacro:property name="_sim_gazebo" value="${sim_gazebo}" lazy_eval="false"/> </xacro:if>
+    <xacro:if value="${add_plate != ''}"> <xacro:property name="_add_plate" value="${add_plate}" lazy_eval="false"/> </xacro:if>
+    <xacro:if value="${add_mount != ''}"> <xacro:property name="_add_mount" value="${add_mount}" lazy_eval="false"/> </xacro:if>
     <xacro:if value="${port != ''}"> <xacro:property name="_port" value="${port}" lazy_eval="false"/> </xacro:if>
     <xacro:if value="${baud != ''}"> <xacro:property name="_baud" value="${baud}" lazy_eval="false"/> </xacro:if>
@@ -58,5 +63,6 @@
       parent="${parent_link}"
       tf_prefix="${_tf_prefix}"
-      add_plate="${add_plate}"
+      add_plate="${_add_plate}"
+      add_mount="${_add_mount}"
       initial_positions="${_initial_positions}"
       parameters_file="${_parameters_file}"
