Commit message: Rebase from 'upstream'

File: clearpath_platform_description/urdf/dd100/drivetrain/wheels.urdf.xacro (robot description, xacro)
@@ -1,4 +1,4 @@
 <?xml version="1.0"?>
-<robot xmlns:xacro="http://ros.org/wiki/xacro" xmlns:ignition="http://gazebosim.org/schema" name="dd100_drivetrain_wheels">
+<robot xmlns:xacro="http://ros.org/wiki/xacro" xmlns:gz="http://gazebosim.org/schema" name="dd100_drivetrain_wheels">
   <xacro:macro name="dd100_drivetrain_wheels" params="front_wheels rear_wheels">
     <xacro:include filename="$(find clearpath_platform_description)/urdf/dd100/drivetrain/wheels/indoor.urdf.xacro"/>

File: clearpath_platform_description/urdf/dd100/drivetrain/wheels/caster.urdf.xacro (robot description, xacro)
@@ -1,4 +1,4 @@
 <?xml version="1.0"?>
-<robot xmlns:xacro="http://ros.org/wiki/xacro" xmlns:ignition="http://gazebosim.org/schema" name="dd100_caster_wheel">
+<robot xmlns:xacro="http://ros.org/wiki/xacro" xmlns:gz="http://gazebosim.org/schema" name="dd100_caster_wheel">
   <xacro:property name="dd100_caster_wheel_radius" value="0.01" />
   <xacro:property name="dd100_caster_wheel_mass" value="0.1" />

File: clearpath_platform_description/urdf/do100/do100.urdf.xacro (robot description, xacro)
@@ -83,4 +83,5 @@
         <visualize>true</visualize>
         <gz_frame_id>imu_0_link</gz_frame_id>
+        <topic>$(arg namespace)/sensors/imu_0/data_raw</topic>
       </sensor>
     </gazebo>

File: clearpath_platform_description/urdf/do100/drivetrain/wheels.urdf.xacro (robot description, xacro)
@@ -1,4 +1,4 @@
 <?xml version="1.0"?>
-<robot xmlns:xacro="http://ros.org/wiki/xacro" xmlns:ignition="http://gazebosim.org/schema" name="do100_drivetrain_wheels">
+<robot xmlns:xacro="http://ros.org/wiki/xacro" xmlns:gz="http://gazebosim.org/schema" name="do100_drivetrain_wheels">
   <xacro:macro name="do100_drivetrain_wheels" params="front_wheels rear_wheels">
     <xacro:include filename="$(find clearpath_platform_description)/urdf/do100/drivetrain/wheels/mecanum.urdf.xacro"/>

File: clearpath_platform_description/urdf/do100/drivetrain/wheels/mecanum.urdf.xacro (robot description, xacro)
@@ -1,4 +1,4 @@
 <?xml version="1.0"?>
-<robot xmlns:xacro="http://ros.org/wiki/xacro" xmlns:ignition="http://gazebosim.org/schema" name="do100_mecanum_wheel">
+<robot xmlns:xacro="http://ros.org/wiki/xacro" xmlns:gz="http://gazebosim.org/schema" name="do100_mecanum_wheel">
   <xacro:property name="do100_mecanum_wheel_radius" value="0.050" />
   <xacro:property name="do100_mecanum_wheel_mass" value="0.4" />
@@ -44,5 +44,5 @@
               <mu>1.0</mu>
               <mu2>0.0</mu2>
-              <fdir1 ignition:expressed_in="base_link">1 ${side} 0</fdir1>
+              <fdir1 gz:expressed_in="base_link">1 ${side} 0</fdir1>
             </ode>
           </friction>

File: clearpath_platform_description/urdf/do150/do150.urdf.xacro (robot description, xacro)
@@ -83,4 +83,5 @@
         <visualize>true</visualize>
         <gz_frame_id>imu_0_link</gz_frame_id>
+        <topic>$(arg namespace)/sensors/imu_0/data_raw</topic>
       </sensor>
     </gazebo>

File: clearpath_platform_description/urdf/generic/drivetrain/control/diff_4wd.urdf.xacro (robot description, xacro)
@@ -1,4 +1,4 @@
 <?xml version="1.0"?>
-<robot xmlns:xacro="http://ros.org/wiki/xacro" xmlns:ignition="http://gazebosim.org/schema" name="generic_drivetrain_control_diff_4wd">
+<robot xmlns:xacro="http://ros.org/wiki/xacro" xmlns:gz="http://gazebosim.org/schema" name="generic_drivetrain_control_diff_4wd">
   <xacro:macro name="generic_drivetrain_control_diff_4wd" params="name hardware_plugin">
     <!-- This is the same as omni_4wd -->

File: clearpath_platform_description/urdf/generic/drivetrain/control/diff_fwd.urdf.xacro (robot description, xacro)
@@ -1,4 +1,4 @@
 <?xml version="1.0"?>
-<robot xmlns:xacro="http://ros.org/wiki/xacro" xmlns:ignition="http://gazebosim.org/schema" name="generic_drivetrain_control_diff_fwd">
+<robot xmlns:xacro="http://ros.org/wiki/xacro" xmlns:gz="http://gazebosim.org/schema" name="generic_drivetrain_control_diff_fwd">
   <xacro:macro name="generic_drivetrain_control_diff_fwd" params="name hardware_plugin">
     <!-- Gazebo Controller -->

File: clearpath_platform_description/urdf/generic/drivetrain/control/diff_rwd.urdf.xacro (robot description, xacro)
@@ -1,4 +1,4 @@
 <?xml version="1.0"?>
-<robot xmlns:xacro="http://ros.org/wiki/xacro" xmlns:ignition="http://gazebosim.org/schema" name="generic_drivetrain_control_diff_rwd">
+<robot xmlns:xacro="http://ros.org/wiki/xacro" xmlns:gz="http://gazebosim.org/schema" name="generic_drivetrain_control_diff_rwd">
   <xacro:macro name="generic_drivetrain_control_diff_rwd" params="name hardware_plugin">
     <!-- Gazebo Controller -->

File: clearpath_platform_description/urdf/generic/drivetrain/control/omni_4wd.urdf.xacro (robot description, xacro)
@@ -1,4 +1,4 @@
 <?xml version="1.0"?>
-<robot xmlns:xacro="http://ros.org/wiki/xacro" xmlns:ignition="http://gazebosim.org/schema" name="generic_drivetrain_control_omni_4wd">
+<robot xmlns:xacro="http://ros.org/wiki/xacro" xmlns:gz="http://gazebosim.org/schema" name="generic_drivetrain_control_omni_4wd">
   <xacro:macro name="generic_drivetrain_control_omni_4wd" params="name hardware_plugin">
     <!-- Gazebo Controller -->

File: clearpath_platform_description/urdf/generic/drivetrain/drivetrain.urdf.xacro (robot description, xacro)
@@ -1,4 +1,4 @@
 <?xml version="1.0"?>
-<robot xmlns:xacro="http://ros.org/wiki/xacro" xmlns:ignition="http://gazebosim.org/schema" name="generic_drivetrain">
+<robot xmlns:xacro="http://ros.org/wiki/xacro" xmlns:gz="http://gazebosim.org/schema" name="generic_drivetrain">
   <xacro:macro name="generic_drivetrain" params="name control front_wheels rear_wheels hardware_plugin">
     <!-- Omni drivetrain -->

File: clearpath_platform_description/urdf/r100/drivetrain/wheels.urdf.xacro (robot description, xacro)
@@ -1,4 +1,4 @@
 <?xml version="1.0"?>
-<robot xmlns:xacro="http://ros.org/wiki/xacro" xmlns:ignition="http://gazebosim.org/schema" name="r100_drivetrain_wheels">
+<robot xmlns:xacro="http://ros.org/wiki/xacro" xmlns:gz="http://gazebosim.org/schema" name="r100_drivetrain_wheels">
   <!-- Includes -->
   <xacro:include filename="$(find clearpath_platform_description)/urdf/r100/rocker.urdf.xacro"/>

File: clearpath_platform_description/urdf/r100/drivetrain/wheels/mecanum.urdf.xacro (robot description, xacro)
@@ -1,4 +1,4 @@
 <?xml version="1.0"?>
-<robot xmlns:xacro="http://ros.org/wiki/xacro" xmlns:ignition="http://gazebosim.org/schema" name="r100_wheel">
+<robot xmlns:xacro="http://ros.org/wiki/xacro" xmlns:gz="http://gazebosim.org/schema" name="r100_wheel">
   <xacro:property name="r100_mecanum_wheel_radius" value="0.0759" />
   <xacro:property name="r100_mecanum_wheel_mass" value="2.5" />
@@ -45,5 +45,5 @@
               <mu>1.0</mu>
               <mu2>0.0</mu2>
-              <fdir1 ignition:expressed_in="base_link">1 ${side} 0</fdir1>
+              <fdir1 gz:expressed_in="base_link">1 ${side} 0</fdir1>
             </ode>
           </friction>

File: clearpath_platform_description/urdf/r100/r100.urdf.xacro (robot description, xacro)
@@ -234,4 +234,5 @@
         <visualize>true</visualize>
         <gz_frame_id>imu_0_link</gz_frame_id>
+        <topic>$(arg namespace)/sensors/imu_0/data_raw</topic>
       </sensor>
     </gazebo>

File: clearpath_sensors_description/urdf/ouster_os1.urdf.xacro (robot description, xacro)
@@ -186,5 +186,5 @@
     <xacro:if value="${cap == 'fins' or cap == 'halo'}">
       <!-- Thermal Cap Joint -->
-      <joint name="{name}_cap_joint" type="fixed">
+      <joint name="${name}_cap_joint" type="fixed">
         <child link="${name}_cap_link"/>
         <parent link="${name}_link"/>
