Commit message: Rebase from 'upstream'

File: clearpath_manipulators_description/urdf/gripper/kinova_2f_lite.urdf.xacro (robot description, xacro)
@@ -79,5 +79,5 @@
       <child link="${name}_right_finger_prox_link" />
       <axis xyz="0 0 -1" />
-      <limit lower="0.0" upper="0.85" effort="1000" velocity="0.6" />
+      <limit lower="-0.1" upper="0.96" effort="10" velocity="0.6" />
     </joint>
     <!-- Right Finger Dist -->
@@ -146,5 +146,5 @@
       <child link="${name}_left_finger_prox_link" />
       <axis xyz="0 0 1" />
-      <limit lower="0.0" upper="0.85" effort="1000" velocity="1000" />
+      <limit lower="-0.1" upper="0.96" effort="10" velocity="0.6" />
       <mimic joint="${name}_right_finger_bottom_joint" multiplier="1.0" offset="0.0" />
     </joint>
