Commit message: Imported upstream version '1.3.11' of 'upstream'

File: clearpath_manipulators_description/urdf/gripper/robotiq_2f_140.urdf.xacro (robot description, xacro)
@@ -294,5 +294,5 @@
           </xacro:if>
           <xacro:if value="${sim_gazebo}">
-            <plugin>gz_ros2_control/GazeboSimSystem</plugin>
+            <plugin>ign_ros2_control/IgnitionSystem</plugin>
           </xacro:if>
           <xacro:if value="${use_fake_hardware}">

File: clearpath_platform_description/urdf/a200/a200.urdf.xacro (robot description, xacro)
@@ -6,6 +6,8 @@
   <xacro:arg name="gazebo_controllers" default="$(find clearpath_control)/config/a200/control.yaml"/>
   <xacro:arg name="use_platform_controllers" default="true"/>
+  <!-- Included URDF/XACRO Files -->
+  <xacro:include filename="$(find clearpath_platform_description)/urdf/a200/wheels/wheel.urdf.xacro" />
   <xacro:property name="M_PI" value="3.14159"/>
-  <xacro:macro name="a200" params="control:='diff_4wd' front_wheels:='outdoor' rear_wheels:='outdoor'">
+  <xacro:macro name="a200" params="wheel:='default'">
     <!-- Base Size -->
     <xacro:property name="base_x_size" value="0.98740000" />
@@ -13,7 +15,10 @@
     <xacro:property name="base_z_size" value="0.24750000" />
     <!-- Wheel Mounting Positions -->
-    <xacro:property name="wheel_base" value="0.5120" />
-    <xacro:property name="wheel_track" value="0.555" />
+    <xacro:property name="wheelbase" value="0.5120" />
+    <xacro:property name="track" value="0.555" />
     <xacro:property name="wheel_vertical_offset" value="0.03282" />
+    <!-- Wheel Properties -->
+    <xacro:property name="wheel_length" value="0.1143" />
+    <xacro:property name="wheel_radius" value="0.1651" />
     <!-- Base link is the center of the robot's bottom plate -->
     <link name="base_link">
@@ -37,4 +42,11 @@
       </collision>
     </link>
+    <!-- Base footprint is on the ground under the robot -->
+    <link name="base_footprint"/>
+    <joint name="base_footprint_joint" type="fixed">
+      <origin xyz="0 0 ${wheel_vertical_offset - wheel_radius}" rpy="0 0 0" />
+      <parent link="base_link" />
+      <child link="base_footprint" />
+    </joint>
     <!-- Spawn A200 chassis -->
     <link name="top_chassis_link">
@@ -64,7 +76,66 @@
       <child link="inertial_link" />
     </joint>
-    <!-- Add wheels -->
-    <xacro:include filename="$(find clearpath_platform_description)/urdf/a200/drivetrain/wheels.urdf.xacro"/>
-    <xacro:a200_drivetrain_wheels front_wheels="${front_wheels}" rear_wheels="${rear_wheels}"/>
+    <!-- A200 wheel macros -->
+    <xacro:a200_wheel wheel_prefix="front_left">
+      <origin xyz="${wheelbase/2} ${track/2} ${wheel_vertical_offset}" rpy="0 0 0" />
+    </xacro:a200_wheel>
+    <xacro:a200_wheel wheel_prefix="front_right">
+      <origin xyz="${wheelbase/2} ${-track/2} ${wheel_vertical_offset}" rpy="0 0 0" />
+    </xacro:a200_wheel>
+    <xacro:a200_wheel wheel_prefix="rear_left">
+      <origin xyz="${-wheelbase/2} ${track/2} ${wheel_vertical_offset}" rpy="0 0 0" />
+    </xacro:a200_wheel>
+    <xacro:a200_wheel wheel_prefix="rear_right">
+      <origin xyz="${-wheelbase/2} ${-track/2} ${wheel_vertical_offset}" rpy="0 0 0" />
+    </xacro:a200_wheel>
+    <gazebo>
+      <plugin filename="libignition-gazebo-wheel-slip-system.so" name="ignition::gazebo::systems::WheelSlip">
+        <wheel link_name="front_left_wheel">
+          <slip_compliance_lateral>1.0</slip_compliance_lateral>
+          <slip_compliance_longitudinal>1.0</slip_compliance_longitudinal>
+          <wheel_normal_force>113</wheel_normal_force>
+          <wheel_radius>${wheel_radius}</wheel_radius>
+        </wheel>
+        <wheel link_name="front_right_wheel">
+          <slip_compliance_lateral>1.0</slip_compliance_lateral>
+          <slip_compliance_longitudinal>1.0</slip_compliance_longitudinal>
+          <wheel_normal_force>113</wheel_normal_force>
+          <wheel_radius>${wheel_radius}</wheel_radius>
+        </wheel>
+        <wheel link_name="rear_left_wheel">
+          <slip_compliance_lateral>1.0</slip_compliance_lateral>
+          <slip_compliance_longitudinal>1.0</slip_compliance_longitudinal>
+          <wheel_normal_force>113</wheel_normal_force>
+          <wheel_radius>${wheel_radius}</wheel_radius>
+        </wheel>
+        <wheel link_name="rear_right_wheel">
+          <slip_compliance_lateral>1.0</slip_compliance_lateral>
+          <slip_compliance_longitudinal>1.0</slip_compliance_longitudinal>
+          <wheel_normal_force>113</wheel_normal_force>
+          <wheel_radius>${wheel_radius}</wheel_radius>
+        </wheel>
+      </plugin>
+    </gazebo>
+    <!-- Front bumper mount -->
+    <link name="front_bumper_mount"/>
+    <joint name="front_bumper_mount_joint" type="fixed">
+      <origin xyz="0.406 0 0.091" rpy="0 0 0" />
+      <parent link="base_link" />
+      <child link="front_bumper_mount" />
+    </joint>
+    <!-- Rear bumper mount -->
+    <link name="rear_bumper_mount"/>
+    <joint name="rear_bumper_mount_joint" type="fixed">
+      <origin xyz="-0.406 0 0.091" rpy="0 0 ${M_PI}" />
+      <parent link="base_link" />
+      <child link="rear_bumper_mount" />
+    </joint>
+    <!-- Default mount -->
+    <link name="default_mount"/>
+    <joint name="default_mount_joint" type="fixed">
+      <child link="default_mount"/>
+      <parent link="base_link"/>
+      <origin xyz="0.0 0.0 0.224"/>
+    </joint>
     <!-- Gazebo Controller -->
     <xacro:include filename="$(find clearpath_platform_description)/urdf/generic/gazebo.urdf.xacro"/>
@@ -74,9 +145,9 @@
         <hardware>
           <xacro:if value="$(arg is_sim)">
-            <plugin>gz_ros2_control/GazeboSimSystem</plugin>
+            <plugin>ign_ros2_control/IgnitionSystem</plugin>
           </xacro:if>
           <xacro:unless value="$(arg is_sim)">
             <plugin>clearpath_hardware_interfaces/A200Hardware</plugin>
-            <param name="wheel_diameter">${front_wheel_radius * 2}</param>
+            <param name="wheel_diameter">0.3302</param>
             <param name="max_accel">5.0</param>
             <param name="max_speed">1.0</param>
@@ -119,32 +190,4 @@
       </ros2_control>
     </xacro:if>
-    <!-- Front bumper mount -->
-    <link name="front_bumper_mount"/>
-    <joint name="front_bumper_mount_joint" type="fixed">
-      <origin xyz="0.406 0 0.091" rpy="0 0 0" />
-      <parent link="base_link" />
-      <child link="front_bumper_mount" />
-    </joint>
-    <!-- Rear bumper mount -->
-    <link name="rear_bumper_mount"/>
-    <joint name="rear_bumper_mount_joint" type="fixed">
-      <origin xyz="-0.406 0 0.091" rpy="0 0 ${M_PI}" />
-      <parent link="base_link" />
-      <child link="rear_bumper_mount" />
-    </joint>
-    <!-- Default mount -->
-    <link name="default_mount"/>
-    <joint name="default_mount_joint" type="fixed">
-      <child link="default_mount"/>
-      <parent link="base_link"/>
-      <origin xyz="0.0 0.0 0.224"/>
-    </joint>
-    <!-- Base footprint is on the ground under the robot -->
-    <link name="base_footprint"/>
-    <joint name="base_footprint_joint" type="fixed">
-      <origin xyz="0 0 ${wheel_vertical_offset - front_wheel_radius}" rpy="0 0 0" />
-      <parent link="base_link" />
-      <child link="base_footprint" />
-    </joint>
   </xacro:macro>
 </robot>

File: clearpath_platform_description/urdf/j100/j100.urdf.xacro (robot description, xacro)
@@ -2,4 +2,5 @@
 <robot name="j100"
   xmlns:xacro="http://www.ros.org/wiki/xacro">
+  <xacro:include filename="$(find clearpath_platform_description)/urdf/j100/wheels/wheel.urdf.xacro"/>
   <xacro:arg name="is_sim" default="false" />
   <xacro:arg name="prefix" default="" />
@@ -12,4 +13,6 @@
   <xacro:property name="wheel_vertical_offset" value="0.0345" />
   <xacro:property name="footprint_vertical_offset" value="-0.0655" />
+  <xacro:property name="wheel_radius" value="0.098" />
+  <xacro:property name="wheel_width" value="0.040" />
   <xacro:property name="chassis_length" value="0.420" />
   <xacro:property name="chassis_width" value="0.310" />
@@ -17,5 +20,45 @@
   <xacro:property name="dummy_inertia" value="1e-09"/>
   <xacro:property name="mount_spacing" value="0.120" />
-  <xacro:macro name="j100" params="control:='diff_4wd' front_wheels:='outdoor' rear_wheels:='outdoor'">
+  <xacro:macro name="j100" params="wheel:='default'">
+    <xacro:j100_wheel prefix="front_left">
+      <origin xyz="${wheelbase/2} ${track/2} ${wheel_vertical_offset}" rpy="0 0 0" />
+    </xacro:j100_wheel>
+    <xacro:j100_wheel prefix="front_right">
+      <origin xyz="${wheelbase/2} ${-track/2} ${wheel_vertical_offset}" rpy="0 0 0" />
+    </xacro:j100_wheel>
+    <xacro:j100_wheel prefix="rear_left">
+      <origin xyz="${-wheelbase/2} ${track/2} ${wheel_vertical_offset}" rpy="0 0 0" />
+    </xacro:j100_wheel>
+    <xacro:j100_wheel prefix="rear_right">
+      <origin xyz="${-wheelbase/2} ${-track/2} ${wheel_vertical_offset}" rpy="0 0 0" />
+    </xacro:j100_wheel>
+    <gazebo>
+      <plugin filename="libignition-gazebo-wheel-slip-system.so" name="ignition::gazebo::systems::WheelSlip">
+        <wheel link_name="front_left_wheel_link">
+          <slip_compliance_lateral>1.0</slip_compliance_lateral>
+          <slip_compliance_longitudinal>1.0</slip_compliance_longitudinal>
+          <wheel_normal_force>40</wheel_normal_force>
+          <wheel_radius>${wheel_radius}</wheel_radius>
+        </wheel>
+        <wheel link_name="front_right_wheel_link">
+          <slip_compliance_lateral>1.0</slip_compliance_lateral>
+          <slip_compliance_longitudinal>1.0</slip_compliance_longitudinal>
+          <wheel_normal_force>40</wheel_normal_force>
+          <wheel_radius>${wheel_radius}</wheel_radius>
+        </wheel>
+        <wheel link_name="rear_left_wheel_link">
+          <slip_compliance_lateral>1.0</slip_compliance_lateral>
+          <slip_compliance_longitudinal>1.0</slip_compliance_longitudinal>
+          <wheel_normal_force>40</wheel_normal_force>
+          <wheel_radius>${wheel_radius}</wheel_radius>
+        </wheel>
+        <wheel link_name="rear_right_wheel_link">
+          <slip_compliance_lateral>1.0</slip_compliance_lateral>
+          <slip_compliance_longitudinal>1.0</slip_compliance_longitudinal>
+          <wheel_normal_force>40</wheel_normal_force>
+          <wheel_radius>${wheel_radius}</wheel_radius>
+        </wheel>
+      </plugin>
+    </gazebo>
     <link name="base_link"></link>
     <joint name="base_link_joint" type="fixed">
@@ -44,25 +87,4 @@
       </inertial>
     </link>
-    <!-- Add wheels -->
-    <xacro:include filename="$(find clearpath_platform_description)/urdf/j100/drivetrain/wheels.urdf.xacro"/>
-    <xacro:j100_drivetrain_wheels front_wheels="${front_wheels}" rear_wheels="${rear_wheels}"/>
-    <!-- Add drivetrain -->
-    <xacro:include filename="$(find clearpath_platform_description)/urdf/generic/drivetrain/drivetrain.urdf.xacro"/>
-    <!-- Hardware  -->
-    <xacro:if value="$(arg is_sim)">
-      <xacro:property name="hardware_plugin" value="gz_ros2_control/GazeboSimSystem"/>
-    </xacro:if>
-    <xacro:unless value="$(arg is_sim)">
-      <xacro:property name="hardware_plugin" value="clearpath_hardware_interfaces/J100Hardware"/>
-    </xacro:unless>
-    <xacro:if value="$(arg use_platform_controllers)">
-      <xacro:generic_drivetrain
-        name="j100"
-        control="${control}"
-        front_wheels="${front_wheels}"
-        rear_wheels="${rear_wheels}"
-        hardware_plugin="${hardware_plugin}"
-      />
-    </xacro:if>
     <link name="imu_0_link">
       <inertial>
@@ -81,5 +103,5 @@
         <update_rate>50</update_rate>
         <visualize>true</visualize>
-        <gz_frame_id>imu_0_link</gz_frame_id>
+        <ignition_frame_id>imu_0_link</ignition_frame_id>
         <topic>$(arg namespace)/sensors/imu_0/data_raw</topic>
       </sensor>
@@ -103,5 +125,5 @@
         <always_on>1</always_on>
         <update_rate>10</update_rate>
-        <gz_frame_id>gps_0_link</gz_frame_id>
+        <ignition_frame_id>gps_0_link</ignition_frame_id>
         <topic>$(arg namespace)/sensors/gps_0/navsat</topic>
       </sensor>
@@ -125,4 +147,39 @@
       <origin xyz="${mount_spacing} 0 0" />
     </joint>
+    <!-- Gazebo Controller -->
+    <xacro:include filename="$(find clearpath_platform_description)/urdf/generic/gazebo.urdf.xacro"/>
+    <!-- ROS2 controls -->
+    <xacro:if value="$(arg use_platform_controllers)">
+      <ros2_control name="j100_hardware" type="system">
+        <hardware>
+          <xacro:if value="$(arg is_sim)">
+            <plugin>ign_ros2_control/IgnitionSystem</plugin>
+          </xacro:if>
+          <xacro:unless value="$(arg is_sim)">
+            <plugin>clearpath_hardware_interfaces/J100Hardware</plugin>
+          </xacro:unless>
+        </hardware>
+        <joint name="front_left_wheel_joint">
+          <command_interface name="velocity"/>
+          <state_interface name="position"/>
+          <state_interface name="velocity"/>
+        </joint>
+        <joint name="rear_left_wheel_joint">
+          <command_interface name="velocity"/>
+          <state_interface name="position"/>
+          <state_interface name="velocity"/>
+        </joint>
+        <joint name="front_right_wheel_joint">
+          <command_interface name="velocity"/>
+          <state_interface name="position"/>
+          <state_interface name="velocity"/>
+        </joint>
+        <joint name="rear_right_wheel_joint">
+          <command_interface name="velocity"/>
+          <state_interface name="position"/>
+          <state_interface name="velocity"/>
+        </joint>
+      </ros2_control>
+    </xacro:if>
   </xacro:macro>
 </robot>

File: clearpath_platform_description/urdf/r100/r100.urdf.xacro (robot description, xacro)
@@ -3,9 +3,15 @@
   <xacro:arg name="namespace" default="" />
   <xacro:arg name="is_sim" default="false" />
-  <xacro:arg name="gazebo_controllers" default="$(find clearpath_control)/config/r100/control/omni_4wd.yaml"/>
+  <xacro:arg name="gazebo_controllers" default="$(find clearpath_control)/config/r100/control.yaml"/>
   <xacro:arg name="use_platform_controllers" default="true"/>
+  <!-- Includes -->
+  <xacro:include filename="$(find clearpath_platform_description)/urdf/r100/wheels/wheel.urdf.xacro"/>
+  <xacro:include filename="$(find clearpath_platform_description)/urdf/r100/rocker.urdf.xacro"/>
   <!-- R100 Platform Macro -->
-  <xacro:macro name="r100" params="control:='omni_4wd' front_wheels:='mecanum' rear_wheels:='mecanum'">
+  <xacro:macro name="r100" params="wheel:='defaut'">
     <!-- Variables -->
+    <xacro:property name="wheel_radius" value="0.0759" />
+    <xacro:property name="wheel_width" value="0.0790" />
+    <xacro:property name="wheel_mass" value="2.5" />
     <xacro:property name="chassis_length" value="0.960" />
     <xacro:property name="chassis_width" value="0.793" />
@@ -13,5 +19,5 @@
     <xacro:property name="deck_height" value="0.280" />
     <xacro:property name="deck_thickness" value="0.005" />
-    <xacro:property name="riser_height" value="0.070" />
+    <xacro:property name="riser_height" value="0.055" />
     <xacro:property name="axle_offset" value="0.0500" />
     <xacro:property name="rocker_offset" value="0.319" />
@@ -194,28 +200,39 @@
       </collision>
     </link>
-    <!-- Add wheels -->
-    <xacro:include filename="$(find clearpath_platform_description)/urdf/r100/drivetrain/wheels.urdf.xacro"/>
-    <xacro:r100_drivetrain_wheels front_wheels="${front_wheels}" rear_wheels="${rear_wheels}"/>
-    <!-- Add drivetrain -->
-    <xacro:include filename="$(find clearpath_platform_description)/urdf/generic/drivetrain/drivetrain.urdf.xacro"/>
-    <!-- Hardware  -->
-    <xacro:if value="$(arg is_sim)">
-      <xacro:property name="hardware_plugin" value="gz_ros2_control/GazeboSimSystem"/>
-    </xacro:if>
-    <xacro:unless value="$(arg is_sim)">
-      <xacro:property name="hardware_plugin" value="clearpath_hardware_interfaces/PumaHardware"/>
-    </xacro:unless>
-    <xacro:unless value="${control == 'omni_4wd' or control == 'diff_4wd'}">
-      <xacro:error message="Invalid drivetrain control ${control}"/>
-    </xacro:unless>
-    <xacro:if value="$(arg use_platform_controllers)">
-      <xacro:generic_drivetrain
-        name="r100"
-        control="${control}"
-        front_wheels="${front_wheels}"
-        rear_wheels="${rear_wheels}"
-        hardware_plugin="${hardware_plugin}"
-      />
-    </xacro:if>
+    <!-- Rocker -->
+    <xacro:r100_rocker prefix="front" joint_type="fixed" location="1" >
+      <limit lower="-0.08726" upper="0.08726" effort="0" velocity="0" />
+    </xacro:r100_rocker>
+    <xacro:r100_rocker prefix="rear" joint_type="fixed" location="-1" >
+      <limit effort="0" velocity="0" />
+    </xacro:r100_rocker>
+    <gazebo>
+      <plugin filename="libignition-gazebo-wheel-slip-system.so" name="ignition::gazebo::systems::WheelSlip">
+        <wheel link_name="front_left_wheel_link">
+          <slip_compliance_lateral>1.0</slip_compliance_lateral>
+          <slip_compliance_longitudinal>1.0</slip_compliance_longitudinal>
+          <wheel_normal_force>200</wheel_normal_force>
+          <wheel_radius>${wheel_radius}</wheel_radius>
+        </wheel>
+        <wheel link_name="front_right_wheel_link">
+          <slip_compliance_lateral>1.0</slip_compliance_lateral>
+          <slip_compliance_longitudinal>1.0</slip_compliance_longitudinal>
+          <wheel_normal_force>200</wheel_normal_force>
+          <wheel_radius>${wheel_radius}</wheel_radius>
+        </wheel>
+        <wheel link_name="rear_left_wheel_link">
+          <slip_compliance_lateral>1.0</slip_compliance_lateral>
+          <slip_compliance_longitudinal>1.0</slip_compliance_longitudinal>
+          <wheel_normal_force>200</wheel_normal_force>
+          <wheel_radius>${wheel_radius}</wheel_radius>
+        </wheel>
+        <wheel link_name="rear_right_wheel_link">
+          <slip_compliance_lateral>1.0</slip_compliance_lateral>
+          <slip_compliance_longitudinal>1.0</slip_compliance_longitudinal>
+          <wheel_normal_force>200</wheel_normal_force>
+          <wheel_radius>${wheel_radius}</wheel_radius>
+        </wheel>
+      </plugin>
+    </gazebo>
     <!-- Internal IMU -->
     <link name="imu_0_link">
@@ -236,6 +253,5 @@
         <update_rate>50</update_rate>
         <visualize>true</visualize>
-        <gz_frame_id>imu_0_link</gz_frame_id>
-        <topic>$(arg namespace)/sensors/imu_0/data_raw</topic>
+        <ignition_frame_id>imu_0_link</ignition_frame_id>
       </sensor>
     </gazebo>
@@ -247,4 +263,39 @@
       <origin xyz="0 0 ${riser_height + deck_thickness}" rpy="0 0 0"/>
     </joint>
+    <!-- Gazebo Controller -->
+    <xacro:include filename="$(find clearpath_platform_description)/urdf/generic/gazebo.urdf.xacro"/>
+    <!-- ROS2 controls -->
+    <xacro:if value="$(arg use_platform_controllers)">
+      <ros2_control name="r100_hardware" type="system">
+        <hardware>
+          <xacro:if value="$(arg is_sim)">
+            <plugin>ign_ros2_control/IgnitionSystem</plugin>
+          </xacro:if>
+          <xacro:unless value="$(arg is_sim)">
+            <plugin>clearpath_hardware_interfaces/PumaHardware</plugin>
+          </xacro:unless>
+        </hardware>
+        <joint name="front_left_wheel_joint">
+          <command_interface name="velocity"/>
+          <state_interface name="position"/>
+          <state_interface name="velocity"/>
+        </joint>
+        <joint name="front_right_wheel_joint">
+          <command_interface name="velocity"/>
+          <state_interface name="position"/>
+          <state_interface name="velocity"/>
+        </joint>
+        <joint name="rear_left_wheel_joint">
+          <command_interface name="velocity"/>
+          <state_interface name="position"/>
+          <state_interface name="velocity"/>
+        </joint>
+        <joint name="rear_right_wheel_joint">
+          <command_interface name="velocity"/>
+          <state_interface name="position"/>
+          <state_interface name="velocity"/>
+        </joint>
+      </ros2_control>
+    </xacro:if>
   </xacro:macro>
 </robot>
