Commit message: Imported upstream version '1.3.11' of 'upstream'

File: clearpath_platform_description/urdf/w200/w200.urdf.xacro (robot description, xacro)
@@ -6,7 +6,9 @@
   <xacro:arg name="use_platform_controllers" default="true"/>
   <!-- Include URDF/XACRO Files -->
+  <xacro:include filename="$(find clearpath_platform_description)/urdf/w200/wheels/track.urdf.xacro"/>
+  <xacro:include filename="$(find clearpath_platform_description)/urdf/w200/wheels/wheel.urdf.xacro"/>
   <xacro:property name="PI" value="3.1415926535897931"/>
   <xacro:include filename="$(find clearpath_platform_description)/urdf/w200/diff_unit.urdf.xacro"/>
-  <xacro:macro name="w200" params="control:='diff_4wd' front_wheels:='outdoor' rear_wheels:='outdoor' color:='yellow'">
+  <xacro:macro name="w200" params="wheel:='default' color:='yellow'">
     <!-- Colors: yellow, orange, olive, sand -->
     <xacro:property name="warthog_color"  value="${'warthog_'+color}"/>
@@ -102,7 +104,34 @@
       <origin xyz="-0.5826 0 0.24979" rpy="0 0 0" />
     </joint>
-    <!-- Add wheels -->
-    <xacro:include filename="$(find clearpath_platform_description)/urdf/w200/drivetrain/wheels.urdf.xacro"/>
-    <xacro:w200_drivetrain_wheels front_wheels="${front_wheels}" rear_wheels="${rear_wheels}"/>
+    <!-- Wheels -->
+    <xacro:if value="${wheel == 'default'}">
+      <xacro:w200_wheel prefix="front" side="left">
+        <origin xyz="${axle_x_offset*1} ${axle_y_offset*1} ${axle_z_offset}" rpy="0 0 0" />
+      </xacro:w200_wheel>
+      <xacro:w200_wheel prefix="front" side="right">
+        <origin xyz="${axle_x_offset*1} ${axle_y_offset*-1} ${axle_z_offset}" rpy="0 0 0" />
+      </xacro:w200_wheel>
+      <xacro:w200_wheel prefix="rear" side="left">
+        <origin xyz="${axle_x_offset*-1} ${axle_y_offset*1} ${axle_z_offset}" rpy="0 0 0" />
+      </xacro:w200_wheel>
+      <xacro:w200_wheel prefix="rear" side="right">
+        <origin xyz="${axle_x_offset*-1} ${axle_y_offset*-1} ${axle_z_offset}" rpy="0 0 0" />
+      </xacro:w200_wheel>
+    </xacro:if>
+    <!-- Tracks -->
+    <xacro:if value="${wheel == 'track'}">
+      <xacro:w200_track prefix="front" side="left">
+        <origin xyz="${axle_x_offset*1} ${axle_y_offset*1} ${axle_z_offset}" rpy="0 0 0" />
+      </xacro:w200_track>
+      <xacro:w200_track prefix="front" side="right">
+        <origin xyz="${axle_x_offset*1} ${axle_y_offset*-1} ${axle_z_offset}" rpy="0 0 0" />
+      </xacro:w200_track>
+      <xacro:w200_track prefix="rear" side="left">
+        <origin xyz="${axle_x_offset*-1} ${axle_y_offset*1} ${axle_z_offset}" rpy="0 0 ${PI}" />
+      </xacro:w200_track>
+      <xacro:w200_track prefix="rear" side="right">
+        <origin xyz="${axle_x_offset*-1} ${axle_y_offset*-1} ${axle_z_offset}" rpy="0 0 ${PI}" />
+      </xacro:w200_track>
+    </xacro:if>
     <!-- Virtual Mounting Point -->
     <link name="default_mount"></link>
@@ -129,5 +158,5 @@
         <update_rate>50</update_rate>
         <visualize>true</visualize>
-        <gz_frame_id>imu_0_link</gz_frame_id>
+        <ignition_frame_id>imu_0_link</ignition_frame_id>
         <topic>$(arg namespace)/sensors/imu_0/data_raw</topic>
       </sensor>
@@ -140,5 +169,5 @@
         <hardware>
           <xacro:if value="$(arg is_sim)">
-            <plugin>gz_ros2_control/GazeboSimSystem</plugin>
+            <plugin>ign_ros2_control/IgnitionSystem</plugin>
           </xacro:if>
           <xacro:unless value="$(arg is_sim)">
@@ -181,4 +210,34 @@
       </ros2_control>
     </xacro:if>
+    <xacro:if value="$(arg is_sim)">
+      <gazebo>
+        <plugin filename="libignition-gazebo-wheel-slip-system.so" name="ignition::gazebo::systems::WheelSlip">
+          <wheel link_name="front_left_wheel_link">
+            <slip_compliance_lateral>1.0</slip_compliance_lateral>
+            <slip_compliance_longitudinal>1.0</slip_compliance_longitudinal>
+            <wheel_normal_force>686</wheel_normal_force>
+            <wheel_radius>${wheel_radius}</wheel_radius>
+          </wheel>
+          <wheel link_name="front_right_wheel_link">
+            <slip_compliance_lateral>1.0</slip_compliance_lateral>
+            <slip_compliance_longitudinal>1.0</slip_compliance_longitudinal>
+            <wheel_normal_force>686</wheel_normal_force>
+            <wheel_radius>${wheel_radius}</wheel_radius>
+          </wheel>
+          <wheel link_name="rear_left_wheel_link">
+            <slip_compliance_lateral>1.0</slip_compliance_lateral>
+            <slip_compliance_longitudinal>1.0</slip_compliance_longitudinal>
+            <wheel_normal_force>686</wheel_normal_force>
+            <wheel_radius>${wheel_radius}</wheel_radius>
+          </wheel>
+          <wheel link_name="rear_right_wheel_link">
+            <slip_compliance_lateral>1.0</slip_compliance_lateral>
+            <slip_compliance_longitudinal>1.0</slip_compliance_longitudinal>
+            <wheel_normal_force>686</wheel_normal_force>
+            <wheel_radius>${wheel_radius}</wheel_radius>
+          </wheel>
+        </plugin>
+      </gazebo>
+    </xacro:if>
   </xacro:macro>
 </robot>

File: clearpath_sensors_description/urdf/stereolabs_zed.urdf.xacro (robot description, xacro)
@@ -1,8 +1,5 @@
 <?xml version="1.0"?>
 <robot xmlns:xacro="http://www.ros.org/wiki/xacro">
-  <xacro:if value="${guard_include_zed}">
-    <xacro:property name="guard_include_zed" value="false" lazy_eval="false"/>
-    <xacro:include filename="$(find zed_description)/urdf/zed_macro.urdf.xacro"/>
-  </xacro:if>
+  <xacro:include filename="$(find zed_description)/urdf/zed_macro.urdf.xacro" />
   <xacro:macro name="stereolabs_zed" params="
     name
@@ -48,5 +45,5 @@
             <far>100</far>
           </clip>
-          <gz_frame_id>${name}_link</gz_frame_id>
+          <ignition_frame_id>${name}_link</ignition_frame_id>
           <optical_frame_id>${name}_left_camera_optical_frame</optical_frame_id>
         </camera>
@@ -54,5 +51,5 @@
         <update_rate>${update_rate}</update_rate>
         <visualize>true</visualize>
-        <gz_frame_id>${name}_link</gz_frame_id>
+        <ignition_frame_id>${name}_link</ignition_frame_id>
         <topic>$(arg namespace)/sensors/${name}</topic>
       </sensor>

Commit message: Rebase from 'upstream'

File: clearpath_manipulators_description/urdf/gripper/robotiq_2f_140.urdf.xacro (robot description, xacro)
@@ -16,8 +16,15 @@
     isaac_joint_commands:=/isaac_joint_commands
     isaac_joint_states:=/isaac_joint_states
-    com_port:=/dev/ttyUSB0">
+    com_port:=/dev/ttyUSB0
+    padding:=true">
     <!-- Variables Mappings -->
     <xacro:property name="prefix" value="${name}_"/>
     <xacro:property name="stroke" value="140"/>
+    <xacro:if value="${padding}">
+      <xacro:property name="upper_finger_joint_limit" value="0.7"/>
+    </xacro:if>
+    <xacro:unless value="${padding}">
+      <xacro:property name="upper_finger_joint_limit" value="0.767"/>
+    </xacro:unless>
     <!-- this is a temporary link to rotate the 2f-140 gripper to match the 2f-85 -->
     <link name="${prefix}robotiq_base_link"/>
@@ -204,5 +211,5 @@
         <child link="${prefix}left_outer_knuckle" />
         <axis xyz="-1 0 0" />
-        <limit lower="0" upper="0.7" velocity="2.0" effort="1000" />
+        <limit lower="0" upper="${upper_finger_joint_limit}" velocity="2.0" effort="1000" />
       </joint>
       <xacro:finger_joints prefix="${prefix}" fingerprefix="left" reflect="1.0"/>
@@ -214,5 +221,5 @@
         <child link="${prefix}right_outer_knuckle" />
         <axis xyz="1 0 0" />
-        <limit lower="-0.725" upper="0.725" velocity="2.0" effort="1000" />
+        <limit lower="-0.775" upper="0.775" velocity="2.0" effort="1000" />
         <mimic joint="${prefix}finger_joint" multiplier="-1" offset="0" />
       </joint>
@@ -259,5 +266,7 @@
       <xacro:inner_knuckle_joint prefix="${prefix}" fingerprefix="${fingerprefix}" reflect="${reflect}"/>
       <xacro:inner_finger_joint prefix="${prefix}" fingerprefix="${fingerprefix}"/>
-      <xacro:inner_finger_pad_joint prefix="${prefix}" fingerprefix="${fingerprefix}"/>
+      <xacro:if value="${padding}">
+        <xacro:inner_finger_pad_joint prefix="${prefix}" fingerprefix="${fingerprefix}"/>
+      </xacro:if>
     </xacro:macro>
     <xacro:macro name="finger_links" params="prefix fingerprefix stroke">
@@ -265,5 +274,7 @@
       <xacro:outer_finger prefix="${prefix}" fingerprefix="${fingerprefix}" stroke="${stroke}"/>
       <xacro:inner_finger prefix="${prefix}" fingerprefix="${fingerprefix}" stroke="${stroke}"/>
-      <xacro:inner_finger_pad prefix="${prefix}" fingerprefix="${fingerprefix}"/>
+      <xacro:if value="${padding}">
+        <xacro:inner_finger_pad prefix="${prefix}" fingerprefix="${fingerprefix}"/>
+      </xacro:if>
       <xacro:inner_knuckle prefix="${prefix}" fingerprefix="${fingerprefix}" stroke="${stroke}"/>
     </xacro:macro>

File: clearpath_sensors_description/urdf/stereolabs_zed.urdf.xacro (robot description, xacro)
@@ -1,5 +1,5 @@
 <?xml version="1.0"?>
 <robot xmlns:xacro="http://www.ros.org/wiki/xacro">
-  <xacro:include filename="$(find zed_wrapper)/urdf/zed_macro.urdf.xacro" />
+  <xacro:include filename="$(find zed_description)/urdf/zed_macro.urdf.xacro" />
   <xacro:macro name="stereolabs_zed" params="
     name
