Commit message: Rebase from 'upstream'

File: clearpath_platform_description/urdf/a200/drivetrain/wheels.urdf.xacro (robot description, xacro)
@@ -4,4 +4,5 @@
     <xacro:include filename="$(find clearpath_platform_description)/urdf/a200/drivetrain/wheels/outdoor.urdf.xacro" />
     <xacro:include filename="$(find clearpath_platform_description)/urdf/a200/drivetrain/wheels/indoor.urdf.xacro" />
+    <xacro:property name="a200_wheel_vertical_offset" value="0.03282" />
     <!-- Front Wheels -->
     <!-- Outdoor -->
@@ -11,9 +12,9 @@
       <!-- Wheel -->
       <xacro:a200_outdoor_wheel prefix="front_left">
-        <origin xyz="${wheel_base/2} ${wheel_track/2} 0" rpy="0 0 0"/>
+        <origin xyz="${wheel_base/2} ${wheel_track/2} ${a200_wheel_vertical_offset}" rpy="0 0 0"/>
       </xacro:a200_outdoor_wheel>
       <!-- Wheel -->
       <xacro:a200_outdoor_wheel prefix="front_right">
-        <origin xyz="${wheel_base/2} ${-wheel_track/2} 0" rpy="0 0 0"/>
+        <origin xyz="${wheel_base/2} ${-wheel_track/2} ${a200_wheel_vertical_offset}" rpy="0 0 0"/>
       </xacro:a200_outdoor_wheel>
     </xacro:if>
@@ -24,9 +25,9 @@
       <!-- Wheel -->
       <xacro:a200_indoor_wheel prefix="front_left">
-        <origin xyz="${wheel_base/2} ${wheel_track/2} 0" rpy="0 0 0"/>
+        <origin xyz="${wheel_base/2} ${wheel_track/2} ${a200_wheel_vertical_offset}" rpy="0 0 0"/>
       </xacro:a200_indoor_wheel>
       <!-- Wheel -->
       <xacro:a200_indoor_wheel prefix="front_right">
-        <origin xyz="${wheel_base/2} ${-wheel_track/2} 0" rpy="0 0 0"/>
+        <origin xyz="${wheel_base/2} ${-wheel_track/2} ${a200_wheel_vertical_offset}" rpy="0 0 0"/>
       </xacro:a200_indoor_wheel>
     </xacro:if>
@@ -38,9 +39,9 @@
       <!-- Wheel -->
       <xacro:a200_outdoor_wheel prefix="rear_left">
-        <origin xyz="${-wheel_base/2} ${wheel_track/2} 0" rpy="0 0 0"/>
+        <origin xyz="${-wheel_base/2} ${wheel_track/2} ${a200_wheel_vertical_offset}" rpy="0 0 0"/>
       </xacro:a200_outdoor_wheel>
       <!-- Wheel -->
       <xacro:a200_outdoor_wheel prefix="rear_right">
-        <origin xyz="${-wheel_base/2} ${-wheel_track/2} 0" rpy="0 0 0"/>
+        <origin xyz="${-wheel_base/2} ${-wheel_track/2} ${a200_wheel_vertical_offset}" rpy="0 0 0"/>
       </xacro:a200_outdoor_wheel>
     </xacro:if>
@@ -51,9 +52,9 @@
       <!-- Wheel -->
       <xacro:a200_indoor_wheel prefix="rear_left">
-        <origin xyz="${-wheel_base/2} ${wheel_track/2} 0" rpy="0 0 0"/>
+        <origin xyz="${-wheel_base/2} ${wheel_track/2} ${a200_wheel_vertical_offset}" rpy="0 0 0"/>
       </xacro:a200_indoor_wheel>
       <!-- Wheel -->
       <xacro:a200_indoor_wheel prefix="rear_right">
-        <origin xyz="${-wheel_base/2} ${-wheel_track/2} 0" rpy="0 0 0"/>
+        <origin xyz="${-wheel_base/2} ${-wheel_track/2} ${a200_wheel_vertical_offset}" rpy="0 0 0"/>
       </xacro:a200_indoor_wheel>
     </xacro:if>
