Commit message: Rebase from 'release/humble/clearpath_manipulators_description'

File: urdf/gripper/robotiq_2f_140.urdf.xacro (robot description, xacro)
@@ -36,5 +36,5 @@
         <origin xyz="0 0 0" rpy="0 0 0" />
         <geometry>
-          <mesh filename="file://$(find clearpath_manipulators_description)/meshes/gripper/robotiq_2f_140_base_link.stl" />
+          <mesh filename="package://clearpath_manipulators_description/meshes/gripper/robotiq_2f_140_base_link.stl" />
         </geometry>
         <material name="">
@@ -45,5 +45,5 @@
         <origin xyz="0 0 0" rpy="0 0 0" />
         <geometry>
-          <mesh filename="file://$(find clearpath_manipulators_description)/meshes/gripper/robotiq_2f_140_base_link_collision.stl" />
+          <mesh filename="package://clearpath_manipulators_description/meshes/gripper/robotiq_2f_140_base_link_collision.stl" />
         </geometry>
       </collision>
@@ -71,5 +71,5 @@
           <origin xyz="0 0 0" rpy="0 0 0" />
           <geometry>
-            <mesh filename="file://$(find clearpath_manipulators_description)/meshes/gripper/robotiq_2f_${stroke}_outer_knuckle.stl" />
+            <mesh filename="package://clearpath_manipulators_description/meshes/gripper/robotiq_2f_${stroke}_outer_knuckle.stl" />
           </geometry>
           <material name="">
@@ -80,5 +80,5 @@
           <origin xyz="0 0 0" rpy="0 0 0" />
           <geometry>
-            <mesh filename="file://$(find clearpath_manipulators_description)/meshes/gripper/robotiq_2f_${stroke}_outer_knuckle_collision.stl" />
+            <mesh filename="package://clearpath_manipulators_description/meshes/gripper/robotiq_2f_${stroke}_outer_knuckle_collision.stl" />
           </geometry>
         </collision>
@@ -101,5 +101,5 @@
           <origin xyz="0 0 0" rpy="0 0 0" />
           <geometry>
-            <mesh filename="file://$(find clearpath_manipulators_description)/meshes/gripper/robotiq_2f_${stroke}_outer_finger.stl" />
+            <mesh filename="package://clearpath_manipulators_description/meshes/gripper/robotiq_2f_${stroke}_outer_finger.stl" />
           </geometry>
           <material name="">
@@ -110,5 +110,5 @@
           <origin xyz="0 0 0" rpy="0 0 0" />
           <geometry>
-            <mesh filename="file://$(find clearpath_manipulators_description)/meshes/gripper/robotiq_2f_${stroke}_outer_finger_collision.stl" />
+            <mesh filename="package://clearpath_manipulators_description/meshes/gripper/robotiq_2f_${stroke}_outer_finger_collision.stl" />
           </geometry>
         </collision>
@@ -131,5 +131,5 @@
           <origin xyz="0 0 0" rpy="0 0 0" />
           <geometry>
-            <mesh filename="file://$(find clearpath_manipulators_description)/meshes/gripper/robotiq_2f_${stroke}_inner_knuckle.stl" />
+            <mesh filename="package://clearpath_manipulators_description/meshes/gripper/robotiq_2f_${stroke}_inner_knuckle.stl" />
           </geometry>
           <material name="">
@@ -140,5 +140,5 @@
           <origin xyz="0 0 0" rpy="0 0 0" />
           <geometry>
-            <mesh filename="file://$(find clearpath_manipulators_description)/meshes/gripper/robotiq_2f_${stroke}_inner_knuckle_collision.stl" />
+            <mesh filename="package://clearpath_manipulators_description/meshes/gripper/robotiq_2f_${stroke}_inner_knuckle_collision.stl" />
           </geometry>
         </collision>
@@ -161,5 +161,5 @@
           <origin xyz="0 0 0" rpy="0 0 0" />
           <geometry>
-            <mesh filename="file://$(find clearpath_manipulators_description)/meshes/gripper/robotiq_2f_${stroke}_inner_finger.stl" />
+            <mesh filename="package://clearpath_manipulators_description/meshes/gripper/robotiq_2f_${stroke}_inner_finger.stl" />
           </geometry>
           <material name="">
@@ -170,5 +170,5 @@
           <origin xyz="0 0 0" rpy="0 0 0" />
           <geometry>
-            <mesh filename="file://$(find clearpath_manipulators_description)/meshes/gripper/robotiq_2f_${stroke}_inner_finger_collision.stl" />
+            <mesh filename="package://clearpath_manipulators_description/meshes/gripper/robotiq_2f_${stroke}_inner_finger_collision.stl" />
           </geometry>
         </collision>
