Commit message: Imported upstream version '1.3.10' of 'upstream'

File: clearpath_manipulators_description/srdf/gripper/robotiq_2f_140.srdf.xacro (robot description, xacro)
@@ -6,11 +6,5 @@
     </group_state>
   </xacro:macro>
-  <xacro:macro name="robotiq_2f_140" params="name padding:=true">
-    <xacro:if value="${padding}">
-      <xacro:property name="upper_finger_joint_limit" value="0.7"/>
-    </xacro:if>
-    <xacro:unless value="${padding}">
-      <xacro:property name="upper_finger_joint_limit" value="0.767"/>
-    </xacro:unless>
+  <xacro:macro name="robotiq_2f_140" params="name">
     <group name="${name}">
         <joint name="${name}_finger_joint"/>
@@ -29,5 +23,5 @@
       name="${name}"
       group_state="close"
-      joint_positions="${[upper_finger_joint_limit]}"
+      joint_positions="${[0.7]}"
     />
     <disable_collisions link1="${name}_left_inner_knuckle" link2="${name}_left_inner_finger" reason="User"/>
@@ -35,7 +29,4 @@
     <disable_collisions link1="${name}_left_outer_knuckle" link2="${name}_left_inner_knuckle" reason="User"/>
     <disable_collisions link1="${name}_right_outer_knuckle" link2="${name}_right_inner_knuckle" reason="User"/>
-    <xacro:if value="${padding}">
-      <disable_collisions link1="${name}_right_inner_finger_pad" link2="${name}_left_inner_finger_pad" reason="User"/>
-    </xacro:if>
   </xacro:macro>
 </robot>

File: clearpath_manipulators_description/urdf/gripper/robotiq_2f_140.urdf.xacro (robot description, xacro)
@@ -16,15 +16,8 @@
     isaac_joint_commands:=/isaac_joint_commands
     isaac_joint_states:=/isaac_joint_states
-    com_port:=/dev/ttyUSB0
-    padding:=true">
+    com_port:=/dev/ttyUSB0">
     <!-- Variables Mappings -->
     <xacro:property name="prefix" value="${name}_"/>
     <xacro:property name="stroke" value="140"/>
-    <xacro:if value="${padding}">
-      <xacro:property name="upper_finger_joint_limit" value="0.7"/>
-    </xacro:if>
-    <xacro:unless value="${padding}">
-      <xacro:property name="upper_finger_joint_limit" value="0.767"/>
-    </xacro:unless>
     <!-- this is a temporary link to rotate the 2f-140 gripper to match the 2f-85 -->
     <link name="${prefix}robotiq_base_link"/>
@@ -211,5 +204,5 @@
         <child link="${prefix}left_outer_knuckle" />
         <axis xyz="-1 0 0" />
-        <limit lower="0" upper="${upper_finger_joint_limit}" velocity="2.0" effort="1000" />
+        <limit lower="0" upper="0.7" velocity="2.0" effort="1000" />
       </joint>
       <xacro:finger_joints prefix="${prefix}" fingerprefix="left" reflect="1.0"/>
@@ -221,5 +214,5 @@
         <child link="${prefix}right_outer_knuckle" />
         <axis xyz="1 0 0" />
-        <limit lower="-0.775" upper="0.775" velocity="2.0" effort="1000" />
+        <limit lower="-0.725" upper="0.725" velocity="2.0" effort="1000" />
         <mimic joint="${prefix}finger_joint" multiplier="-1" offset="0" />
       </joint>
@@ -266,7 +259,5 @@
       <xacro:inner_knuckle_joint prefix="${prefix}" fingerprefix="${fingerprefix}" reflect="${reflect}"/>
       <xacro:inner_finger_joint prefix="${prefix}" fingerprefix="${fingerprefix}"/>
-      <xacro:if value="${padding}">
-        <xacro:inner_finger_pad_joint prefix="${prefix}" fingerprefix="${fingerprefix}"/>
-      </xacro:if>
+      <xacro:inner_finger_pad_joint prefix="${prefix}" fingerprefix="${fingerprefix}"/>
     </xacro:macro>
     <xacro:macro name="finger_links" params="prefix fingerprefix stroke">
@@ -274,7 +265,5 @@
       <xacro:outer_finger prefix="${prefix}" fingerprefix="${fingerprefix}" stroke="${stroke}"/>
       <xacro:inner_finger prefix="${prefix}" fingerprefix="${fingerprefix}" stroke="${stroke}"/>
-      <xacro:if value="${padding}">
-        <xacro:inner_finger_pad prefix="${prefix}" fingerprefix="${fingerprefix}"/>
-      </xacro:if>
+      <xacro:inner_finger_pad prefix="${prefix}" fingerprefix="${fingerprefix}"/>
       <xacro:inner_knuckle prefix="${prefix}" fingerprefix="${fingerprefix}" stroke="${stroke}"/>
     </xacro:macro>
@@ -294,5 +283,5 @@
           </xacro:if>
           <xacro:if value="${sim_gazebo}">
-            <plugin>gz_ros2_control/GazeboSimSystem</plugin>
+            <plugin>ign_ros2_control/IgnitionSystem</plugin>
           </xacro:if>
           <xacro:if value="${use_fake_hardware}">
