Commit message: Imported upstream version '2.9.6' of 'upstream'

File: clearpath_manipulators_description/urdf/gripper/robotiq_2f_140.urdf.xacro (robot description, xacro)
@@ -16,8 +16,15 @@
     isaac_joint_commands:=/isaac_joint_commands
     isaac_joint_states:=/isaac_joint_states
-    com_port:=/dev/ttyUSB0">
+    com_port:=/dev/ttyUSB0
+    padding:=true">
     <!-- Variables Mappings -->
     <xacro:property name="prefix" value="${name}_"/>
     <xacro:property name="stroke" value="140"/>
+    <xacro:if value="${padding}">
+      <xacro:property name="upper_finger_joint_limit" value="0.7"/>
+    </xacro:if>
+    <xacro:unless value="${padding}">
+      <xacro:property name="upper_finger_joint_limit" value="0.767"/>
+    </xacro:unless>
     <!-- this is a temporary link to rotate the 2f-140 gripper to match the 2f-85 -->
     <link name="${prefix}robotiq_base_link"/>
@@ -204,5 +211,5 @@
         <child link="${prefix}left_outer_knuckle" />
         <axis xyz="-1 0 0" />
-        <limit lower="0" upper="0.7" velocity="2.0" effort="1000" />
+        <limit lower="0" upper="${upper_finger_joint_limit}" velocity="2.0" effort="1000" />
       </joint>
       <xacro:finger_joints prefix="${prefix}" fingerprefix="left" reflect="1.0"/>
@@ -214,5 +221,5 @@
         <child link="${prefix}right_outer_knuckle" />
         <axis xyz="1 0 0" />
-        <limit lower="-0.725" upper="0.725" velocity="2.0" effort="1000" />
+        <limit lower="-0.775" upper="0.775" velocity="2.0" effort="1000" />
         <mimic joint="${prefix}finger_joint" multiplier="-1" offset="0" />
       </joint>
@@ -259,5 +266,7 @@
       <xacro:inner_knuckle_joint prefix="${prefix}" fingerprefix="${fingerprefix}" reflect="${reflect}"/>
       <xacro:inner_finger_joint prefix="${prefix}" fingerprefix="${fingerprefix}"/>
-      <xacro:inner_finger_pad_joint prefix="${prefix}" fingerprefix="${fingerprefix}"/>
+      <xacro:if value="${padding}">
+        <xacro:inner_finger_pad_joint prefix="${prefix}" fingerprefix="${fingerprefix}"/>
+      </xacro:if>
     </xacro:macro>
     <xacro:macro name="finger_links" params="prefix fingerprefix stroke">
@@ -265,5 +274,7 @@
       <xacro:outer_finger prefix="${prefix}" fingerprefix="${fingerprefix}" stroke="${stroke}"/>
       <xacro:inner_finger prefix="${prefix}" fingerprefix="${fingerprefix}" stroke="${stroke}"/>
-      <xacro:inner_finger_pad prefix="${prefix}" fingerprefix="${fingerprefix}"/>
+      <xacro:if value="${padding}">
+        <xacro:inner_finger_pad prefix="${prefix}" fingerprefix="${fingerprefix}"/>
+      </xacro:if>
       <xacro:inner_knuckle prefix="${prefix}" fingerprefix="${fingerprefix}" stroke="${stroke}"/>
     </xacro:macro>
@@ -283,5 +294,5 @@
           </xacro:if>
           <xacro:if value="${sim_gazebo}">
-            <plugin>ign_ros2_control/IgnitionSystem</plugin>
+            <plugin>gz_ros2_control/GazeboSimSystem</plugin>
           </xacro:if>
           <xacro:if value="${use_fake_hardware}">
