Commit message: Rebase from 'upstream'

File: clearpath_platform_description/urdf/a200/a200.urdf.xacro (robot description, xacro)
@@ -7,5 +7,5 @@
   <xacro:arg name="use_platform_controllers" default="true"/>
   <xacro:property name="M_PI" value="3.14159"/>
-  <xacro:macro name="a200" params="control:='diff_fwd' front_wheels:='outdoor' rear_wheels:='outdoor'">
+  <xacro:macro name="a200" params="control:='diff_4wd' front_wheels:='outdoor' rear_wheels:='outdoor'">
     <!-- Base Size -->
     <xacro:property name="base_x_size" value="0.98740000" />

File: clearpath_platform_description/urdf/j100/j100.urdf.xacro (robot description, xacro)
@@ -17,5 +17,5 @@
   <xacro:property name="dummy_inertia" value="1e-09"/>
   <xacro:property name="mount_spacing" value="0.120" />
-  <xacro:macro name="j100" params="control:='diff_fwd' front_wheels:='outdoor' rear_wheels:='outdoor'">
+  <xacro:macro name="j100" params="control:='diff_4wd' front_wheels:='outdoor' rear_wheels:='outdoor'">
     <link name="base_link"></link>
     <joint name="base_link_joint" type="fixed">

File: clearpath_platform_description/urdf/w200/w200.urdf.xacro (robot description, xacro)
@@ -8,5 +8,5 @@
   <xacro:property name="PI" value="3.1415926535897931"/>
   <xacro:include filename="$(find clearpath_platform_description)/urdf/w200/diff_unit.urdf.xacro"/>
-  <xacro:macro name="w200" params="control:='diff_fwd' front_wheels:='outdoor' rear_wheels:='outdoor' color:='yellow'">
+  <xacro:macro name="w200" params="control:='diff_4wd' front_wheels:='outdoor' rear_wheels:='outdoor' color:='yellow'">
     <!-- Colors: yellow, orange, olive, sand -->
     <xacro:property name="warthog_color"  value="${'warthog_'+color}"/>

File: clearpath_sensors_description/urdf/stereolabs_zed.urdf.xacro (robot description, xacro)
@@ -3,5 +3,5 @@
   <xacro:if value="${guard_include_zed}">
     <xacro:property name="guard_include_zed" value="false" lazy_eval="false"/>
-    <xacro:include filename="$(find zed_wrapper)/urdf/zed_macro.urdf.xacro"/>
+    <xacro:include filename="$(find zed_description)/urdf/zed_macro.urdf.xacro"/>
   </xacro:if>
   <xacro:macro name="stereolabs_zed" params="
