Commit message: Rebase from 'upstream'

File: clearpath_platform_description/urdf/a300/drivetrain/wheels.urdf.xacro (robot description, xacro)
@@ -3,4 +3,5 @@
   <xacro:macro name="a300_drivetrain_wheels" params="front_wheels rear_wheels">
     <xacro:include filename="$(find clearpath_platform_description)/urdf/a300/drivetrain/wheels/outdoor.urdf.xacro" />
+    <xacro:include filename="$(find clearpath_platform_description)/urdf/a300/drivetrain/wheels/indoor.urdf.xacro" />
     <xacro:include filename="$(find clearpath_platform_description)/urdf/a300/drivetrain/wheels/mecanum.urdf.xacro" />
     <xacro:include filename="$(find clearpath_platform_description)/urdf/a300/drivetrain/wheels/caster.urdf.xacro" />
@@ -27,4 +28,14 @@
       <xacro:a300_mecanum_wheel prefix="front" side="left"/>
       <xacro:a300_mecanum_wheel prefix="front" side="right"/>
+    </xacro:if>
+    <xacro:if value="${front_wheels == 'indoor'}">
+      <xacro:property name="front_wheel_radius" value="${a300_indoor_wheel_radius}" scope="parent"/>
+      <xacro:property name="front_wheel_width" value="${a300_indoor_wheel_width}" scope="parent"/>
+      <!-- Motors -->
+      <xacro:a300_motor prefix="front" side="left"/>
+      <xacro:a300_motor prefix="front" side="right"/>
+      <!-- Wheels -->
+      <xacro:a300_indoor_wheel prefix="front" side="left"/>
+      <xacro:a300_indoor_wheel prefix="front" side="right"/>
     </xacro:if>
     <xacro:if value="${front_wheels == 'caster'}">
@@ -59,4 +70,14 @@
       <xacro:a300_mecanum_wheel prefix="rear" side="right"/>
     </xacro:if>
+    <xacro:if value="${rear_wheels == 'indoor'}">
+      <xacro:property name="rear_wheel_radius" value="${a300_indoor_wheel_radius}" scope="parent"/>
+      <xacro:property name="rear_wheel_width" value="${a300_indoor_wheel_width}" scope="parent"/>
+      <!-- Motors -->
+      <xacro:a300_motor prefix="rear" side="left"/>
+      <xacro:a300_motor prefix="rear" side="right"/>
+      <!-- Wheels -->
+      <xacro:a300_indoor_wheel prefix="rear" side="left"/>
+      <xacro:a300_indoor_wheel prefix="rear" side="right"/>
+    </xacro:if>
     <xacro:if value="${rear_wheels == 'caster'}">
       <xacro:property name="rear_wheel_radius" value="${a300_caster_wheel_radius}" scope="parent"/>
