Commit message: Rebase from 'upstream'

File: clearpath_platform_description/urdf/a300/drivetrain/motor.urdf.xacro (robot description, xacro)
@@ -16,4 +16,5 @@
           <mesh filename="package://clearpath_platform_description/meshes/a300/drivetrain/motor.stl"/>
         </geometry>
+        <origin rpy="0 0 ${rotation_yaw}"/>
       </collision>
     </link>

File: clearpath_platform_description/urdf/a300/drivetrain/suspension_beam.urdf.xacro (robot description, xacro)
@@ -4,4 +4,5 @@
     <xacro:property name="rotation_yaw" value="${math.pi if side == 'right' else 0}"/>
     <xacro:property name="spacer_offset" value="${-0.0159 if side == 'right' else 0.0159}"/>
+    <xacro:property name="mount_offset" value="${-0.0095 if side == 'right' else 0.0095}"/>
     <!-- Suspension beam spacer -->
     <link name="${side}_suspension_beam_spacer_link">
@@ -17,4 +18,5 @@
           <mesh filename="package://clearpath_platform_description/meshes/a300/drivetrain/suspension_spacer.stl"/>
         </geometry>
+        <origin rpy="0 0 ${rotation_yaw}"/>
       </collision>
     </link>
@@ -36,4 +38,5 @@
           <mesh filename="package://clearpath_platform_description/meshes/a300/drivetrain/suspension_beam.stl"/>
         </geometry>
+        <origin rpy="0 0 ${rotation_yaw}"/>
       </collision>
     </link>
@@ -49,10 +52,10 @@
       <parent link="${side}_suspension_beam_link"/>
       <child link="${side}_suspension_beam_front_mount"/>
-      <origin xyz="0.256 0.0095 -0.0085" rpy="0 0 0"/>
+      <origin xyz="0.256 ${mount_offset} -0.0085" rpy="0 0 0"/>
     </joint>
     <joint name="${side}_suspension_beam_rear_mount_joint" type="fixed">
       <parent link="${side}_suspension_beam_link"/>
       <child link="${side}_suspension_beam_rear_mount"/>
-      <origin xyz="-0.256 0.0095 -0.0085" rpy="0 0 0"/>
+      <origin xyz="-0.256 ${mount_offset} -0.0085" rpy="0 0 0"/>
     </joint>
   </xacro:macro>

File: clearpath_sensors_description/urdf/intel_realsense.urdf.xacro (robot description, xacro)
@@ -5,5 +5,5 @@
     <xacro:if value="${model == 'd405'}">
       <xacro:include filename="$(find clearpath_sensors_description)/urdf/intel/d405.urdf.xacro" />
-      <xacro:sensor_d405 name="${name}" parent="${parent_link}">
+      <xacro:sensor_d405 name="${name}" parent="${parent_link}" use_nominal_extrinsics="$(arg is_sim)">
         <xacro:insert_block name="origin" />
       </xacro:sensor_d405>
@@ -11,5 +11,5 @@
     <xacro:if value="${model == 'd415'}">
       <xacro:include filename="$(find clearpath_sensors_description)/urdf/intel/d415.urdf.xacro" />
-      <xacro:sensor_d415 name="${name}" parent="${parent_link}">
+      <xacro:sensor_d415 name="${name}" parent="${parent_link}" use_nominal_extrinsics="$(arg is_sim)">
         <xacro:insert_block name="origin" />
       </xacro:sensor_d415>
@@ -17,5 +17,5 @@
     <xacro:if value="${model == 'd435'}">
       <xacro:include filename="$(find clearpath_sensors_description)/urdf/intel/d435.urdf.xacro" />
-      <xacro:sensor_d435 name="${name}" parent="${parent_link}">
+      <xacro:sensor_d435 name="${name}" parent="${parent_link}" use_nominal_extrinsics="$(arg is_sim)">
         <xacro:insert_block name="origin" />
       </xacro:sensor_d435>
@@ -23,5 +23,5 @@
     <xacro:if value="${model == 'd435i'}">
       <xacro:include filename="$(find clearpath_sensors_description)/urdf/intel/d435i.urdf.xacro" />
-      <xacro:sensor_d435i name="${name}" parent="${parent_link}">
+      <xacro:sensor_d435i name="${name}" parent="${parent_link}" use_nominal_extrinsics="$(arg is_sim)">
         <xacro:insert_block name="origin" />
       </xacro:sensor_d435i>
@@ -29,5 +29,5 @@
     <xacro:if value="${model == 'd455'}">
       <xacro:include filename="$(find clearpath_sensors_description)/urdf/intel/d455.urdf.xacro" />
-      <xacro:sensor_d455 name="${name}" parent="${parent_link}">
+      <xacro:sensor_d455 name="${name}" parent="${parent_link}" use_nominal_extrinsics="$(arg is_sim)">
         <xacro:insert_block name="origin" />
       </xacro:sensor_d455>
@@ -35,5 +35,5 @@
     <xacro:if value="${model == 'd456'}">
       <xacro:include filename="$(find clearpath_sensors_description)/urdf/intel/d456.urdf.xacro" />
-      <xacro:sensor_d456 name="${name}" parent="${parent_link}">
+      <xacro:sensor_d456 name="${name}" parent="${parent_link}" use_nominal_extrinsics="$(arg is_sim)">
         <xacro:insert_block name="origin" />
       </xacro:sensor_d456>

File: clearpath_sensors_description/urdf/luxonis_oakd.urdf.xacro (robot description, xacro)
@@ -128,4 +128,5 @@
       <update_rate>${update_rate}</update_rate>
       <visualize>true</visualize>
+      <gz_frame_id>${name}_link</gz_frame_id>
       <topic>$(arg namespace)/sensors/${name}</topic>
     </sensor>
