Commit message: Rebase from 'upstream'

File: clearpath_platform_description/urdf/r100/attachments/hams.urdf.xacro (robot description, xacro)
@@ -75,5 +75,5 @@
     </joint>
     <joint name="${name}_arm_mount_joint" type="fixed">
-      <parent link="${parent_link}" />
+      <parent link="${name}_base_link" />
       <child link="${name}_arm_mount" />
       <origin xyz="${arm_pos_x} ${arm_pos_y} ${mount_height}" rpy="0 0 0"/>
