Commit message: Rebase from 'upstream'

File: clearpath_platform_description/urdf/a300/drivetrain/wheels/caster.urdf.xacro (robot description, xacro)
@@ -36,10 +36,20 @@
       </visual>
     </link>
-    <joint name="${prefix}_${side}_bracket_swivel_joint" type="fixed">
-      <parent link="${prefix}_${side}_bracket_plate_link"/>
-      <child link="${prefix}_${side}_bracket_swivel_link"/>
-      <origin xyz="0 0 -0.006237119"/>
-      <axis xyz="0 0 1"/>
-    </joint>
+    <!-- Simulated as continuous so Gazebo can articulate it, fixed on real hardware since it is not measured. -->
+    <xacro:if value="$(arg is_sim)">
+      <joint name="${prefix}_${side}_bracket_swivel_joint" type="continuous">
+        <parent link="${prefix}_${side}_bracket_plate_link"/>
+        <child link="${prefix}_${side}_bracket_swivel_link"/>
+        <origin xyz="0 0 -0.006237119"/>
+        <axis xyz="0 0 1"/>
+      </joint>
+    </xacro:if>
+    <xacro:unless value="$(arg is_sim)">
+      <joint name="${prefix}_${side}_bracket_swivel_joint" type="fixed">
+        <parent link="${prefix}_${side}_bracket_plate_link"/>
+        <child link="${prefix}_${side}_bracket_swivel_link"/>
+        <origin xyz="0 0 -0.006237119"/>
+      </joint>
+    </xacro:unless>
     <gazebo reference="${prefix}_${side}_bracket_swivel_joint">
       <springStiffness>0.5</springStiffness>
@@ -89,10 +99,20 @@
       </plugin>
     </gazebo> -->
-    <joint name="${prefix}_${side}_wheel_joint" type="continuous">
-      <parent link="${prefix}_${side}_bracket_swivel_link"/>
-      <child link="${prefix}_${side}_wheel_link"/>
-      <origin xyz="-0.054 0 -0.108762881" rpy="0 0 0"/>
-      <axis xyz="0 1 0"/>
-    </joint>
+    <!-- Simulated as continuous so Gazebo can articulate it, fixed on real hardware since it is not measured. -->
+    <xacro:if value="$(arg is_sim)">
+      <joint name="${prefix}_${side}_wheel_joint" type="continuous">
+        <parent link="${prefix}_${side}_bracket_swivel_link"/>
+        <child link="${prefix}_${side}_wheel_link"/>
+        <origin xyz="-0.054 0 -0.108762881" rpy="0 0 0"/>
+        <axis xyz="0 1 0"/>
+      </joint>
+    </xacro:if>
+    <xacro:unless value="$(arg is_sim)">
+      <joint name="${prefix}_${side}_wheel_joint" type="fixed">
+        <parent link="${prefix}_${side}_bracket_swivel_link"/>
+        <child link="${prefix}_${side}_wheel_link"/>
+        <origin xyz="-0.054 0 -0.108762881" rpy="0 0 0"/>
+      </joint>
+    </xacro:unless>
   </xacro:macro>
 </robot>

File: clearpath_sensors_description/urdf/hokuyo_ust.urdf.xacro (robot description, xacro)
@@ -13,4 +13,10 @@
         <material name="clearpath_dark_grey" />
       </visual>
+      <collision>
+        <origin xyz="0.0 0.0 0.04" rpy="0 0 0"/>
+        <geometry>
+          <box size="0.06 0.06 0.08"/>
+        </geometry>
+      </collision>
     </link>
     <link name="${name}_laser">

File: clearpath_sensors_description/urdf/intel_realsense.urdf.xacro (robot description, xacro)
@@ -3,4 +3,10 @@
   <xacro:macro name="intel_realsense" params="name parent_link model *origin
                                               update_rate:=30.0 image_height:=480 image_width:=640">
+    <xacro:if value="${model == 'd405'}">
+      <xacro:include filename="$(find clearpath_sensors_description)/urdf/intel/d405.urdf.xacro" />
+      <xacro:sensor_d405 name="${name}" parent="${parent_link}">
+        <xacro:insert_block name="origin" />
+      </xacro:sensor_d405>
+    </xacro:if>
     <xacro:if value="${model == 'd415'}">
       <xacro:include filename="$(find clearpath_sensors_description)/urdf/intel/d415.urdf.xacro" />
