Commit message: Rebase from 'upstream'

File: clearpath_sensors_description/urdf/intel/d405.urdf.xacro (robot description, xacro)
@@ -21,5 +21,4 @@
 <robot name="sensor_d405" xmlns:xacro="http://ros.org/wiki/xacro">
   <!-- Includes -->
-  <xacro:include filename="$(find realsense2_description)/urdf/_materials.urdf.xacro" />
   <xacro:include filename="$(find realsense2_description)/urdf/_usb_plug.urdf.xacro" />
   <xacro:macro name="sensor_d405" params="parent *origin name:=camera use_nominal_extrinsics:=false">
@@ -68,5 +67,5 @@
           <mesh filename="package://realsense2_description/meshes/d405.stl" scale="0.001 0.001 0.001" />
         </geometry>
-        <material name="aluminum"/>
+        <material name="clearpath_aluminum"/>
       </visual>
       <collision>
